File: EAGLE 9.3.0/EAGLE_Lib/projects/RN41_smartBobber/RN41_Schematic.sch (EAGLE design)
At the start: 1 part

Commit message: Update RN41_Schematic.sch
Changed lines of the file:
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@@
 <parts>
 <part name="J1" library="SparkFun-Connectors" deviceset="CONN_06" device="FEMALE_LOCK"/>
+<part name="R1" library="docu-dummy" library_urn="urn:adsk.eagle:library:215" deviceset="R" device=""/>
 </parts>
 <sheets>
@@
 <attribute name="NAME" x="20.32" y="71.628" size="1.778" layer="95" font="vector"/>
 </instance>
+<instance part="R1" gate="G$1" x="43.18" y="63.5" smashed="yes"/>
 </instances>
 <busses>
@@
 </schematic>
 </drawing>
+<compatibility>
+<note version="8.2" severity="warning">
+Since Version 8.2, EAGLE supports online libraries. The ids
+of those online libraries will not be understood (or retained)
+with this version.
+</note>
+<note version="8.3" severity="warning">
+Since Version 8.3, EAGLE supports URNs for individual library
+assets (packages, symbols, and devices). The URNs of those assets
+will not be understood (or retained) with this version.
+</note>
+</compatibility>
 </eagle>
