File: eagle/projects/RN-41 Board/RN41Board/RN41Board.brd (EAGLE design)
At the start: 38.1 x 16 mm, 18 parts, among them Q1 MOSFET-NCHANNELSMD, U1 BLUETOOTH-RN41, U3 3.3V

Commit message: RN41Board UPDATE
Parts:
- removed J2: (no value), SparkFun-Connectors:JST-5-PTH
- removed U$1: LOGO-SFENEW, SparkFun:SFE-NEW-WEBLOGO
- added J3: (no value), SparkFun-Connectors:1X05
- moved C1 28.4 mm to (5.71, 10.5), turned to 0 degrees
- moved C4 26.0 mm to (6.03, 6.03), turned to 270 degrees
- moved R9 25.2 mm to (4.13, 6.03), turned to 90 degrees
- moved R3 24.2 mm to (8.26, 6.03), turned to 270 degrees
- moved R6 20.8 mm to (16.8, 7.30), turned to 270 degrees
- moved D2 19.7 mm to (14.5, 7.30), turned to 0 degrees
- moved D1 18.4 mm to (12.6, 7.30)
- moved R1 18.3 mm to (10.5, 6.03)
- moved R4 16.2 mm to (21.3, 7.30), turned to 270 degrees
- moved R5 13.4 mm to (19.1, 7.30), turned to 90 degrees
- moved U1 11.6 mm to (19.6, -3.10)
- moved Q1 9.53 mm to (23.8, 6.99)
- moved U3 1.85 mm to (28.3, 6.99)
- moved C3 0.71 mm to (27.9, 10.2), turned to 180 degrees
Connections:
- net GND: now also J3.5; no longer J2.5
- net PIO2: now also J3.1; no longer J2.1
- net RX_5V: now also J3.2; no longer J2.2
- net TX_5V: now also J3.3; no longer J2.3
- net VCC: now also J3.4; no longer J2.4
Routing:
- net VCC: track 0.00 -> 32.2 mm
- net 3.3V: track 0.00 -> 29.2 mm, vias 0 -> 2
- net TX: track 0.00 -> 21.3 mm
- net PIO4: track 0.01 -> 19.2 mm
- net PIO2: track 0.00 -> 6.17 mm
- net N$1: track 0.00 -> 5.57 mm
- net RX_5V: track 0.00 -> 4.10 mm
- net TX_5V: track 0.00 -> 3.33 mm
- net D1: track 0.00 -> 2.64 mm
- net D2: track 3.03 -> 2.39 mm
Other:
- board size 38.1 x 16 mm -> 27.9 x 23 mm
- board text removed: "BlueSMiRF"
- board text removed: "CTS"
- board text removed: "CTS-I"
- board text removed: "GND"
- board text removed: "Gold"
- board text removed: "HID"
- board text removed: "PIO4"
- board text removed: "RTS"
- board text removed: "RTS-O"
- board text removed: "RX-I"
- board text removed: "Silver"
- board text removed: "TX-O"
- board text removed: "V16"
- board text removed: "VCC"

Commit message: RN41 Board UPDATE
Parts:
- moved J3 10.2 mm to (12.1, 10.8), turned to 0 degrees
- moved C1 0.64 mm to (5.71, 11.1)
- moved C3 0.63 mm to (27.9, 10.8)
Routing:
- net 3.3V: track 29.2 -> 51.1 mm
- net RX: track 0.00 -> 11.7 mm, vias 0 -> 2
- net TX: track 21.3 -> 26.9 mm
- net PIO2: track 6.17 -> 11.4 mm
- net TX_5V: track 3.33 -> 8.33 mm
- net VCC: track 32.2 -> 36.6 mm
- net RX_5V: track 4.10 -> 5.54 mm
- net PIO4: track 19.2 -> 20.4 mm
Other:
- board size 27.9 x 23 mm -> 27.9 x 23.6 mm

Commit message: Update
Parts:
- added H2, H3, H4: STAND-OFF, SparkFun-Hardware:STAND-OFF
- added H5: MOUNT-HOLE3.0, holes:3,0
Other:
- board size 27.9 x 23.6 mm -> 32.1 x 23.6 mm
Changed lines of the file:
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@@
 <drawing>
 <settings>
-<setting alwaysvectorfont="no"/>
+<setting alwaysvectorfont="yes"/>
 <setting keepoldvectorfont="yes"/>
 <setting verticaltext="up"/>
@@
 </layers>
 <board>
-<fusionsync huburn="a.cGVyc29uYWw6dWUyYjM3ODg3" projecturn="a.cGVyc29uYWw6dWUyYWMxYjVmIzIwMTgxMDEwMTUzNzU1MDgx" f3durn="urn:adsk.wipprod:dm.lineage:k2WqZ-njSuu7LwTuK9Immw" pcbguid="4452ec3a-aa0f-4bfe-a20e-56efe7cd2703" lastpulledtime="" lastsyncedchangeguid="f65097ca-226c-eff5-f624-b30cac9bbc91"/>
+<fusionsync huburn="a.cGVyc29uYWw6dWUyYjM3ODg3" projecturn="a.cGVyc29uYWw6dWUyYWMxYjVmIzIwMTgxMDEwMTUzNzU1MDgx" f3durn="urn:adsk.wipprod:dm.lineage:k2WqZ-njSuu7LwTuK9Immw" pcbguid="4452ec3a-aa0f-4bfe-a20e-56efe7cd2703" lastpulledtime="" lastsyncedchangeguid="ab07457a-26b4-d7f3-a878-5f0a30939cf6"/>
 <plain>
-<wire x1="3.175" y1="-11.1125" x2="31.115" y2="-11.1125" width="0.2032" layer="20"/>
+<wire x1="-0.9525" y1="-11.1125" x2="31.115" y2="-11.1125" width="0.2032" layer="20"/>
 <wire x1="31.115" y1="-11.1125" x2="31.115" y2="12.5095" width="0.2032" layer="20"/>
-<wire x1="31.115" y1="12.5095" x2="3.175" y2="12.5095" width="0.2032" layer="20"/>
-<wire x1="3.175" y1="12.5095" x2="3.175" y2="-11.1125" width="0.2032" layer="20"/>
+<wire x1="31.115" y1="12.5095" x2="-0.9525" y2="12.5095" width="0.2032" layer="20"/>
+<wire x1="-0.9525" y1="12.5095" x2="-0.9525" y2="-11.1125" width="0.2032" layer="20"/>
 <text x="33.274" y="0.889" size="0.8128" layer="21" font="vector" ratio="15">Stat</text>
 <text x="31.369" y="13.081" size="0.8128" layer="21" font="vector" ratio="15">Connect</text>
@@
 <attribute name="VALUE" x="10.795" y="8.763" size="0.6096" layer="27" font="vector" ratio="20"/>
 </element>
+<element name="H2" library="SparkFun-Hardware" package="STAND-OFF" value="STAND-OFF" x="-26.67" y="-9.525" smashed="yes">
+<attribute name="NAME" x="-26.67" y="-7.493" size="0.6096" layer="25" font="vector" ratio="20" align="bottom-center"/>
+<attribute name="VALUE" x="-26.67" y="-11.557" size="0.6096" layer="27" font="vector" ratio="20" align="top-center"/>
+</element>
+<element name="H3" library="SparkFun-Hardware" package="STAND-OFF" value="STAND-OFF" x="-32.385" y="-9.525" smashed="yes">
+<attribute name="NAME" x="-32.385" y="-7.493" size="0.6096" layer="25" font="vector" ratio="20" align="bottom-center"/>
+<attribute name="VALUE" x="-32.385" y="-11.557" size="0.6096" layer="27" font="vector" ratio="20" align="top-center"/>
+</element>
+<element name="H4" library="SparkFun-Hardware" package="STAND-OFF" value="STAND-OFF" x="-38.1" y="-9.525" smashed="yes">
+<attribute name="NAME" x="-38.1" y="-7.493" size="0.6096" layer="25" font="vector" ratio="20" align="bottom-center"/>
+<attribute name="VALUE" x="-38.1" y="-11.557" size="0.6096" layer="27" font="vector" ratio="20" align="top-center"/>
+</element>
+<element name="H5" library="holes" library_urn="urn:adsk.eagle:library:237" package="3,0" package3d_urn="urn:adsk.eagle:package:14277/1" value="MOUNT-HOLE3.0" x="1.27" y="10.16" smashed="yes"/>
 </elements>
 <signals>
@@
 </drawing>
 <compatibility>
+<note version="8.2" severity="warning">
+Since Version 8.2, EAGLE supports online libraries. The ids
+of those online libraries will not be understood (or retained)
+with this version.
+</note>
 <note version="8.3" severity="warning">
 Since Version 8.3, EAGLE supports Fusion synchronisation.
@@
 the document will break the link to the Fusion PCB feature.
 </note>
+<note version="8.3" severity="warning">
+Since Version 8.3, EAGLE supports URNs for individual library
+assets (packages, symbols, and devices). The URNs of those assets
+will not be understood (or retained) with this version.
+</note>
+<note version="8.3" severity="warning">
+Since Version 8.3, EAGLE supports the association of 3D packages
+with devices in libraries, schematics, and board files. Those 3D
+packages will not be understood (or retained) with this version.
+</note>
 </compatibility>

Commit message: RN41 Updates
Parts:
- removed H2, H3, H4: STAND-OFF, SparkFun-Hardware:STAND-OFF
- removed H5: MOUNT-HOLE3.0, holes:3,0
- removed J3: (no value), SparkFun-Connectors:1X05
- added J1: 640456-5, 640456-5:TE_640456-5
- moved C1 11.2 mm to (6.99, 22.2)
- moved C4 11.2 mm to (7.30, 17.1)
- moved Q1 11.2 mm to (25.1, 18.1)
- moved R1 11.2 mm to (11.7, 17.1)
- moved R3 11.2 mm to (9.53, 17.1)
- moved R9 11.2 mm to (5.40, 17.1)
- moved U3 11.2 mm to (29.5, 18.1)
- moved C3 11.2 mm to (29.2, 21.9)
- moved D1 11.2 mm to (13.9, 18.4)
- moved D2 11.2 mm to (15.7, 18.4)
- moved R4 11.2 mm to (22.5, 18.4)
- moved R5 11.2 mm to (20.3, 18.4)
- moved R6 11.2 mm to (18.1, 18.4)
- moved U1 11.2 mm to (20.8, 8.01)
- moved FRAME1 11.2 mm to (4.02, 2.22)
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Connections:
- net GND: now also J1.5; no longer J3.5
- net PIO2: now also J1.1; no longer J3.1
- net RX_5V: now also J1.2; no longer J3.2
- net TX_5V: now also J1.3; no longer J3.3
- net VCC: now also J1.4; no longer J3.4
Routing:
- net VCC: track 36.6 -> 32.8 mm
- net TX_5V: track 8.33 -> 6.09 mm
- net PIO2: track 11.4 -> 9.17 mm
- net RX_5V: track 5.54 -> 3.29 mm
Other:
- board size 32.1 x 23.6 mm -> 37.8 x 23.6 mm

Commit message: RN41 Update
Parts:
- moved U$2 49.8 mm to (-30.4, 18.7)
- moved C1 28.4 mm to (22.9, -1.27), turned to 270 degrees
- moved U3 25.7 mm to (12.7, -1.27), turned to 270 degrees
- moved C3 24.7 mm to (17.8, 0.00)
- moved R4 15.5 mm to (11.4, 7.62), flipped to the bottom, turned to 180 degrees
- moved Q1 15.2 mm to (11.4, 11.4), flipped to the bottom, turned to 180 degrees
- moved C4 14.2 mm to (17.8, 7.62), flipped to the bottom, turned to 0 degrees
- moved J1 13.4 mm to (27.9, 15.2), flipped to the bottom, turned to 270 degrees
- moved R3 10.0 mm to (17.8, 11.4), flipped to the bottom, turned to 180 degrees
- moved U1 6.00 mm to (15.2, 10.2)
- moved D1 5.81 mm to (10.2, 22.9), turned to 270 degrees
- moved R9 5.72 mm to (10.2, 20.3), turned to 0 degrees
- moved R1 5.65 mm to (15.2, 21.6), turned to 0 degrees
- moved FRAME1 5.39 mm to (-0.98, 4.22)
- moved R6 4.55 mm to (19.1, 22.9), turned to 180 degrees
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Routing:
- net PIO4: track 20.4 -> 4.04 mm
- net TX_5V: track 6.09 -> 19.2 mm
- net RX_5V: track 3.29 -> 15.7 mm
- net VCC: track 32.8 -> 44.4 mm, vias 0 -> 1
- net TX: track 26.9 -> 15.5 mm, vias 0 -> 2
- net PIO2: track 9.17 -> 18.2 mm, vias 0 -> 1
- net 3.3V: track 51.1 -> 42.2 mm
- net RX: track 11.7 -> 6.42 mm, vias 2 -> 0
- net N$1: track 5.57 -> 9.03 mm
- net D1: track 2.64 -> 4.01 mm
- net GND: track 0.81 -> 0.06 mm
Other:
- board size 37.8 x 23.6 mm -> 33 x 27.9 mm
- board text removed: "Connect"
- board text removed: "Stat"

Commit message: Update RN41
Parts:
- removed U$2: REVISION, SparkFun-Aesthetics:REVISION
- moved R9 6.48 mm to (8.89, 26.7), turned to 180 degrees
- moved C4 6.35 mm to (12.7, 11.4)
- moved J1 6.35 mm to (22.9, 19.1)
- moved R3 6.35 mm to (12.7, 15.2)
- moved Q1 6.35 mm to (6.35, 15.2)
- moved R4 6.35 mm to (6.35, 11.4)
- moved U1 6.35 mm to (10.2, 14.0)
- moved R1 5.68 mm to (12.7, 26.7)
- moved D2 5.39 mm to (15.2, 24.1)
- moved R6 4.58 mm to (16.5, 26.7)
- moved C1 4.58 mm to (20.3, 2.54)
- moved C3 4.58 mm to (15.2, 3.81)
- moved FRAME1 4.58 mm to (-3.52, 0.41)
- moved U3 4.58 mm to (10.2, 2.54)
- moved R5 4.58 mm to (20.3, 25.4)
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Routing:
- net N$1: track 9.03 -> 4.60 mm
- net PIO4: track 4.04 -> 7.67 mm
- net RX_5V: track 15.7 -> 12.8 mm
- net VCC: track 44.4 -> 41.6 mm
- net RX: track 6.42 -> 8.46 mm
- net 3.3V: track 42.2 -> 40.4 mm
- net D1: track 4.01 -> 3.46 mm
- net D2: track 2.58 -> 3.11 mm
Other:
- board size 33 x 27.9 mm -> 29.2 x 27.9 mm
- board text added: "3.3V"
- board text added: "CONN"
- board text added: "GND"
- board text added: "PIO2"
- board text added: "RX"
- board text added: "STAT"
- board text added: "TX"
- board text added: "smartBobber"

Commit message: Update RN41Board.brd
Parts:
- moved R6 1.27 mm to (17.8, 26.7), turned to 0 degrees
Routing:
- net N$1: track 4.60 -> 3.97 mm
- added copper zone on layer 1, net GND
- added copper zone on layer 16, net GND

Commit message: RN-41 Complete
Parts:
- moved R9 13.3 mm to (5.08, 14.0), flipped to the bottom, turned to 90 degrees
- moved R5 10.9 mm to (14.0, 16.5), flipped to the bottom, turned to 180 degrees
- moved C4 2.84 mm to (15.2, 12.7), turned to 90 degrees
- moved D2 2.84 mm to (17.8, 25.4), turned to 0 degrees
- moved Q1 2.84 mm to (8.89, 14.0)
- moved R6 2.84 mm to (20.3, 25.4), turned to 270 degrees
- moved R3 2.54 mm to (12.7, 12.7), turned to 90 degrees
- moved R1 1.80 mm to (11.4, 25.4), turned to 270 degrees
- moved R4 1.80 mm to (7.62, 10.2)
- moved D1 1.27 mm to (8.89, 25.4), turned to 0 degrees
Routing:
- net 3.3V: track 40.4 -> 21.1 mm, vias 2 -> 1
- net RX_5V: track 12.8 -> 8.04 mm
- net TX_5V: track 19.2 -> 22.1 mm
- net TX: track 15.5 -> 12.9 mm, vias 2 -> 1
- net PIO2: track 18.2 -> 19.9 mm, vias 1 -> 0
- net VCC: track 41.5 -> 40.0 mm
- net RX: track 7.99 -> 6.81 mm, vias 0 -> 1
- net D1: track 3.76 -> 2.58 mm
- net PIO4: track 7.21 -> 6.11 mm, vias 0 -> 1
- net N$1: track 3.97 -> 4.80 mm
