File: eagle/projects/RN-41 Board/RN41Board/RN41Board.brd (EAGLE design)
At the start: 29.2 x 27.9 mm, 16 parts, among them J1 640456-5, Q1 MOSFET-NCHANNELSMD, U1 BLUETOOTH-RN41, U3 3.3V

Commit message: Update RN41Board.brd
Routing:
- net GND: track 0.06 -> 0.00 mm, vias 1 -> 2
Changed lines of the file:
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@@
 <drawing>
 <settings>
-<setting alwaysvectorfont="yes"/>
+<setting alwaysvectorfont="no"/>
 <setting keepoldvectorfont="yes"/>
 <setting verticaltext="up"/>
@@
 <hole x="26.67" y="25.4" drill="2.99999375"/>
 <hole x="26.67" y="2.54" drill="2.99999375"/>
-<text x="29.21" y="6.35" size="1.778" layer="21" rot="R90">smartBobber</text>
+<text x="28.575" y="6.35" size="1.778" layer="21" rot="R90">smartBobber</text>
 <text x="26.67" y="20.32" size="0.8128" layer="21" rot="R180">PIO2</text>
 <text x="24.13" y="16.51" size="0.8128" layer="21">RX</text>
@@
 <contactref element="R6" pad="2"/>
 <contactref element="R9" pad="1"/>
-<wire x1="19.56" y1="10.87" x2="19.599" y2="10.909" width="0.254" layer="1"/>
 <via x="4.144" y="10.255" extent="1-16" drill="0.508"/>
 <contactref element="J1" pad="5"/>
@@
 <vertex x="2.54" y="5.08"/>
 </polygon>
+<via x="22.86" y="24.13" extent="1-16" drill="0.35"/>
 </signal>
 <signal name="TX">

Commit message: Update RN41Board.brd
Parts:
- moved R1 1.27 mm to (12.7, 25.4)
- moved R6 1.27 mm to (21.6, 25.4)
Routing:
- net D2: track 2.58 -> 3.85 mm
- net D1: track 2.58 -> 3.85 mm
Changed lines of the file:
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@@
 <drawing>
 <settings>
-<setting alwaysvectorfont="no"/>
+<setting alwaysvectorfont="yes"/>
 <setting keepoldvectorfont="yes"/>
 <setting verticaltext="up"/>
 </settings>
-<grid distance="0.05" unitdist="inch" unit="inch" style="lines" multiple="1" display="yes" altdistance="0.005" altunitdist="inch" altunit="inch"/>
+<grid distance="0.05" unitdist="inch" unit="mil" style="lines" multiple="1" display="yes" altdistance="0.005" altunitdist="inch" altunit="inch"/>
 <layers>
 <layer number="1" name="Top" color="4" fill="1" visible="yes" active="yes"/>
@@
 </layers>
 <board>
-<fusionsync huburn="a.cGVyc29uYWw6dWUyYjM3ODg3" projecturn="a.cGVyc29uYWw6dWUyYWMxYjVmIzIwMTgxMDEwMTUzNzU1MDgx" f3durn="urn:adsk.wipprod:dm.lineage:k2WqZ-njSuu7LwTuK9Immw" pcbguid="4452ec3a-aa0f-4bfe-a20e-56efe7cd2703" lastpulledtime="" lastsyncedchangeguid="49f6bae7-4b09-7fad-3a19-45946278e437"/>
+<fusionsync huburn="a.cGVyc29uYWw6dWUyYjM3ODg3" projecturn="a.cGVyc29uYWw6dWUyYWMxYjVmIzIwMTgxMDEwMTUzNzU1MDgx" f3durn="urn:adsk.wipprod:dm.lineage:k2WqZ-njSuu7LwTuK9Immw" pcbguid="4452ec3a-aa0f-4bfe-a20e-56efe7cd2703" lastpulledtime="" lastsyncedchangeguid="15ca1456-0d3a-be79-2579-b16d677f4cd2"/>
 <plain>
 <wire x1="0" y1="0" x2="29.21" y2="0" width="0.2032" layer="20"/>
@@
 <hole x="26.67" y="2.54" drill="2.99999375"/>
 <text x="28.575" y="6.35" size="1.778" layer="21" rot="R90">smartBobber</text>
-<text x="26.67" y="20.32" size="0.8128" layer="21" rot="R180">PIO2</text>
-<text x="24.13" y="16.51" size="0.8128" layer="21">RX</text>
-<text x="24.13" y="13.97" size="0.8128" layer="21">TX</text>
-<text x="24.13" y="11.43" size="0.8128" layer="21">3.3V</text>
-<text x="24.13" y="8.89" size="0.8128" layer="21">GND</text>
-<text x="19.05" y="19.05" size="0.8128" layer="22" rot="MR0">PIO2</text>
-<text x="19.05" y="16.51" size="0.8128" layer="22" rot="MR0">RX</text>
-<text x="19.05" y="13.97" size="0.8128" layer="22" rot="MR0">TX</text>
-<text x="19.05" y="11.43" size="0.8128" layer="22" rot="MR0">3.3V</text>
-<text x="19.05" y="8.89" size="0.8128" layer="22" rot="MR0">GND</text>
-<text x="7.62" y="22.86" size="1.016" layer="21" rot="R90">STAT</text>
-<text x="16.51" y="22.86" size="1.016" layer="21" rot="R90">CONN</text>
+<text x="26.416" y="19.431" size="0.8128" layer="21" rot="R180">PIO2</text>
+<text x="24.003" y="16.129" size="0.8128" layer="21">RX</text>
+<text x="24.003" y="13.589" size="0.8128" layer="21">TX</text>
+<text x="24.003" y="11.049" size="0.8128" layer="21">3.3V</text>
+<text x="24.003" y="8.509" size="0.8128" layer="21">GND</text>
+<text x="19.812" y="18.669" size="1.016" layer="22" rot="MR0">PIO2</text>
+<text x="19.685" y="16.002" size="1.016" layer="22" rot="MR0">RX</text>
+<text x="19.812" y="13.462" size="1.016" layer="22" rot="MR0">TX</text>
+<text x="19.812" y="11.049" size="0.8128" layer="22" rot="MR0">3.3V</text>
+<text x="19.939" y="8.509" size="0.8128" layer="22" rot="MR0">GND</text>
+<text x="8.128" y="23.241" size="1.27" layer="21" rot="R90">STAT</text>
+<text x="17.145" y="22.479" size="1.27" layer="21" rot="R90">CONN</text>
 <circle x="11.43" y="5.08" radius="2.83980625" width="0.254" layer="22"/>
 <wire x1="13.97" y1="5.08" x2="15.24" y2="5.08" width="0.254" layer="22"/>
@@
 <elements>
 <element name="C4" library="SparkFun" package="0603-CAP" value="1uF" x="15.24" y="12.7" smashed="yes" rot="MR90">
-<attribute name="NAME" x="13.97" y="12.7" size="0.4064" layer="26" rot="MR90"/>
+<attribute name="NAME" x="13.335" y="11.557" size="1.27" layer="26" rot="MR90"/>
 <attribute name="VALUE" x="14.3256" y="11.5443" size="0.4064" layer="28" rot="MR90"/>
 </element>
 <element name="U3" library="SparkFun" package="SOT23-5" value="3.3V" x="10.16" y="2.54" smashed="yes" rot="R270">
-<attribute name="NAME" x="10.884" y="4.746" size="0.4064" layer="25" rot="R90"/>
-</element>
-<element name="R1" library="SparkFun" package="0603-RES" value="330" x="11.43" y="25.4" smashed="yes" rot="R270">
-<attribute name="NAME" x="12.7" y="24.13" size="0.4064" layer="25" rot="R90"/>
-<attribute name="VALUE" x="12.0142" y="25.2857" size="0.4064" layer="27" rot="R270"/>
+<attribute name="NAME" x="11.256" y="5.423" size="1.27" layer="25" rot="R180"/>
+</element>
+<element name="R1" library="SparkFun" package="0603-RES" value="330" x="12.7" y="25.4" smashed="yes" rot="R270">
+<attribute name="NAME" x="14.732" y="24.13" size="1.27" layer="25" rot="R90"/>
+<attribute name="VALUE" x="13.2842" y="25.2857" size="0.4064" layer="27" rot="R270"/>
 </element>
 <element name="C1" library="SparkFun" package="EIA3216" value="10uF" x="20.32" y="2.54" smashed="yes" rot="R270">
-<attribute name="NAME" x="22.6982" y="2.7244" size="0.4064" layer="25" rot="R90"/>
+<attribute name="NAME" x="21.4056" y="6.5692" size="1.27" layer="25" rot="R180"/>
 <attribute name="VALUE" x="20.2708" y="5.2182" size="0.4064" layer="27"/>
 </element>
 <element name="C3" library="SparkFun" package="EIA3216" value="10uF" x="15.24" y="3.81" smashed="yes" rot="R180">
-<attribute name="NAME" x="15.4526" y="2.3368" size="0.4064" layer="25" rot="R270"/>
+<attribute name="NAME" x="14.1732" y="1.1016" size="1.27" layer="25"/>
 <attribute name="VALUE" x="17.9944" y="3.8592" size="0.4064" layer="27" rot="R270"/>
 </element>
 <element name="Q1" library="SparkFun" package="SOT23-3" value="MOSFET-NCHANNELSMD" x="8.89" y="13.97" smashed="yes" rot="MR180">
-<attribute name="NAME" x="6.35" y="13.97" size="0.4064" layer="26" rot="MR90"/>
+<attribute name="NAME" x="7.366" y="15.367" size="1.27" layer="26" rot="MR270"/>
 <attribute name="VALUE" x="10.901" y="15.0112" size="0.4064" layer="28" rot="MR270"/>
 </element>
 <element name="R3" library="SparkFun" package="0603-RES" value="10K" x="12.7" y="12.7" smashed="yes" rot="MR90">
-<attribute name="NAME" x="11.43" y="12.7" size="0.4064" layer="26" rot="MR90"/>
+<attribute name="NAME" x="10.795" y="11.684" size="1.27" layer="26" rot="MR90"/>
 <attribute name="VALUE" x="11.7602" y="11.6967" size="0.4064" layer="28" rot="MR90"/>
 </element>
 <element name="R4" library="SparkFun" package="0603-RES" value="10K" x="7.62" y="10.16" smashed="yes" rot="MR180">
-<attribute name="NAME" x="7.62" y="11.43" size="0.4064" layer="26" rot="MR270"/>
+<attribute name="NAME" x="6.096" y="11.049" size="1.27" layer="26" rot="MR270"/>
 <attribute name="VALUE" x="6.4897" y="11.1252" size="0.4064" layer="28" rot="MR180"/>
 </element>
 <element name="R5" library="SparkFun" package="0603-RES" value="10K" x="13.97" y="16.51" smashed="yes" rot="MR180">
-<attribute name="NAME" x="13.97" y="15.24" size="0.4064" layer="26" rot="MR0"/>
+<attribute name="NAME" x="12.319" y="17.653" size="1.27" layer="26" rot="MR270"/>
 <attribute name="VALUE" x="13.9573" y="17.5006" size="0.4064" layer="28" rot="MR180"/>
 </element>
 <element name="D2" library="SparkFun" package="LED-0603" value="Green" x="17.78" y="25.4" smashed="yes">
-<attribute name="NAME" x="19.05" y="24.13" size="0.4064" layer="25" rot="R90"/>
+<attribute name="NAME" x="19.685" y="24.13" size="1.27" layer="25" rot="R90"/>
 <attribute name="VALUE" x="18.8341" y="24.638" size="0.4064" layer="27" ratio="12" rot="R90"/>
 </element>
-<element name="R6" library="SparkFun" package="0603-RES" value="330" x="20.32" y="25.4" smashed="yes" rot="R270">
-<attribute name="NAME" x="21.59" y="24.13" size="0.4064" layer="25" rot="R90"/>
-<attribute name="VALUE" x="19.4056" y="25.2603" size="0.4064" layer="27" rot="R270"/>
+<element name="R6" library="SparkFun" package="0603-RES" value="330" x="21.59" y="25.4" smashed="yes" rot="R270">
+<attribute name="NAME" x="23.622" y="24.13" size="1.27" layer="25" rot="R90"/>
+<attribute name="VALUE" x="20.6756" y="25.2603" size="0.4064" layer="27" rot="R270"/>
 </element>
 <element name="U1" library="SparkFun-RF" package="RN41" value="BLUETOOTH-RN41" x="10.16" y="13.97" smashed="yes"/>
 <element name="D1" library="SparkFun" package="LED-0603" value="Red" x="8.89" y="25.4" smashed="yes">
-<attribute name="NAME" x="10.16" y="24.13" size="0.4064" layer="25" rot="R90"/>
+<attribute name="NAME" x="10.922" y="24.13" size="1.27" layer="25" rot="R90"/>
 <attribute name="VALUE" x="8.1915" y="25.019" size="0.4064" layer="27" ratio="12" rot="R90"/>
 </element>
 <element name="R9" library="SparkFun" package="0603-RES" value="10K" x="5.08" y="13.97" smashed="yes" rot="MR90">
-<attribute name="NAME" x="3.81" y="13.97" size="0.4064" layer="26" rot="MR90"/>
+<attribute name="NAME" x="3.175" y="13.081" size="1.27" layer="26" rot="MR90"/>
 <attribute name="VALUE" x="5.6388" y="12.9667" size="0.4064" layer="28" rot="MR90"/>
 </element>
@@
 <vertex x="2.54" y="5.08"/>
 </polygon>
-<via x="22.86" y="24.13" extent="1-16" drill="0.35"/>
+<via x="24.13" y="22.86" extent="1-16" drill="0.35"/>
 </signal>
 <signal name="TX">
@@
 <contactref element="D1" pad="C"/>
 <wire x1="8.89" y1="26.15" x2="8.99" y2="26.25" width="0.254" layer="1"/>
-<wire x1="8.99" y1="26.25" x2="11.43" y2="26.25" width="0.254" layer="1"/>
+<wire x1="8.99" y1="26.25" x2="12.7" y2="26.25" width="0.254" layer="1"/>
 </signal>
 <signal name="RX">
@@
 <contactref element="R6" pad="1"/>
 <wire x1="17.78" y1="26.15" x2="17.88" y2="26.25" width="0.254" layer="1"/>
-<wire x1="17.88" y1="26.25" x2="20.32" y2="26.25" width="0.254" layer="1"/>
+<wire x1="17.88" y1="26.25" x2="21.59" y2="26.25" width="0.254" layer="1"/>
 </signal>
 <signal name="N$1">
