File: eagle/projects/RN-41 Board/RN41Board/RN41Board.brd (EAGLE design)
At the start: 29.2 x 27.9 mm, 16 parts, among them J1 640456-5, Q1 MOSFET-NCHANNELSMD, U1 BLUETOOTH-RN41, U3 3.3V

Commit message: OSHPark .dru and RN-41 Update
Parts:
- removed FRAME1: FRAME-LETTER, SparkFun-Aesthetics:CREATIVE_COMMONS
- moved C1 1.27 mm to (20.3, 3.81)
- moved U3 1.27 mm to (10.2, 3.81)
Routing:
- net VCC: track 40.0 -> 38.9 mm
Other:
- board text removed: "J. Lindblom"
- board text removed: "T. Klopfenstein"

Commit message: Update
Connections:
- net RX_5V: now also J1.3; no longer J1.2
- net TX_5V: now also J1.2; no longer J1.3
Routing:
- net RX_5V: track 8.04 -> 16.0 mm
- net TX_5V: track 22.1 -> 24.6 mm
Changed lines of the file:
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@@
 <drawing>
 <settings>
-<setting alwaysvectorfont="yes"/>
+<setting alwaysvectorfont="no"/>
 <setting keepoldvectorfont="yes"/>
 <setting verticaltext="up"/>
 </settings>
-<grid distance="0.05" unitdist="inch" unit="mm" style="lines" multiple="1" display="yes" altdistance="0.005" altunitdist="inch" altunit="inch"/>
+<grid distance="0.05" unitdist="inch" unit="mil" style="lines" multiple="1" display="yes" altdistance="0.005" altunitdist="inch" altunit="inch"/>
 <layers>
 <layer number="1" name="Top" color="4" fill="1" visible="yes" active="yes"/>
@@
 <contactref element="Q1" pad="3"/>
 <contactref element="R4" pad="2"/>
-<contactref element="J1" pad="3"/>
 <wire x1="8.47" y1="10.16" x2="8.89" y2="10.58" width="0.254" layer="16"/>
 <wire x1="8.89" y1="10.58" x2="8.89" y2="12.87" width="0.254" layer="16"/>
 <wire x1="8.89" y1="12.87" x2="12.87" y2="8.89" width="0.254" layer="16"/>
-<wire x1="12.87" y1="8.89" x2="20.32" y2="8.89" width="0.254" layer="16"/>
-<wire x1="20.32" y1="8.89" x2="20.32" y2="11.43" width="0.254" layer="16"/>
-<wire x1="20.32" y1="11.43" x2="22.86" y2="13.97" width="0.254" layer="16"/>
+<wire x1="20.32" y1="8.89" x2="12.87" y2="8.89" width="0.254" layer="16"/>
+<contactref element="J1" pad="2"/>
+<wire x1="22.86" y1="16.51" x2="20.32" y2="13.97" width="0.254" layer="16"/>
+<wire x1="20.32" y1="13.97" x2="20.32" y2="8.89" width="0.254" layer="16"/>
 </signal>
 <signal name="D1">
@@
 <signal name="RX_5V">
 <contactref element="R5" pad="2"/>
-<contactref element="J1" pad="2"/>
-<wire x1="14.82" y1="16.51" x2="22.86" y2="16.51" width="0.254" layer="16"/>
+<contactref element="J1" pad="3"/>
+<wire x1="14.82" y1="16.51" x2="20.32" y2="16.51" width="0.254" layer="16"/>
+<wire x1="20.32" y1="16.51" x2="21.59" y2="17.78" width="0.254" layer="16"/>
+<wire x1="21.59" y1="17.78" x2="24.13" y2="17.78" width="0.254" layer="16"/>
+<wire x1="24.13" y1="17.78" x2="25.4" y2="16.51" width="0.254" layer="16"/>
+<wire x1="25.4" y1="16.51" x2="25.4" y2="15.24" width="0.254" layer="16"/>
+<wire x1="25.4" y1="15.24" x2="24.13" y2="13.97" width="0.254" layer="16"/>
+<wire x1="24.13" y1="13.97" x2="22.86" y2="13.97" width="0.254" layer="16"/>
 </signal>
 <signal name="VCC">
