File: eagle/projects/HutsonProjects/Design/PCB_Tutorial.brd (EAGLE design)
At the start: 160 x 100 mm, 15 parts, among them J1 POWER_JACKPTH_BREAD, J3 AVR_SPI_PROG_3X2PTH, J4 6_PIN_SERIAL_CABLEPTH, U1 328P

Commit message: Dimensions
Parts:
- moved J4 18.6 mm to (14.8, 54.0)
- moved J3 7.75 mm to (28.5, 44.3)
- moved J2 6.74 mm to (50.8, 72.6)
- moved U1 6.34 mm to (31.2, 70.0), turned to 270 degrees
- moved R2 5.90 mm to (45.6, 61.5)
- moved D1 5.83 mm to (45.5, 67.5)
- moved D2 5.41 mm to (45.8, 55.8)
- moved R3 5.25 mm to (46.2, 50.1)
- moved D3 5.16 mm to (46.3, 44.2)
- moved R4 4.47 mm to (47.0, 38.9)
- moved C2 3.93 mm to (24.1, 68.1)
Other:
- board size 160 x 100 mm -> 41.9 x 57.2 mm

Commit message: routing
Routing:
- net VCC: track 0.00 -> 48.5 mm
- net N$8: track 0.00 -> 16.4 mm
- net N$5: track 0.00 -> 16.4 mm
- net N$3: track 0.00 -> 16.4 mm
- net N$6: track 0.00 -> 16.4 mm
- net N$4: track 0.00 -> 16.4 mm
- net N$7: track 0.00 -> 16.3 mm
Changed lines of the file:
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@@
 <contactref element="J4" pad="GND"/>
 <contactref element="J3" pad="6"/>
-<wire x1="41.749978125" y1="61.52769375" x2="50.7657125" y2="90.410028125" width="0" layer="19" extent="1-1"/>
-<wire x1="27.381203125" y1="68.712078125" x2="41.749978125" y2="61.52769375" width="0" layer="19" extent="1-1"/>
-<wire x1="35.001203125" y1="71.252078125" x2="27.381203125" y2="68.712078125" width="0" layer="19" extent="1-1"/>
-<wire x1="42.35323125" y1="50.1294375" x2="41.749978125" y2="61.52769375" width="0" layer="19" extent="1-1"/>
-<wire x1="43.1507875" y1="38.8874" x2="42.35323125" y2="50.1294375" width="0" layer="19" extent="1-1"/>
-<wire x1="33.55975" y1="46.79315" x2="43.1507875" y2="38.8874" width="0" layer="19" extent="1-1"/>
-<wire x1="19.203671875" y1="75.1078" x2="35.001203125" y2="71.252078125" width="0" layer="19" extent="1-1"/>
+<wire x1="50.7657125" y1="90.410028125" x2="35.001203125" y2="71.252078125" width="0" layer="19" extent="1-1"/>
+<wire x1="27.381203125" y1="68.712078125" x2="35.001203125" y2="71.252078125" width="0" layer="19" extent="1-1"/>
+<wire x1="19.203671875" y1="75.1078" x2="27.381203125" y2="68.712078125" width="0" layer="19" extent="1-1"/>
 <wire x1="19.9862375" y1="83.23131875" x2="19.203671875" y2="75.1078" width="0" layer="19" extent="1-1"/>
 <wire x1="17.1862375" y1="88.03131875" x2="19.9862375" y2="83.23131875" width="0" layer="19" extent="1-1"/>
-<wire x1="14.801853125" y1="66.737228125" x2="35.001203125" y2="71.252078125" width="0" layer="19" extent="1-1"/>
+<wire x1="14.801853125" y1="66.737228125" x2="19.203671875" y2="75.1078" width="0" layer="19" extent="1-1"/>
+<wire x1="41.749978125" y1="61.52769375" x2="35.001203125" y2="71.252078125" width="0" layer="19" extent="1-1"/>
+<wire x1="42.35323125" y1="50.1294375" x2="41.749978125" y2="61.52769375" width="0" layer="19" extent="1-1"/>
+<wire x1="33.55975" y1="46.79315" x2="42.35323125" y2="50.1294375" width="0" layer="19" extent="1-1"/>
+<wire x1="43.1507875" y1="38.8874" x2="42.35323125" y2="50.1294375" width="0" layer="19" extent="1-1"/>
 </signal>
 <signal name="VCC">
@@
 <contactref element="J4" pad="VCC"/>
 <contactref element="J3" pad="2"/>
-<wire x1="27.381203125" y1="71.252078125" x2="50.7657125" y2="72.630028125" width="0" layer="19" extent="1-1"/>
-<wire x1="35.001203125" y1="66.172078125" x2="27.381203125" y2="71.252078125" width="0" layer="19" extent="1-1"/>
-<wire x1="21.69921875" y1="78.70316875" x2="35.001203125" y2="66.172078125" width="0" layer="19" extent="1-1"/>
+<wire x1="50.7657125" y1="72.630028125" x2="43.420028125" y2="72.630028125" width="0.1524" layer="1"/>
+<wire x1="36.962078125" y1="66.172078125" x2="35.001203125" y2="66.172078125" width="0.1524" layer="1"/>
+<wire x1="43.420028125" y1="72.630028125" x2="36.962078125" y2="66.172078125" width="0.1524" layer="1"/>
+<wire x1="27.807921875" y1="71.252078125" x2="27.381203125" y2="71.252078125" width="0.1524" layer="1"/>
+<wire x1="24.23921875" y1="86.7783375" x2="24.23921875" y2="81.24316875" width="0.1524" layer="1"/>
+<wire x1="21.69921875" y1="78.70316875" x2="24.23921875" y2="81.24316875" width="0.1524" layer="1"/>
+<wire x1="22.9862375" y1="88.03131875" x2="24.23921875" y2="86.7783375" width="0.1524" layer="1"/>
+<wire x1="26.3398" y1="73.36071875" x2="26.3398" y2="74.0625875" width="0.1524" layer="1"/>
+<wire x1="26.3398" y1="74.0625875" x2="21.69921875" y2="78.70316875" width="0.1524" layer="1"/>
+<wire x1="27.381203125" y1="71.252078125" x2="27.381203125" y2="72.319315625" width="0.1524" layer="1"/>
+<wire x1="27.381203125" y1="72.319315625" x2="26.3398" y2="73.36071875" width="0.1524" layer="1"/>
+<wire x1="35.001203125" y1="66.172078125" x2="30.48" y2="68.58" width="0.1524" layer="1" curve="-56.07813"/>
+<wire x1="30.48" y1="68.58" x2="27.807921875" y2="71.252078125" width="0.1524" layer="1" curve="22.156273"/>
 <wire x1="16.409671875" y1="75.1078" x2="21.69921875" y2="78.70316875" width="0" layer="19" extent="1-1"/>
-<wire x1="22.9862375" y1="88.03131875" x2="21.69921875" y2="78.70316875" width="0" layer="19" extent="1-1"/>
-<wire x1="28.47975" y1="46.79315" x2="27.381203125" y2="71.252078125" width="0" layer="19" extent="1-1"/>
-<wire x1="14.801853125" y1="61.657228125" x2="28.47975" y2="46.79315" width="0" layer="19" extent="1-1"/>
+<wire x1="14.801853125" y1="61.657228125" x2="16.409671875" y2="75.1078" width="0" layer="19" extent="1-1"/>
+<wire x1="28.47975" y1="46.79315" x2="14.801853125" y2="61.657228125" width="0" layer="19" extent="1-1"/>
 </signal>
 <signal name="N$3">
 <contactref element="U1" pad="23"/>
 <contactref element="J2" pad="2"/>
-<wire x1="35.001203125" y1="73.792078125" x2="50.7657125" y2="75.170028125" width="0" layer="19" extent="1-1"/>
+<wire x1="50.7657125" y1="75.170028125" x2="48.500028125" y2="75.170028125" width="0.1524" layer="1"/>
+<wire x1="48.500028125" y1="75.170028125" x2="46.99" y2="73.66" width="0.1524" layer="1"/>
+<wire x1="46.99" y1="73.66" x2="35.13328125" y2="73.66" width="0.1524" layer="1"/>
+<wire x1="35.13328125" y1="73.66" x2="35.001203125" y2="73.792078125" width="0.1524" layer="1"/>
 </signal>
 <signal name="N$4">
 <contactref element="U1" pad="24"/>
 <contactref element="J2" pad="3"/>
-<wire x1="35.001203125" y1="76.332078125" x2="50.7657125" y2="77.710028125" width="0" layer="19" extent="1-1"/>
+<wire x1="50.7657125" y1="77.710028125" x2="48.500028125" y2="77.710028125" width="0.1524" layer="1"/>
+<wire x1="48.500028125" y1="77.710028125" x2="46.99" y2="76.2" width="0.1524" layer="1"/>
+<wire x1="46.99" y1="76.2" x2="35.13328125" y2="76.2" width="0.1524" layer="1"/>
+<wire x1="35.13328125" y1="76.2" x2="35.001203125" y2="76.332078125" width="0.1524" layer="1"/>
 </signal>
 <signal name="N$5">
 <contactref element="U1" pad="25"/>
 <contactref element="J2" pad="4"/>
-<wire x1="35.001203125" y1="78.872078125" x2="50.7657125" y2="80.250028125" width="0" layer="19" extent="1-1"/>
+<wire x1="50.7657125" y1="80.250028125" x2="48.500028125" y2="80.250028125" width="0.1524" layer="1"/>
+<wire x1="48.500028125" y1="80.250028125" x2="46.99" y2="78.74" width="0.1524" layer="1"/>
+<wire x1="46.99" y1="78.74" x2="35.13328125" y2="78.74" width="0.1524" layer="1"/>
+<wire x1="35.13328125" y1="78.74" x2="35.001203125" y2="78.872078125" width="0.1524" layer="1"/>
 </signal>
 <signal name="N$6">
 <contactref element="U1" pad="26"/>
 <contactref element="J2" pad="5"/>
-<wire x1="35.001203125" y1="81.412078125" x2="50.7657125" y2="82.790028125" width="0" layer="19" extent="1-1"/>
+<wire x1="50.7657125" y1="82.790028125" x2="48.500028125" y2="82.790028125" width="0.1524" layer="1"/>
+<wire x1="48.500028125" y1="82.790028125" x2="46.99" y2="81.28" width="0.1524" layer="1"/>
+<wire x1="46.99" y1="81.28" x2="35.13328125" y2="81.28" width="0.1524" layer="1"/>
+<wire x1="35.13328125" y1="81.28" x2="35.001203125" y2="81.412078125" width="0.1524" layer="1"/>
 </signal>
 <signal name="N$7">
 <contactref element="U1" pad="27"/>
 <contactref element="J2" pad="6"/>
-<wire x1="35.001203125" y1="83.952078125" x2="50.7657125" y2="85.330028125" width="0" layer="19" extent="1-1"/>
+<wire x1="50.7657125" y1="85.330028125" x2="49.3877625" y2="83.952078125" width="0.1524" layer="1"/>
+<wire x1="49.3877625" y1="83.952078125" x2="35.001203125" y2="83.952078125" width="0.1524" layer="1"/>
 </signal>
 <signal name="N$8">
 <contactref element="U1" pad="28"/>
 <contactref element="J2" pad="7"/>
-<wire x1="35.001203125" y1="86.492078125" x2="50.7657125" y2="87.870028125" width="0" layer="19" extent="1-1"/>
+<wire x1="50.7657125" y1="87.870028125" x2="48.500028125" y2="87.870028125" width="0.1524" layer="1"/>
+<wire x1="48.500028125" y1="87.870028125" x2="46.99" y2="86.36" width="0.1524" layer="1"/>
+<wire x1="46.99" y1="86.36" x2="35.13328125" y2="86.36" width="0.1524" layer="1"/>
+<wire x1="35.13328125" y1="86.36" x2="35.001203125" y2="86.492078125" width="0.1524" layer="1"/>
 </signal>
 <signal name="N$9">
@@
 <contactref element="U1" pad="14"/>
 <contactref element="D3" pad="A"/>
-<wire x1="45.06468125" y1="44.203625" x2="27.381203125" y2="53.472078125" width="0" layer="19" extent="1-1"/>
+<wire x1="27.381203125" y1="53.472078125" x2="45.06468125" y2="44.203625" width="0" layer="19" extent="1-1"/>
 </signal>
 <signal name="N$13">
 <contactref element="U1" pad="15"/>
 <contactref element="D2" pad="A"/>
-<wire x1="44.571921875" y1="55.79871875" x2="35.001203125" y2="53.472078125" width="0" layer="19" extent="1-1"/>
+<wire x1="35.001203125" y1="53.472078125" x2="44.571921875" y2="55.79871875" width="0" layer="19" extent="1-1"/>
 </signal>
 <signal name="N$14">
@@
 <contactref element="U1" pad="1"/>
 <contactref element="R1" pad="P$1"/>
-<wire x1="14.07921875" y1="78.70316875" x2="24.062690625" y2="69.52106875" width="0" layer="19" extent="1-1"/>
-<wire x1="27.381203125" y1="86.492078125" x2="24.062690625" y2="69.52106875" width="0" layer="19" extent="1-1"/>
-<wire x1="33.55975" y1="44.25315" x2="27.381203125" y2="86.492078125" width="0" layer="19" extent="1-1"/>
+<wire x1="14.07921875" y1="78.70316875" x2="27.381203125" y2="86.492078125" width="0" layer="19" extent="1-1"/>
+<wire x1="24.062690625" y1="69.52106875" x2="14.07921875" y2="78.70316875" width="0" layer="19" extent="1-1"/>
+<wire x1="33.55975" y1="44.25315" x2="24.062690625" y2="69.52106875" width="0" layer="19" extent="1-1"/>
 </signal>
 </signals>

Commit message: finished routing
Routing:
- net GND: track 0.00 -> 120.6 mm
- net RESET: track 0.00 -> 63.6 mm, vias 0 -> 1
- net VCC: track 48.5 -> 98.3 mm, vias 0 -> 1
- net TX: track 0.00 -> 31.2 mm, vias 0 -> 1
- net SCK: track 0.00 -> 30.8 mm, vias 0 -> 1
- net N$12: track 0.00 -> 29.9 mm
- net RX: track 0.00 -> 29.6 mm, vias 0 -> 3
- net MISO: track 0.00 -> 20.2 mm
- net DTR: track 0.00 -> 17.8 mm, vias 0 -> 2
- net N$14: track 0.00 -> 14.7 mm
- net MOSI: track 0.00 -> 13.6 mm
- net N$13: track 0.00 -> 9.85 mm
- net N$9: track 0.00 -> 6.46 mm
- net N$10: track 0.00 -> 6.35 mm
- net N$11: track 0.00 -> 6.19 mm
