File: eagle/projects/smartBobber Mother Board/motherBoard/motherboard_Embedded.sch (EAGLE design)
At the start: 26 parts, among them Q1 2A/20V/150mΩ, Q2 MMBT3904, Y1 ECS-40-S-4X

Commit message: Update motherboard_Embedded.sch
Parts:
- added R1, R9: 10K, SparkFun-Resistors:RESISTOR0603
- added S1: (no value), SparkFun-Switches:MOMENTARY-SWITCH-SPST-2-SMD-4.6X2.8MM
Connections:
- net VDD renamed 3.3V
- removed net TEMP_SENS: U$1.RC3/SCK/SCL
- new net N$5: R1.1, S1.3, S1.4, U$1.~MCLR/VPP
- new net TEMP_DQ: J3.2, R9.2, U$1.RC3/SCK/SCL
- new net VCC: J3.3, R1.2, R9.1, U$1.VDD
- net GND: now also J3.1, S1.1, S1.2, U$1.VSS, U$1.VSS_2
Other:
- moved on the sheet: J3
Changed lines of the file:
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@@
 <setting verticaltext="up"/>
 </settings>
-<grid distance="0.1" unitdist="inch" unit="inch" style="lines" multiple="1" display="no" altdistance="0.01" altunitdist="inch" altunit="inch"/>
+<grid distance="0.1" unitdist="inch" unit="inch" style="lines" multiple="1" display="yes" altdistance="0.01" altunitdist="inch" altunit="inch"/>
 <layers>
 <layer number="1" name="Top" color="4" fill="1" visible="no" active="no"/>
@@
 <part name="J2" library="SparkFun-Connectors" deviceset="CONN_06" device="POLAR"/>
 <part name="J3" library="SparkFun-Connectors" deviceset="CONN_03" device="POLAR"/>
+<part name="S1" library="SparkFun-Switches" deviceset="MOMENTARY-SWITCH-SPST-2" device="-SMD-4.6X2.8MM"/>
+<part name="GND6" library="SparkFun-PowerSymbols" deviceset="GND" device=""/>
+<part name="R1" library="SparkFun-Resistors" deviceset="RESISTOR" device="0603" value=" 10K"/>
+<part name="3.3V" library="supply1" library_urn="urn:adsk.eagle:library:371" deviceset="VCC" device="" value="3.3V"/>
+<part name="GND7" library="SparkFun-PowerSymbols" deviceset="GND" device=""/>
+<part name="R9" library="SparkFun-Resistors" deviceset="RESISTOR" device="0603" value=" 10K"/>
+<part name="3.3V1" library="supply1" library_urn="urn:adsk.eagle:library:371" deviceset="VCC" device="" value="3.3V"/>
+<part name="GND8" library="SparkFun-PowerSymbols" deviceset="GND" device=""/>
 </parts>
 <sheets>
@@
 <attribute name="NAME" x="99.06" y="150.368" size="1.778" layer="95" font="vector"/>
 </instance>
-<instance part="J3" gate="J$1" x="58.42" y="167.64" smashed="yes">
-<attribute name="VALUE" x="55.88" y="160.274" size="1.778" layer="96" font="vector"/>
-<attribute name="NAME" x="55.88" y="173.228" size="1.778" layer="95" font="vector"/>
+<instance part="J3" gate="J$1" x="53.34" y="160.02" smashed="yes">
+<attribute name="VALUE" x="50.8" y="152.654" size="1.778" layer="96" font="vector"/>
+<attribute name="NAME" x="50.8" y="165.608" size="1.778" layer="95" font="vector"/>
+</instance>
+<instance part="S1" gate="G$1" x="2.54" y="99.06" smashed="yes">
+<attribute name="NAME" x="2.54" y="103.886" size="1.778" layer="95" font="vector" align="bottom-center"/>
+<attribute name="VALUE" x="2.54" y="96.266" size="1.778" layer="96" font="vector" align="top-center"/>
+</instance>
+<instance part="GND6" gate="1" x="-12.7" y="88.9" smashed="yes">
+<attribute name="VALUE" x="-12.7" y="88.646" size="1.778" layer="96" align="top-center"/>
+</instance>
+<instance part="R1" gate="G$1" x="15.24" y="104.14" smashed="yes" rot="R90">
+<attribute name="NAME" x="13.716" y="104.14" size="1.778" layer="95" font="vector" rot="R90" align="bottom-center"/>
+<attribute name="VALUE" x="16.764" y="104.14" size="1.778" layer="96" font="vector" rot="R90" align="top-center"/>
+</instance>
+<instance part="3.3V" gate="VCC" x="15.24" y="119.38" smashed="yes">
+<attribute name="VALUE" x="12.7" y="116.84" size="1.778" layer="96" rot="R90"/>
+</instance>
+<instance part="GND7" gate="1" x="71.12" y="147.32" smashed="yes">
+<attribute name="VALUE" x="71.12" y="147.066" size="1.778" layer="96" align="top-center"/>
+</instance>
+<instance part="R9" gate="G$1" x="76.2" y="162.56" smashed="yes">
+<attribute name="NAME" x="76.2" y="164.084" size="1.778" layer="95" font="vector" align="bottom-center"/>
+<attribute name="VALUE" x="76.2" y="161.036" size="1.778" layer="96" font="vector" align="top-center"/>
+</instance>
+<instance part="3.3V1" gate="VCC" x="66.04" y="172.72" smashed="yes">
+<attribute name="VALUE" x="63.5" y="170.18" size="1.778" layer="96" rot="R90"/>
+</instance>
+<instance part="GND8" gate="1" x="22.86" y="38.1" smashed="yes">
+<attribute name="VALUE" x="22.86" y="37.846" size="1.778" layer="96" align="top-center"/>
 </instance>
 </instances>
@@
 <label x="114.3" y="162.56" size="1.778" layer="95"/>
 </segment>
+<segment>
+<pinref part="S1" gate="G$1" pin="1"/>
+<wire x1="-2.54" y1="99.06" x2="-5.08" y2="99.06" width="0.1524" layer="91"/>
+<pinref part="S1" gate="G$1" pin="2"/>
+<wire x1="-5.08" y1="99.06" x2="-5.08" y2="96.52" width="0.1524" layer="91"/>
+<wire x1="-5.08" y1="96.52" x2="-2.54" y2="96.52" width="0.1524" layer="91"/>
+<wire x1="-5.08" y1="99.06" x2="-12.7" y2="99.06" width="0.1524" layer="91"/>
+<junction x="-5.08" y="99.06"/>
+<wire x1="-12.7" y1="99.06" x2="-12.7" y2="91.44" width="0.1524" layer="91"/>
+<pinref part="GND6" gate="1" pin="GND"/>
+</segment>
+<segment>
+<pinref part="J3" gate="J$1" pin="1"/>
+<wire x1="60.96" y1="157.48" x2="71.12" y2="157.48" width="0.1524" layer="91"/>
+<pinref part="GND7" gate="1" pin="GND"/>
+<wire x1="71.12" y1="157.48" x2="71.12" y2="149.86" width="0.1524" layer="91"/>
+</segment>
+<segment>
+<pinref part="U$1" gate="A" pin="VSS_2"/>
+<wire x1="33.02" y1="50.8" x2="22.86" y2="50.8" width="0.1524" layer="91"/>
+<pinref part="U$1" gate="A" pin="VSS"/>
+<wire x1="22.86" y1="50.8" x2="22.86" y2="48.26" width="0.1524" layer="91"/>
+<wire x1="22.86" y1="48.26" x2="33.02" y2="48.26" width="0.1524" layer="91"/>
+<wire x1="22.86" y1="48.26" x2="22.86" y2="40.64" width="0.1524" layer="91"/>
+<junction x="22.86" y="48.26"/>
+<pinref part="GND8" gate="1" pin="GND"/>
+</segment>
 </net>
 <net name="SOLENOID_ON/OFF" class="0">
@@
 <wire x1="-91.44" y1="152.4" x2="-81.28" y2="152.4" width="0.1524" layer="91"/>
 <label x="-104.14" y="152.4" size="1.778" layer="95"/>
-</segment>
-</net>
-<net name="TEMP_SENS" class="0">
-<segment>
-<pinref part="U$1" gate="A" pin="RC3/SCK/SCL"/>
-<wire x1="119.38" y1="91.44" x2="129.54" y2="91.44" width="0.1524" layer="91"/>
-<label x="124.46" y="91.44" size="1.778" layer="95"/>
 </segment>
 </net>
@@
 </segment>
 </net>
-<net name="VDD" class="0">
+<net name="3.3V" class="0">
 <segment>
 <pinref part="J1" gate="G$1" pin="2"/>
@@
 </segment>
 </net>
+<net name="N$5" class="0">
+<segment>
+<pinref part="S1" gate="G$1" pin="3"/>
+<wire x1="7.62" y1="99.06" x2="10.16" y2="99.06" width="0.1524" layer="91"/>
+<pinref part="S1" gate="G$1" pin="4"/>
+<wire x1="10.16" y1="99.06" x2="10.16" y2="96.52" width="0.1524" layer="91"/>
+<wire x1="10.16" y1="96.52" x2="7.62" y2="96.52" width="0.1524" layer="91"/>
+<pinref part="U$1" gate="A" pin="~MCLR/VPP"/>
+<wire x1="10.16" y1="99.06" x2="15.24" y2="99.06" width="0.1524" layer="91"/>
+<junction x="10.16" y="99.06"/>
+<pinref part="R1" gate="G$1" pin="1"/>
+<wire x1="15.24" y1="99.06" x2="33.02" y2="99.06" width="0.1524" layer="91"/>
+<junction x="15.24" y="99.06"/>
+</segment>
+</net>
+<net name="VCC" class="0">
+<segment>
+<pinref part="U$1" gate="A" pin="VDD"/>
+<wire x1="33.02" y1="104.14" x2="25.4" y2="104.14" width="0.1524" layer="91"/>
+<wire x1="25.4" y1="104.14" x2="25.4" y2="109.22" width="0.1524" layer="91"/>
+<pinref part="R1" gate="G$1" pin="2"/>
+<wire x1="25.4" y1="109.22" x2="15.24" y2="109.22" width="0.1524" layer="91"/>
+<wire x1="15.24" y1="109.22" x2="15.24" y2="116.84" width="0.1524" layer="91"/>
+<junction x="15.24" y="109.22"/>
+<pinref part="3.3V" gate="VCC" pin="VCC"/>
+</segment>
+<segment>
+<pinref part="J3" gate="J$1" pin="3"/>
+<wire x1="60.96" y1="162.56" x2="66.04" y2="162.56" width="0.1524" layer="91"/>
+<pinref part="R9" gate="G$1" pin="1"/>
+<wire x1="66.04" y1="162.56" x2="71.12" y2="162.56" width="0.1524" layer="91"/>
+<wire x1="66.04" y1="162.56" x2="66.04" y2="170.18" width="0.1524" layer="91"/>
+<junction x="66.04" y="162.56"/>
+<pinref part="3.3V1" gate="VCC" pin="VCC"/>
+</segment>
+</net>
+<net name="TEMP_DQ" class="0">
+<segment>
+<pinref part="J3" gate="J$1" pin="2"/>
+<wire x1="60.96" y1="160.02" x2="83.82" y2="160.02" width="0.1524" layer="91"/>
+<wire x1="83.82" y1="160.02" x2="83.82" y2="162.56" width="0.1524" layer="91"/>
+<pinref part="R9" gate="G$1" pin="2"/>
+<wire x1="83.82" y1="162.56" x2="81.28" y2="162.56" width="0.1524" layer="91"/>
+<wire x1="83.82" y1="160.02" x2="93.98" y2="160.02" width="0.1524" layer="91"/>
+<junction x="83.82" y="160.02"/>
+<label x="83.82" y="160.02" size="1.778" layer="95"/>
+</segment>
+<segment>
+<pinref part="U$1" gate="A" pin="RC3/SCK/SCL"/>
+<wire x1="119.38" y1="91.44" x2="127" y2="91.44" width="0.1524" layer="91"/>
+<label x="124.46" y="91.44" size="1.778" layer="95"/>
+<wire x1="127" y1="91.44" x2="129.54" y2="91.44" width="0.1524" layer="91"/>
+<wire x1="129.54" y1="91.44" x2="132.08" y2="91.44" width="0.1524" layer="91"/>
+</segment>
+</net>

Commit message: Update motherboard_Embedded.sch
Parts:
- removed J1: (no value), SparkFun-Connectors:CONN_06POLAR
- added J4: (no value), SparkFun-Connectors:CONN_06SILK_FEMALE_PTH
- J2: device SparkFun-Connectors:CONN_06POLAR -> SparkFun-Connectors:CONN_05JST-VERT
Connections:
- removed net 12V: Q1G1.S, R4.1
- removed net N$11: J2.6
- removed net N$12: J2.5
- removed net N$13: J2.4
- removed net N$14: J2.3
- removed net N$15: J2.2
- removed net N$16: J2.1
- new net BLUETOOTH_ON/OFF: J2.1, U$1.RB0/INT
- net 3.3V: now also J2.4, J4.2; no longer J1.2
- net GND: now also J2.5, J4.3; no longer J1.3
- net LVP: now also J4.6; no longer J1.6
- net MCLR: now also J4.1; no longer J1.1
- net PGC: now also J4.5; no longer J1.5
- net PGD: now also J4.4; no longer J1.4
- net PWM: no longer R6.2
- net RX: now also J2.3
- net SOLENOID_ON/OFF: no longer R2.1
- net TX: now also J2.2
- net VCC: now also Q1G1.S, R4.1
Other:
- note removed: "Nicholas Champ Spoutz"
- moved on the sheet: BLED1, BLED2, BLED3, C1, C2, C4, D1, D2, J3, Q1G1, Q2, R1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

Commit message: Update motherboard_Embedded.sch
Parts:
- added J5: (no value), SparkFun-Connectors:CONN_02
Connections:
- new net N$2: R6.2
- new net N$7: R2.1
- net GND: now also J5.1
- net VCC: now also J5.2
Other:
- note added: "EXTERNAL CLOCK"
- note added: "HEADERS"
- note added: "LED ARRAYS"
- note added: "MICROCONTROLLER"
- note added: "SOLENOID DETECTOR"
- note added: "SOLENOID DRIVER"
- note added: "TEST POWER SUPPLY"
- moved on the sheet: BLED1, BLED2, BLED3, C1, C2, C4, D1, D2, J2, J3, Q1G1, Q2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
