File: eagle/projects/smartBobber Mother Board/motherBoard/motherboard_Embedded.sch (EAGLE design)
At the start: 30 parts, among them Q1 2A/20V/150mΩ, Q2 MMBT3904, Y1 ECS-40-S-4X

Commit message: Update motherboard_Embedded.sch
Other:
- note added: "Nicholas Champ Spoutz"
Changed lines of the file:
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@@
 <text x="182.88" y="170.18" size="2.54" layer="94">LED ARRAYS</text>
 <text x="91.44" y="106.68" size="2.54" layer="94">MICROCONTROLLER</text>
+<text x="215.9" y="10.16" size="2.54" layer="94">Nicholas Champ Spoutz</text>
 </plain>
 <instances>
@@
 </instance>
 <instance part="FRAME2" gate="G$1" x="0" y="0" smashed="yes">
-<attribute name="DRAWING_NAME" x="217.17" y="20.32" size="2.54" layer="94"/>
-<attribute name="LAST_DATE_TIME" x="217.17" y="15.24" size="2.286" layer="94"/>
+<attribute name="DRAWING_NAME" x="215.9" y="20.32" size="2.54" layer="94"/>
+<attribute name="LAST_DATE_TIME" x="215.9" y="15.24" size="2.286" layer="94"/>
 <attribute name="SHEET" x="230.505" y="5.08" size="2.54" layer="94"/>
 </instance>

Commit message: Update motherboard_Embedded.sch
Parts:
- added U$2: PTS645, PTS645button:PTS645
Changed lines of the file:
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@@
 <part name="GND9" library="supply1" library_urn="urn:adsk.eagle:library:371" deviceset="GND" device=""/>
 <part name="3.3V2" library="supply1" library_urn="urn:adsk.eagle:library:371" deviceset="VCC" device="" value="3.3V"/>
+<part name="U$2" library="PTS645button" deviceset="PTS645" device=""/>
 </parts>
 <sheets>
@@
 <attribute name="VALUE" x="116.84" y="154.94" size="1.778" layer="96" rot="R90"/>
 </instance>
+<instance part="U$2" gate="G$1" x="106.68" y="99.06" smashed="yes"/>
 </instances>
 <busses>

Commit message: Update motherboard_Embedded.sch
Parts:
- removed S1: (no value), SparkFun-Switches:MOMENTARY-SWITCH-SPST-2-SMD-4.6X2.8MM
- removed U$2: PTS645, PTS645button:PTS645
- added R10: 10k, SparkFun-Resistors:RESISTOR0603
- added S2: Button, SparkFun-Switches:MOMENTARY-SWITCH-SPST-SMD-5.2MM
Connections:
- removed net N$2: R6.2
- removed net N$7: R2.1
- net BLUETOOTH_ON/OFF: now also R10.2
- net GND: now also R10.1, S2.1; no longer S1.1, S1.2
- net N$5: now also S2.2; no longer S1.3, S1.4
- net PWM: now also R6.2
- net SOLENOID_ON/OFF: now also R2.1
Changed lines of the file:
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@@
 <setting verticaltext="up"/>
 </settings>
-<grid distance="0.1" unitdist="inch" unit="inch" style="lines" multiple="1" display="no" altdistance="0.01" altunitdist="inch" altunit="inch"/>
+<grid distance="0.1" unitdist="inch" unit="inch" style="lines" multiple="1" display="yes" altdistance="0.01" altunitdist="inch" altunit="inch"/>
 <layers>
 <layer number="1" name="Top" color="4" fill="1" visible="no" active="no"/>
@@
 <part name="R8" library="SparkFun-Resistors" deviceset="RESISTOR" device="0603" value=" 1"/>
 <part name="J3" library="SparkFun-Connectors" deviceset="CONN_03" device="POLAR"/>
-<part name="S1" library="SparkFun-Switches" deviceset="MOMENTARY-SWITCH-SPST-2" device="-SMD-4.6X2.8MM"/>
 <part name="GND6" library="SparkFun-PowerSymbols" deviceset="GND" device=""/>
 <part name="R1" library="SparkFun-Resistors" deviceset="RESISTOR" device="0603" value=" 10K"/>
@@
 <part name="GND9" library="supply1" library_urn="urn:adsk.eagle:library:371" deviceset="GND" device=""/>
 <part name="3.3V2" library="supply1" library_urn="urn:adsk.eagle:library:371" deviceset="VCC" device="" value="3.3V"/>
-<part name="U$2" library="PTS645button" deviceset="PTS645" device=""/>
+<part name="R10" library="SparkFun-Resistors" deviceset="RESISTOR" device="0603" value=" 10k"/>
+<part name="GND10" library="SparkFun-PowerSymbols" deviceset="GND" device=""/>
+<part name="S2" library="SparkFun-Switches" deviceset="MOMENTARY-SWITCH-SPST" device="-SMD-5.2MM" value="Button"/>
 </parts>
 <sheets>
@@
 <attribute name="NAME" x="38.1" y="48.768" size="1.778" layer="95" font="vector"/>
 </instance>
-<instance part="S1" gate="G$1" x="119.38" y="86.36" smashed="yes">
-<attribute name="NAME" x="119.38" y="91.186" size="1.778" layer="95" font="vector" align="bottom-center"/>
-<attribute name="VALUE" x="119.38" y="83.566" size="1.778" layer="96" font="vector" align="top-center"/>
-</instance>
 <instance part="GND6" gate="1" x="104.14" y="76.2" smashed="yes">
 <attribute name="VALUE" x="104.14" y="75.946" size="1.778" layer="96" align="top-center"/>
@@
 </instance>
 <instance part="3.3V" gate="VCC" x="132.08" y="106.68" smashed="yes">
-<attribute name="VALUE" x="129.54" y="104.14" size="1.778" layer="96" rot="R90"/>
+<attribute name="VALUE" x="139.7" y="106.68" size="1.778" layer="96" rot="R180"/>
 </instance>
 <instance part="GND7" gate="1" x="58.42" y="30.48" smashed="yes">
@@
 <attribute name="VALUE" x="116.84" y="154.94" size="1.778" layer="96" rot="R90"/>
 </instance>
-<instance part="U$2" gate="G$1" x="106.68" y="99.06" smashed="yes"/>
+<instance part="R10" gate="G$1" x="134.62" y="60.96" smashed="yes">
+<attribute name="NAME" x="134.62" y="62.484" size="1.778" layer="95" font="vector" align="bottom-center"/>
+<attribute name="VALUE" x="134.62" y="59.436" size="1.778" layer="96" font="vector" align="top-center"/>
+</instance>
+<instance part="GND10" gate="1" x="116.84" y="50.8" smashed="yes">
+<attribute name="VALUE" x="116.84" y="50.546" size="1.778" layer="96" align="top-center"/>
+</instance>
+<instance part="S2" gate="G$1" x="119.38" y="86.36" smashed="yes">
+<attribute name="NAME" x="119.38" y="87.884" size="1.778" layer="95" font="vector" align="bottom-center"/>
+<attribute name="VALUE" x="119.38" y="85.852" size="1.778" layer="96" font="vector" align="top-center"/>
+</instance>
 </instances>
 <busses>
@@
 <wire x1="236.22" y1="81.28" x2="246.38" y2="81.28" width="0.1524" layer="91"/>
 <label x="241.3" y="81.28" size="1.778" layer="95"/>
+</segment>
+<segment>
+<pinref part="R6" gate="G$1" pin="2"/>
+<wire x1="17.78" y1="96.52" x2="7.62" y2="96.52" width="0.1524" layer="91"/>
+<label x="7.62" y="96.52" size="1.778" layer="95"/>
 </segment>
 </net>
@@
 </segment>
 <segment>
-<pinref part="S1" gate="G$1" pin="1"/>
-<wire x1="114.3" y1="86.36" x2="111.76" y2="86.36" width="0.1524" layer="91"/>
-<pinref part="S1" gate="G$1" pin="2"/>
-<wire x1="111.76" y1="86.36" x2="111.76" y2="83.82" width="0.1524" layer="91"/>
-<wire x1="111.76" y1="83.82" x2="114.3" y2="83.82" width="0.1524" layer="91"/>
-<wire x1="111.76" y1="86.36" x2="104.14" y2="86.36" width="0.1524" layer="91"/>
-<junction x="111.76" y="86.36"/>
+<wire x1="114.3" y1="86.36" x2="104.14" y2="86.36" width="0.1524" layer="91"/>
 <wire x1="104.14" y1="86.36" x2="104.14" y2="78.74" width="0.1524" layer="91"/>
 <pinref part="GND6" gate="1" pin="GND"/>
+<pinref part="S2" gate="G$1" pin="1"/>
 </segment>
 <segment>
@@
 <pinref part="GND9" gate="1" pin="GND"/>
 </segment>
+<segment>
+<pinref part="R10" gate="G$1" pin="1"/>
+<wire x1="129.54" y1="60.96" x2="116.84" y2="60.96" width="0.1524" layer="91"/>
+<wire x1="116.84" y1="60.96" x2="116.84" y2="53.34" width="0.1524" layer="91"/>
+<pinref part="GND10" gate="1" pin="GND"/>
+</segment>
 </net>
 <net name="SOLENOID_ON/OFF" class="0">
@@
 <wire x1="149.86" y1="48.26" x2="139.7" y2="48.26" width="0.1524" layer="91"/>
 <label x="124.46" y="48.26" size="1.778" layer="95"/>
+</segment>
+<segment>
+<pinref part="R2" gate="G$1" pin="1"/>
+<wire x1="15.24" y1="137.16" x2="7.62" y2="137.16" width="0.1524" layer="91"/>
+<label x="7.62" y="127" size="1.778" layer="95" rot="R90"/>
 </segment>
 </net>
@@
 <net name="N$5" class="0">
 <segment>
-<pinref part="S1" gate="G$1" pin="3"/>
-<wire x1="124.46" y1="86.36" x2="127" y2="86.36" width="0.1524" layer="91"/>
-<pinref part="S1" gate="G$1" pin="4"/>
-<wire x1="127" y1="86.36" x2="127" y2="83.82" width="0.1524" layer="91"/>
-<wire x1="127" y1="83.82" x2="124.46" y2="83.82" width="0.1524" layer="91"/>
 <pinref part="U$1" gate="A" pin="~MCLR/VPP"/>
-<wire x1="127" y1="86.36" x2="132.08" y2="86.36" width="0.1524" layer="91"/>
-<junction x="127" y="86.36"/>
+<wire x1="124.46" y1="86.36" x2="132.08" y2="86.36" width="0.1524" layer="91"/>
 <pinref part="R1" gate="G$1" pin="1"/>
 <wire x1="132.08" y1="86.36" x2="149.86" y2="86.36" width="0.1524" layer="91"/>
 <junction x="132.08" y="86.36"/>
+<pinref part="S2" gate="G$1" pin="2"/>
 </segment>
 </net>
@@
 <segment>
 <pinref part="U$1" gate="A" pin="RB0/INT"/>
-<wire x1="149.86" y1="60.96" x2="139.7" y2="60.96" width="0.1524" layer="91"/>
-<label x="121.92" y="60.96" size="1.778" layer="95"/>
-</segment>
-</net>
-<net name="N$2" class="0">
-<segment>
-<pinref part="R6" gate="G$1" pin="2"/>
-<wire x1="17.78" y1="96.52" x2="7.62" y2="96.52" width="0.1524" layer="91"/>
-</segment>
-</net>
-<net name="N$7" class="0">
-<segment>
-<pinref part="R2" gate="G$1" pin="1"/>
-<wire x1="15.24" y1="137.16" x2="7.62" y2="137.16" width="0.1524" layer="91"/>
-</segment>
-</net>
+<wire x1="149.86" y1="60.96" x2="144.78" y2="60.96" width="0.1524" layer="91"/>
+<label x="144.78" y="71.12" size="1.778" layer="95" rot="R180"/>
+<pinref part="R10" gate="G$1" pin="2"/>
+<wire x1="144.78" y1="60.96" x2="139.7" y2="60.96" width="0.1524" layer="91"/>
+<wire x1="144.78" y1="60.96" x2="144.78" y2="71.12" width="0.1524" layer="91"/>
+<junction x="144.78" y="60.96"/>
+</segment>
+</net>

Commit message: Board update
Parts:
- added R11: 100k, SparkFun-Resistors:RESISTOR0603
Connections:
- net ADC: now also R11.1, R11.2
Changed lines of the file:
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@@
 <setting verticaltext="up"/>
 </settings>
-<grid distance="0.1" unitdist="inch" unit="inch" style="lines" multiple="1" display="yes" altdistance="0.01" altunitdist="inch" altunit="inch"/>
+<grid distance="0.1" unitdist="inch" unit="inch" style="lines" multiple="1" display="no" altdistance="0.01" altunitdist="inch" altunit="inch"/>
 <layers>
 <layer number="1" name="Top" color="4" fill="1" visible="no" active="no"/>
@@
 <part name="GND10" library="SparkFun-PowerSymbols" deviceset="GND" device=""/>
 <part name="S2" library="SparkFun-Switches" deviceset="MOMENTARY-SWITCH-SPST" device="-SMD-5.2MM" value="Button"/>
+<part name="R11" library="SparkFun-Resistors" deviceset="RESISTOR" device="0603" value=" 100k"/>
 </parts>
 <sheets>
@@
 <attribute name="VALUE" x="119.38" y="85.852" size="1.778" layer="96" font="vector" align="top-center"/>
 </instance>
+<instance part="R11" gate="G$1" x="78.74" y="96.52" smashed="yes">
+<attribute name="NAME" x="78.74" y="98.044" size="1.778" layer="95" font="vector" align="bottom-center"/>
+<attribute name="VALUE" x="78.74" y="94.996" size="1.778" layer="96" font="vector" align="top-center"/>
+</instance>
 </instances>
 <busses>
@@
 <pinref part="R5" gate="G$1" pin="2"/>
 <wire x1="58.42" y1="96.52" x2="71.12" y2="96.52" width="0.1524" layer="91"/>
-<wire x1="71.12" y1="96.52" x2="86.36" y2="96.52" width="0.1524" layer="91"/>
 <wire x1="58.42" y1="96.52" x2="58.42" y2="88.9" width="0.1524" layer="91"/>
 <junction x="58.42" y="96.52"/>
 <pinref part="C4" gate="G$1" pin="1"/>
 <wire x1="71.12" y1="96.52" x2="71.12" y2="88.9" width="0.1524" layer="91"/>
+<pinref part="R11" gate="G$1" pin="1"/>
+<wire x1="71.12" y1="96.52" x2="73.66" y2="96.52" width="0.1524" layer="91"/>
 <junction x="71.12" y="96.52"/>
-<label x="81.28" y="96.52" size="1.778" layer="95"/>
 </segment>
 <segment>
@@
 <label x="139.7" y="78.74" size="1.778" layer="95"/>
 </segment>
+<segment>
+<pinref part="R11" gate="G$1" pin="2"/>
+<wire x1="83.82" y1="96.52" x2="83.82" y2="104.14" width="0.1524" layer="91"/>
+<label x="81.28" y="104.14" size="1.778" layer="95"/>
+</segment>
 </net>

Commit message: Update motherboard_Embedded.sch
Parts:
- added C3, C5: 1.0uF, SparkFun-Capacitors:1.0UF-0603-16V-10%-X7R
Changed lines of the file:
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@@
 <part name="S2" library="SparkFun-Switches" deviceset="MOMENTARY-SWITCH-SPST" device="-SMD-5.2MM" value="Button"/>
 <part name="R11" library="SparkFun-Resistors" deviceset="RESISTOR" device="0603" value=" 100k"/>
+<part name="C3" library="SparkFun-Capacitors" deviceset="1.0UF" device="-0603-16V-10%-X7R" value="1.0uF"/>
+<part name="C5" library="SparkFun-Capacitors" deviceset="1.0UF" device="-0603-16V-10%-X7R" value="1.0uF"/>
 </parts>
 <sheets>
@@
 <attribute name="VALUE" x="78.74" y="94.996" size="1.778" layer="96" font="vector" align="top-center"/>
 </instance>
+<instance part="C3" gate="G$1" x="93.98" y="43.18" smashed="yes">
+<attribute name="NAME" x="95.504" y="46.101" size="1.778" layer="95" font="vector"/>
+<attribute name="VALUE" x="95.504" y="41.021" size="1.778" layer="96" font="vector"/>
+</instance>
+<instance part="C5" gate="G$1" x="101.6" y="43.18" smashed="yes">
+<attribute name="NAME" x="103.124" y="46.101" size="1.778" layer="95" font="vector"/>
+<attribute name="VALUE" x="103.124" y="41.021" size="1.778" layer="96" font="vector"/>
+</instance>
 </instances>

Commit message: Update motherboard_Embedded.sch
Parts:
- removed C3, C5: 1.0uF, SparkFun-Capacitors:1.0UF-0603-16V-10%-X7R
- added C6: 0.1uF, SparkFun-Capacitors:0.1UF-0603-25V-5%
Connections:
- net 3.3V: now also C6.1, R1.2, U$1.VDD
- net GND: now also C6.2
- net VCC: no longer R1.2, U$1.VDD
Changed lines of the file:
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@@
 <part name="S2" library="SparkFun-Switches" deviceset="MOMENTARY-SWITCH-SPST" device="-SMD-5.2MM" value="Button"/>
 <part name="R11" library="SparkFun-Resistors" deviceset="RESISTOR" device="0603" value=" 100k"/>
-<part name="C3" library="SparkFun-Capacitors" deviceset="1.0UF" device="-0603-16V-10%-X7R" value="1.0uF"/>
-<part name="C5" library="SparkFun-Capacitors" deviceset="1.0UF" device="-0603-16V-10%-X7R" value="1.0uF"/>
+<part name="C6" library="SparkFun-Capacitors" deviceset="0.1UF" device="-0603-25V-5%" value="0.1uF"/>
+<part name="GND11" library="SparkFun-PowerSymbols" deviceset="GND" device=""/>
 </parts>
 <sheets>
@@
 <attribute name="VALUE" x="133.604" y="91.44" size="1.778" layer="96" font="vector" rot="R90" align="top-center"/>
 </instance>
-<instance part="3.3V" gate="VCC" x="132.08" y="106.68" smashed="yes">
-<attribute name="VALUE" x="139.7" y="106.68" size="1.778" layer="96" rot="R180"/>
-</instance>
+<instance part="3.3V" gate="VCC" x="132.08" y="106.68" smashed="yes"/>
 <instance part="GND7" gate="1" x="58.42" y="30.48" smashed="yes">
 <attribute name="VALUE" x="58.42" y="30.226" size="1.778" layer="96" align="top-center"/>
@@
 <attribute name="VALUE" x="78.74" y="94.996" size="1.778" layer="96" font="vector" align="top-center"/>
 </instance>
-<instance part="C3" gate="G$1" x="93.98" y="43.18" smashed="yes">
-<attribute name="NAME" x="95.504" y="46.101" size="1.778" layer="95" font="vector"/>
-<attribute name="VALUE" x="95.504" y="41.021" size="1.778" layer="96" font="vector"/>
-</instance>
-<instance part="C5" gate="G$1" x="101.6" y="43.18" smashed="yes">
-<attribute name="NAME" x="103.124" y="46.101" size="1.778" layer="95" font="vector"/>
-<attribute name="VALUE" x="103.124" y="41.021" size="1.778" layer="96" font="vector"/>
+<instance part="C6" gate="G$1" x="99.06" y="43.18" smashed="yes">
+<attribute name="NAME" x="100.584" y="46.101" size="1.778" layer="95" font="vector"/>
+<attribute name="VALUE" x="100.584" y="41.021" size="1.778" layer="96" font="vector"/>
+</instance>
+<instance part="GND11" gate="1" x="99.06" y="30.48" smashed="yes">
+<attribute name="VALUE" x="99.06" y="30.226" size="1.778" layer="96" align="top-center"/>
 </instance>
 </instances>
@@
 <pinref part="GND10" gate="1" pin="GND"/>
 </segment>
+<segment>
+<pinref part="C6" gate="G$1" pin="2"/>
+<wire x1="99.06" y1="40.64" x2="99.06" y2="33.02" width="0.1524" layer="91"/>
+<pinref part="GND11" gate="1" pin="GND"/>
+</segment>
 </net>
 <net name="SOLENOID_ON/OFF" class="0">
@@
 <label x="25.4" y="15.24" size="1.778" layer="95"/>
 </segment>
-</net>
-<net name="PGD" class="0">
-<segment>
-<pinref part="J4" gate="G$1" pin="4"/>
-<wire x1="20.32" y1="20.32" x2="30.48" y2="20.32" width="0.1524" layer="91"/>
-<label x="25.4" y="20.32" size="1.778" layer="95"/>
-</segment>
-</net>
-<net name="PGC" class="0">
-<segment>
-<pinref part="J4" gate="G$1" pin="5"/>
-<wire x1="20.32" y1="22.86" x2="30.48" y2="22.86" width="0.1524" layer="91"/>
-<label x="25.4" y="22.86" size="1.778" layer="95"/>
-</segment>
-</net>
-<net name="LVP" class="0">
-<segment>
-<pinref part="J4" gate="G$1" pin="6"/>
-<wire x1="20.32" y1="25.4" x2="30.48" y2="25.4" width="0.1524" layer="91"/>
-<label x="25.4" y="25.4" size="1.778" layer="95"/>
-</segment>
-</net>
-<net name="N$5" class="0">
-<segment>
-<pinref part="U$1" gate="A" pin="~MCLR/VPP"/>
-<wire x1="124.46" y1="86.36" x2="132.08" y2="86.36" width="0.1524" layer="91"/>
-<pinref part="R1" gate="G$1" pin="1"/>
-<wire x1="132.08" y1="86.36" x2="149.86" y2="86.36" width="0.1524" layer="91"/>
-<junction x="132.08" y="86.36"/>
-<pinref part="S2" gate="G$1" pin="2"/>
-</segment>
-</net>
-<net name="VCC" class="0">
 <segment>
 <pinref part="U$1" gate="A" pin="VDD"/>
@@
 <junction x="132.08" y="96.52"/>
 <pinref part="3.3V" gate="VCC" pin="VCC"/>
-</segment>
+<label x="134.62" y="101.6" size="1.778" layer="95"/>
+</segment>
+<segment>
+<pinref part="C6" gate="G$1" pin="1"/>
+<wire x1="99.06" y1="48.26" x2="99.06" y2="55.88" width="0.1524" layer="91"/>
+<label x="99.06" y="55.88" size="1.778" layer="95"/>
+</segment>
+</net>
+<net name="PGD" class="0">
+<segment>
+<pinref part="J4" gate="G$1" pin="4"/>
+<wire x1="20.32" y1="20.32" x2="30.48" y2="20.32" width="0.1524" layer="91"/>
+<label x="25.4" y="20.32" size="1.778" layer="95"/>
+</segment>
+</net>
+<net name="PGC" class="0">
+<segment>
+<pinref part="J4" gate="G$1" pin="5"/>
+<wire x1="20.32" y1="22.86" x2="30.48" y2="22.86" width="0.1524" layer="91"/>
+<label x="25.4" y="22.86" size="1.778" layer="95"/>
+</segment>
+</net>
+<net name="LVP" class="0">
+<segment>
+<pinref part="J4" gate="G$1" pin="6"/>
+<wire x1="20.32" y1="25.4" x2="30.48" y2="25.4" width="0.1524" layer="91"/>
+<label x="25.4" y="25.4" size="1.778" layer="95"/>
+</segment>
+</net>
+<net name="N$5" class="0">
+<segment>
+<pinref part="U$1" gate="A" pin="~MCLR/VPP"/>
+<wire x1="124.46" y1="86.36" x2="132.08" y2="86.36" width="0.1524" layer="91"/>
+<pinref part="R1" gate="G$1" pin="1"/>
+<wire x1="132.08" y1="86.36" x2="149.86" y2="86.36" width="0.1524" layer="91"/>
+<junction x="132.08" y="86.36"/>
+<pinref part="S2" gate="G$1" pin="2"/>
+</segment>
+</net>
+<net name="VCC" class="0">
 <segment>
 <pinref part="J3" gate="J$1" pin="3"/>

Commit message: Update motherboard_Embedded.sch
Parts:
- removed J2: (no value), SparkFun-Connectors:CONN_05JST-VERT
- removed J3: (no value), SparkFun-Connectors:CONN_03POLAR
- removed SOLENOID: (no value), SparkFun-Connectors:CONN_02
- added J1: 640456-2, 640456-2:640456-2
- added J6: 640456-3, 640456-3:640456-3
- added J7: 640456-5, 640456-5:640456-5
Connections:
- net 3.3V: now also J7.2; no longer J2.4
- net BLUETOOTH_ON/OFF: now also J7.5; no longer J2.1
- net DRIVER: now also J1.P1; no longer SOLENOID.1
- net GND: now also J1.P2, J6.1, J7.1; no longer J2.5, J3.1, SOLENOID.2
- net RX: now also J7.3; no longer J2.3
- net TEMP_DQ: now also J6.2; no longer J3.2
- net TX: now also J7.4; no longer J2.2
- net VCC: now also J6.3; no longer J3.3
Other:
- moved on the sheet: J4
