File: eagle/projects/smartBobber Mother Board/motherBoard/motherboard_Embedded.sch (EAGLE design)
At the start: 33 parts, among them J1 640456-2, J6 640456-3, J7 640456-5, Q1 2A/20V/150mΩ, Q2 MMBT3904, Y1 ECS-40-S-4X

Commit message: Update
Parts:
- removed J5: (no value), SparkFun-Connectors:CONN_02
- added J2: 640456-2, 640456-2:640456-2
Connections:
- net GND: now also J2.P1; no longer J5.1
- net VCC: now also J2.P2; no longer J5.2
Changed lines of the file:
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@@
 <part name="FRAME2" library="frames" library_urn="urn:adsk.eagle:library:229" deviceset="A4L-LOC" device=""/>
 <part name="12V" library="SparkFun-PowerSymbols" deviceset="VCC" device="" value="12V"/>
-<part name="J5" library="SparkFun-Connectors" deviceset="CONN_02" device=""/>
 <part name="GND9" library="supply1" library_urn="urn:adsk.eagle:library:371" deviceset="GND" device=""/>
 <part name="3.3V2" library="supply1" library_urn="urn:adsk.eagle:library:371" deviceset="VCC" device="" value="3.3V"/>
@@
 <part name="J7" library="640456-5" deviceset="640456-5" device=""/>
 <part name="D1" library="1N4002" deviceset="1N4002" device=""/>
+<part name="J2" library="640456-2" deviceset="640456-2" device=""/>
 </parts>
 <sheets>
@@
 <attribute name="VALUE" x="73.66" y="165.354" size="1.778" layer="96" align="bottom-center"/>
 </instance>
-<instance part="J5" gate="G$1" x="104.14" y="144.78" smashed="yes">
-<attribute name="VALUE" x="101.6" y="139.954" size="1.778" layer="96" font="vector"/>
-<attribute name="NAME" x="101.6" y="150.368" size="1.778" layer="95" font="vector"/>
-</instance>
 <instance part="GND9" gate="1" x="119.38" y="134.62" smashed="yes">
 <attribute name="VALUE" x="116.84" y="132.08" size="1.778" layer="96"/>
@@
 <attribute name="NAME" x="43.40551875" y="99.16511875" size="1.78036875" layer="95"/>
 <attribute name="VALUE" x="43.150440625" y="92.016909375" size="1.78088125" layer="96"/>
+</instance>
+<instance part="J2" gate="G$1" x="106.68" y="144.78" smashed="yes" rot="R180">
+<attribute name="NAME" x="111.76463125" y="138.678440625" size="1.271159375" layer="95" rot="R180"/>
+<attribute name="VALUE" x="111.767859375" y="152.411790625" size="1.271959375" layer="96" rot="R180"/>
 </instance>
 </instances>
@@
 </segment>
 <segment>
-<pinref part="J5" gate="G$1" pin="1"/>
-<wire x1="111.76" y1="144.78" x2="119.38" y2="144.78" width="0.1524" layer="91"/>
-<wire x1="119.38" y1="144.78" x2="119.38" y2="137.16" width="0.1524" layer="91"/>
-<pinref part="GND9" gate="1" pin="GND"/>
-</segment>
-<segment>
 <pinref part="R10" gate="G$1" pin="1"/>
 <wire x1="129.54" y1="60.96" x2="116.84" y2="60.96" width="0.1524" layer="91"/>
@@
 <wire x1="99.06" y1="40.64" x2="99.06" y2="33.02" width="0.1524" layer="91"/>
 <pinref part="GND11" gate="1" pin="GND"/>
+</segment>
+<segment>
+<pinref part="J2" gate="G$1" pin="P1"/>
+<wire x1="114.3" y1="142.24" x2="119.38" y2="142.24" width="0.1524" layer="91"/>
+<pinref part="GND9" gate="1" pin="GND"/>
+<wire x1="119.38" y1="142.24" x2="119.38" y2="137.16" width="0.1524" layer="91"/>
 </segment>
 </net>
@@
 </segment>
 <segment>
-<pinref part="J5" gate="G$1" pin="2"/>
-<wire x1="111.76" y1="147.32" x2="119.38" y2="147.32" width="0.1524" layer="91"/>
+<pinref part="J2" gate="G$1" pin="P2"/>
+<wire x1="114.3" y1="147.32" x2="119.38" y2="147.32" width="0.1524" layer="91"/>
+<pinref part="3.3V2" gate="VCC" pin="VCC"/>
 <wire x1="119.38" y1="147.32" x2="119.38" y2="154.94" width="0.1524" layer="91"/>
-<pinref part="3.3V2" gate="VCC" pin="VCC"/>
-</segment>
-</net>
+</segment>
+</net>
