File: eagle/projects/smartBobber Mother Board/motherBoard/motherBoard_Power.sch (EAGLE design)
At the start: 20 parts, among them J4 10118193-0001LF, U1 MCP7384XX, U2 MT3608

Commit message: Update motherBoard_Power.sch
Parts:
- added U$1: CDRH104R, CDRH104R:CDRH104R
Changed lines of the file:
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@@
 <setting verticaltext="up"/>
 </settings>
-<grid distance="0.1" unitdist="inch" unit="inch" style="lines" multiple="1" display="no" altdistance="0.01" altunitdist="inch" altunit="inch"/>
+<grid distance="0.1" unitdist="inch" unit="inch" style="lines" multiple="1" display="yes" altdistance="0.01" altunitdist="inch" altunit="inch"/>
 <layers>
 <layer number="1" name="Top" color="4" fill="1" visible="no" active="no"/>
@@
 <part name="D5" library="SS34" deviceset="SS34" device=""/>
 <part name="J4" library="10118193-0001LF" deviceset="10118193-0001LF" device=""/>
+<part name="U$1" library="CDRH104R" deviceset="CDRH104R" device=""/>
 </parts>
 <sheets>
@@
 <attribute name="VALUE" x="-114.30193125" y="35.5503" size="1.778" layer="96"/>
 </instance>
+<instance part="U$1" gate="G$1" x="142.24" y="81.28" smashed="yes"/>
 </instances>
 <busses>

Commit message: Update motherBoard_Power.sch
Connections:
- new net N$1: U$1.1, U2.IN
- new net N$3: U$1.2, U2.SW
Changed lines of the file:
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@@
 <attribute name="VALUE" x="-114.30193125" y="35.5503" size="1.778" layer="96"/>
 </instance>
-<instance part="U$1" gate="G$1" x="142.24" y="81.28" smashed="yes"/>
+<instance part="U$1" gate="G$1" x="142.24" y="78.74" smashed="yes"/>
 </instances>
 <busses>
@@
 </segment>
 </net>
+<net name="N$1" class="0">
+<segment>
+<pinref part="U2" gate="G$1" pin="IN"/>
+<wire x1="129.54" y1="66.04" x2="127" y2="66.04" width="0.1524" layer="91"/>
+<pinref part="U$1" gate="G$1" pin="1"/>
+<wire x1="127" y1="66.04" x2="127" y2="78.74" width="0.1524" layer="91"/>
+<wire x1="127" y1="78.74" x2="134.62" y2="78.74" width="0.1524" layer="91"/>
+</segment>
+</net>
+<net name="N$3" class="0">
+<segment>
+<pinref part="U$1" gate="G$1" pin="2"/>
+<wire x1="149.86" y1="78.74" x2="157.48" y2="78.74" width="0.1524" layer="91"/>
+<wire x1="157.48" y1="78.74" x2="157.48" y2="68.58" width="0.1524" layer="91"/>
+<pinref part="U2" gate="G$1" pin="SW"/>
+<wire x1="157.48" y1="68.58" x2="154.94" y2="68.58" width="0.1524" layer="91"/>
+</segment>
+</net>

Commit message: Power - Hutson
Parts:
- added C1, C2: 22uF, SparkFun-Capacitors:22NF/22,000PF-0603-50V-10%
- added R1: (no value), rcl:R-TRIMM3296P
- added R2: 1k, SparkFun-Resistors:1KOHM-0603-1/10W-1%
Changed lines of the file:
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@@
 <part name="J4" library="10118193-0001LF" deviceset="10118193-0001LF" device=""/>
 <part name="U$1" library="CDRH104R" deviceset="CDRH104R" device=""/>
+<part name="R1" library="rcl" deviceset="R-TRIMM" device="3296P"/>
+<part name="R2" library="SparkFun-Resistors" deviceset="1KOHM" device="-0603-1/10W-1%" value="1k"/>
+<part name="C1" library="SparkFun-Capacitors" deviceset="22NF/22,000PF" device="-0603-50V-10%" value="22uF"/>
+<part name="C2" library="SparkFun-Capacitors" deviceset="22NF/22,000PF" device="-0603-50V-10%" value="22uF"/>
 </parts>
 <sheets>
@@
 </instance>
 <instance part="U$1" gate="G$1" x="142.24" y="78.74" smashed="yes"/>
+<instance part="R1" gate="G$1" x="170.18" y="73.66" smashed="yes" rot="R180">
+<attribute name="NAME" x="176.149" y="77.47" size="1.778" layer="95" rot="R270"/>
+<attribute name="VALUE" x="173.99" y="77.47" size="1.778" layer="96" rot="R270"/>
+</instance>
+<instance part="R2" gate="G$1" x="170.18" y="55.88" smashed="yes" rot="R90">
+<attribute name="NAME" x="168.656" y="55.88" size="1.778" layer="95" font="vector" rot="R90" align="bottom-center"/>
+<attribute name="VALUE" x="171.704" y="55.88" size="1.778" layer="96" font="vector" rot="R90" align="top-center"/>
+</instance>
+<instance part="C1" gate="G$1" x="134.62" y="93.98" smashed="yes" rot="R180">
+<attribute name="NAME" x="133.096" y="91.059" size="1.778" layer="95" font="vector" rot="R180"/>
+<attribute name="VALUE" x="133.096" y="96.139" size="1.778" layer="96" font="vector" rot="R180"/>
+</instance>
+<instance part="C2" gate="G$1" x="147.32" y="96.52" smashed="yes" rot="R180">
+<attribute name="NAME" x="145.796" y="93.599" size="1.778" layer="95" font="vector" rot="R180"/>
+<attribute name="VALUE" x="145.796" y="98.679" size="1.778" layer="96" font="vector" rot="R180"/>
+</instance>
 </instances>
 <busses>

Commit message: Power - Hutson
Connections:
- new net N$12: R1.A, R2.2, U2.FB
- new net N$14: C2.2, D4.C, R1.E
- net N$1: now also C1.2, S1.2, U2.EN
- net N$25: now also C1.1, C2.1, R2.1, U2.GND
- net N$3: now also D4.A
Other:
- moved on the sheet: C1, C2, R2
Changed lines of the file:
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@@
 <attribute name="VALUE" x="173.99" y="77.47" size="1.778" layer="96" rot="R270"/>
 </instance>
-<instance part="R2" gate="G$1" x="170.18" y="55.88" smashed="yes" rot="R90">
-<attribute name="NAME" x="168.656" y="55.88" size="1.778" layer="95" font="vector" rot="R90" align="bottom-center"/>
-<attribute name="VALUE" x="171.704" y="55.88" size="1.778" layer="96" font="vector" rot="R90" align="top-center"/>
-</instance>
-<instance part="C1" gate="G$1" x="134.62" y="93.98" smashed="yes" rot="R180">
-<attribute name="NAME" x="133.096" y="91.059" size="1.778" layer="95" font="vector" rot="R180"/>
-<attribute name="VALUE" x="133.096" y="96.139" size="1.778" layer="96" font="vector" rot="R180"/>
-</instance>
-<instance part="C2" gate="G$1" x="147.32" y="96.52" smashed="yes" rot="R180">
-<attribute name="NAME" x="145.796" y="93.599" size="1.778" layer="95" font="vector" rot="R180"/>
-<attribute name="VALUE" x="145.796" y="98.679" size="1.778" layer="96" font="vector" rot="R180"/>
+<instance part="R2" gate="G$1" x="170.18" y="53.34" smashed="yes" rot="R90">
+<attribute name="NAME" x="168.656" y="53.34" size="1.778" layer="95" font="vector" rot="R90" align="bottom-center"/>
+<attribute name="VALUE" x="171.704" y="53.34" size="1.778" layer="96" font="vector" rot="R90" align="top-center"/>
+</instance>
+<instance part="C1" gate="G$1" x="121.92" y="60.96" smashed="yes" rot="R180">
+<attribute name="NAME" x="120.396" y="58.039" size="1.778" layer="95" font="vector" rot="R180"/>
+<attribute name="VALUE" x="120.396" y="63.119" size="1.778" layer="96" font="vector" rot="R180"/>
+</instance>
+<instance part="C2" gate="G$1" x="185.42" y="66.04" smashed="yes" rot="R180">
+<attribute name="NAME" x="183.896" y="63.119" size="1.778" layer="95" font="vector" rot="R180"/>
+<attribute name="VALUE" x="183.896" y="68.199" size="1.778" layer="96" font="vector" rot="R180"/>
 </instance>
 </instances>
@@
 <pinref part="2.7K" gate="A" pin="R2"/>
 <wire x1="101.6" y1="35.56" x2="101.6" y2="48.26" width="0.1524" layer="91"/>
+<pinref part="C1" gate="G$1" pin="1"/>
+<wire x1="121.92" y1="55.88" x2="121.92" y2="35.56" width="0.1524" layer="91"/>
+<wire x1="121.92" y1="35.56" x2="101.6" y2="35.56" width="0.1524" layer="91"/>
+<junction x="101.6" y="35.56"/>
+<pinref part="U2" gate="G$1" pin="GND"/>
+<wire x1="154.94" y1="66.04" x2="157.48" y2="66.04" width="0.1524" layer="91"/>
+<wire x1="157.48" y1="66.04" x2="157.48" y2="35.56" width="0.1524" layer="91"/>
+<wire x1="157.48" y1="35.56" x2="121.92" y2="35.56" width="0.1524" layer="91"/>
+<junction x="121.92" y="35.56"/>
+<pinref part="R2" gate="G$1" pin="1"/>
+<wire x1="170.18" y1="48.26" x2="170.18" y2="35.56" width="0.1524" layer="91"/>
+<wire x1="170.18" y1="35.56" x2="157.48" y2="35.56" width="0.1524" layer="91"/>
+<junction x="157.48" y="35.56"/>
+<pinref part="C2" gate="G$1" pin="1"/>
+<wire x1="185.42" y1="60.96" x2="185.42" y2="35.56" width="0.1524" layer="91"/>
+<wire x1="185.42" y1="35.56" x2="170.18" y2="35.56" width="0.1524" layer="91"/>
+<junction x="170.18" y="35.56"/>
 </segment>
 </net>
@@
 <wire x1="127" y1="66.04" x2="127" y2="78.74" width="0.1524" layer="91"/>
 <wire x1="127" y1="78.74" x2="134.62" y2="78.74" width="0.1524" layer="91"/>
+<pinref part="U2" gate="G$1" pin="EN"/>
+<wire x1="129.54" y1="63.5" x2="127" y2="63.5" width="0.1524" layer="91"/>
+<wire x1="127" y1="63.5" x2="127" y2="66.04" width="0.1524" layer="91"/>
+<junction x="127" y="66.04"/>
+<pinref part="C1" gate="G$1" pin="2"/>
+<wire x1="121.92" y1="63.5" x2="121.92" y2="66.04" width="0.1524" layer="91"/>
+<wire x1="121.92" y1="66.04" x2="127" y2="66.04" width="0.1524" layer="91"/>
+<wire x1="121.92" y1="66.04" x2="121.92" y2="81.28" width="0.1524" layer="91"/>
+<junction x="121.92" y="66.04"/>
+<pinref part="S1" gate="G$1" pin="2"/>
+<wire x1="121.92" y1="81.28" x2="81.28" y2="81.28" width="0.1524" layer="91"/>
 </segment>
 </net>
@@
 <pinref part="U2" gate="G$1" pin="SW"/>
 <wire x1="157.48" y1="68.58" x2="154.94" y2="68.58" width="0.1524" layer="91"/>
-</segment>
-</net>
+<pinref part="D4" gate="A" pin="A"/>
+<wire x1="160.02" y1="88.9" x2="157.48" y2="88.9" width="0.1524" layer="91"/>
+<wire x1="157.48" y1="88.9" x2="157.48" y2="78.74" width="0.1524" layer="91"/>
+<junction x="157.48" y="78.74"/>
+</segment>
+</net>
+<net name="N$12" class="0">
+<segment>
+<pinref part="U2" gate="G$1" pin="FB"/>
+<wire x1="154.94" y1="63.5" x2="170.18" y2="63.5" width="0.1524" layer="91"/>
+<pinref part="R1" gate="G$1" pin="A"/>
+<wire x1="170.18" y1="63.5" x2="170.18" y2="68.58" width="0.1524" layer="91"/>
+<pinref part="R2" gate="G$1" pin="2"/>
+<wire x1="170.18" y1="63.5" x2="170.18" y2="58.42" width="0.1524" layer="91"/>
+<junction x="170.18" y="63.5"/>
+</segment>
+</net>
+<net name="N$14" class="0">
+<segment>
+<pinref part="R1" gate="G$1" pin="E"/>
+<wire x1="170.18" y1="78.74" x2="170.18" y2="88.9" width="0.1524" layer="91"/>
+<pinref part="D4" gate="A" pin="C"/>
+<wire x1="170.18" y1="88.9" x2="165.1" y2="88.9" width="0.1524" layer="91"/>
+<pinref part="C2" gate="G$1" pin="2"/>
+<wire x1="170.18" y1="88.9" x2="185.42" y2="88.9" width="0.1524" layer="91"/>
+<wire x1="185.42" y1="88.9" x2="185.42" y2="68.58" width="0.1524" layer="91"/>
+<junction x="170.18" y="88.9"/>
+</segment>
+</net>

Commit message: Power Schematic
Parts:
- added 10UH: MLZ2012N100LT000, MLZ2012N100LT000:MLZ2012N100LT000
- added C3: 2.2uF, SparkFun-Capacitors:2.2UF-0603-10V-20%
- added C4: 10uF, SparkFun-Capacitors:10UF-0603-6.3V-20%
- added U3: LTC3531ES6-3_3, LTC3531ES6-3_3:LTC3531ES6-3_3
Connections:
- removed net N$1: C1.2, S1.2, U$1.1, U2.EN, U2.IN
- new net N$11: C1.2, C3.1, S1.2, U$1.1, U2.EN, U2.IN, U3.*SHDN, U3.VIN
- new net N$26: C4.1, U3.VOUT
- new net N$4: 10UH.1, U3.SW1
- new net N$6: 10UH.2, U3.SW2
- net N$25: now also C3.2, C4.2, U3.GND/PGND
Changed lines of the file:
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@@
 <part name="C1" library="SparkFun-Capacitors" deviceset="22NF/22,000PF" device="-0603-50V-10%" value="22uF"/>
 <part name="C2" library="SparkFun-Capacitors" deviceset="22NF/22,000PF" device="-0603-50V-10%" value="22uF"/>
+<part name="U3" library="LTC3531ES6-3_3" deviceset="LTC3531ES6-3_3" device=""/>
+<part name="C3" library="SparkFun-Capacitors" deviceset="2.2UF" device="-0603-10V-20%" value="2.2uF"/>
+<part name="C4" library="SparkFun-Capacitors" deviceset="10UF" device="-0603-6.3V-20%" value="10uF"/>
+<part name="10UH" library="MLZ2012N100LT000" deviceset="MLZ2012N100LT000" device=""/>
 </parts>
 <sheets>
@@
 <attribute name="NAME" x="183.896" y="63.119" size="1.778" layer="95" font="vector" rot="R180"/>
 <attribute name="VALUE" x="183.896" y="68.199" size="1.778" layer="96" font="vector" rot="R180"/>
+</instance>
+<instance part="U3" gate="A" x="294.64" y="66.04" smashed="yes" rot="MR0">
+<attribute name="NAME" x="263.8044" y="75.1586" size="2.0828" layer="95" ratio="6" rot="SMR0"/>
+<attribute name="VALUE" x="264.4394" y="72.6186" size="2.0828" layer="96" ratio="6" rot="SMR0"/>
+</instance>
+<instance part="C3" gate="G$1" x="210.82" y="58.42" smashed="yes">
+<attribute name="NAME" x="212.344" y="61.341" size="1.778" layer="95" font="vector"/>
+<attribute name="VALUE" x="212.344" y="56.261" size="1.778" layer="96" font="vector"/>
+</instance>
+<instance part="C4" gate="G$1" x="307.34" y="55.88" smashed="yes">
+<attribute name="NAME" x="308.864" y="58.801" size="1.778" layer="95" font="vector"/>
+<attribute name="VALUE" x="308.864" y="53.721" size="1.778" layer="96" font="vector"/>
+</instance>
+<instance part="10UH" gate="G$1" x="254" y="81.28" smashed="yes">
+<attribute name="NAME" x="248.91533125" y="83.822340625" size="1.779640625" layer="95"/>
+<attribute name="VALUE" x="248.915609375" y="78.737809375" size="1.77953125" layer="96"/>
 </instance>
 </instances>
@@
 <wire x1="185.42" y1="35.56" x2="170.18" y2="35.56" width="0.1524" layer="91"/>
 <junction x="170.18" y="35.56"/>
+<pinref part="C3" gate="G$1" pin="2"/>
+<wire x1="210.82" y1="55.88" x2="210.82" y2="35.56" width="0.1524" layer="91"/>
+<wire x1="210.82" y1="35.56" x2="185.42" y2="35.56" width="0.1524" layer="91"/>
+<junction x="185.42" y="35.56"/>
+<pinref part="U3" gate="A" pin="GND/PGND"/>
+<wire x1="294.64" y1="63.5" x2="297.18" y2="63.5" width="0.1524" layer="91"/>
+<wire x1="297.18" y1="63.5" x2="297.18" y2="35.56" width="0.1524" layer="91"/>
+<wire x1="297.18" y1="35.56" x2="210.82" y2="35.56" width="0.1524" layer="91"/>
+<junction x="210.82" y="35.56"/>
+<pinref part="C4" gate="G$1" pin="2"/>
+<wire x1="307.34" y1="53.34" x2="307.34" y2="35.56" width="0.1524" layer="91"/>
+<wire x1="307.34" y1="35.56" x2="297.18" y2="35.56" width="0.1524" layer="91"/>
+<junction x="297.18" y="35.56"/>
 </segment>
 </net>
@@
 </segment>
 </net>
-<net name="N$1" class="0">
-<segment>
+<net name="N$3" class="0">
+<segment>
+<pinref part="U$1" gate="G$1" pin="2"/>
+<wire x1="149.86" y1="78.74" x2="157.48" y2="78.74" width="0.1524" layer="91"/>
+<wire x1="157.48" y1="78.74" x2="157.48" y2="68.58" width="0.1524" layer="91"/>
+<pinref part="U2" gate="G$1" pin="SW"/>
+<wire x1="157.48" y1="68.58" x2="154.94" y2="68.58" width="0.1524" layer="91"/>
+<pinref part="D4" gate="A" pin="A"/>
+<wire x1="160.02" y1="88.9" x2="157.48" y2="88.9" width="0.1524" layer="91"/>
+<wire x1="157.48" y1="88.9" x2="157.48" y2="78.74" width="0.1524" layer="91"/>
+<junction x="157.48" y="78.74"/>
+</segment>
+</net>
+<net name="N$12" class="0">
+<segment>
+<pinref part="U2" gate="G$1" pin="FB"/>
+<wire x1="154.94" y1="63.5" x2="170.18" y2="63.5" width="0.1524" layer="91"/>
+<pinref part="R1" gate="G$1" pin="A"/>
+<wire x1="170.18" y1="63.5" x2="170.18" y2="68.58" width="0.1524" layer="91"/>
+<pinref part="R2" gate="G$1" pin="2"/>
+<wire x1="170.18" y1="63.5" x2="170.18" y2="58.42" width="0.1524" layer="91"/>
+<junction x="170.18" y="63.5"/>
+</segment>
+</net>
+<net name="N$14" class="0">
+<segment>
+<pinref part="R1" gate="G$1" pin="E"/>
+<wire x1="170.18" y1="78.74" x2="170.18" y2="88.9" width="0.1524" layer="91"/>
+<pinref part="D4" gate="A" pin="C"/>
+<wire x1="170.18" y1="88.9" x2="165.1" y2="88.9" width="0.1524" layer="91"/>
+<pinref part="C2" gate="G$1" pin="2"/>
+<wire x1="170.18" y1="88.9" x2="185.42" y2="88.9" width="0.1524" layer="91"/>
+<wire x1="185.42" y1="88.9" x2="185.42" y2="68.58" width="0.1524" layer="91"/>
+<junction x="170.18" y="88.9"/>
+</segment>
+</net>
+<net name="N$4" class="0">
+<segment>
+<pinref part="U3" gate="A" pin="SW1"/>
+<wire x1="223.52" y1="66.04" x2="218.44" y2="66.04" width="0.1524" layer="91"/>
+<pinref part="10UH" gate="G$1" pin="1"/>
+<wire x1="218.44" y1="66.04" x2="218.44" y2="81.28" width="0.1524" layer="91"/>
+<wire x1="218.44" y1="81.28" x2="248.92" y2="81.28" width="0.1524" layer="91"/>
+</segment>
+</net>
+<net name="N$6" class="0">
+<segment>
+<pinref part="10UH" gate="G$1" pin="2"/>
+<wire x1="259.08" y1="81.28" x2="297.18" y2="81.28" width="0.1524" layer="91"/>
+<wire x1="297.18" y1="81.28" x2="297.18" y2="66.04" width="0.1524" layer="91"/>
+<pinref part="U3" gate="A" pin="SW2"/>
+<wire x1="297.18" y1="66.04" x2="294.64" y2="66.04" width="0.1524" layer="91"/>
+</segment>
+</net>
+<net name="N$11" class="0">
+<segment>
+<pinref part="U3" gate="A" pin="VIN"/>
+<pinref part="C3" gate="G$1" pin="1"/>
+<wire x1="223.52" y1="63.5" x2="218.44" y2="63.5" width="0.1524" layer="91"/>
+<pinref part="U3" gate="A" pin="*SHDN"/>
+<wire x1="218.44" y1="63.5" x2="210.82" y2="63.5" width="0.1524" layer="91"/>
+<wire x1="223.52" y1="60.96" x2="218.44" y2="60.96" width="0.1524" layer="91"/>
+<wire x1="218.44" y1="60.96" x2="218.44" y2="63.5" width="0.1524" layer="91"/>
+<junction x="218.44" y="63.5"/>
+<wire x1="210.82" y1="63.5" x2="210.82" y2="99.06" width="0.1524" layer="91"/>
+<junction x="210.82" y="63.5"/>
 <pinref part="U2" gate="G$1" pin="IN"/>
 <wire x1="129.54" y1="66.04" x2="127" y2="66.04" width="0.1524" layer="91"/>
@@
 <pinref part="S1" gate="G$1" pin="2"/>
 <wire x1="121.92" y1="81.28" x2="81.28" y2="81.28" width="0.1524" layer="91"/>
-</segment>
-</net>
-<net name="N$3" class="0">
-<segment>
-<pinref part="U$1" gate="G$1" pin="2"/>
-<wire x1="149.86" y1="78.74" x2="157.48" y2="78.74" width="0.1524" layer="91"/>
-<wire x1="157.48" y1="78.74" x2="157.48" y2="68.58" width="0.1524" layer="91"/>
-<pinref part="U2" gate="G$1" pin="SW"/>
-<wire x1="157.48" y1="68.58" x2="154.94" y2="68.58" width="0.1524" layer="91"/>
-<pinref part="D4" gate="A" pin="A"/>
-<wire x1="160.02" y1="88.9" x2="157.48" y2="88.9" width="0.1524" layer="91"/>
-<wire x1="157.48" y1="88.9" x2="157.48" y2="78.74" width="0.1524" layer="91"/>
-<junction x="157.48" y="78.74"/>
-</segment>
-</net>
-<net name="N$12" class="0">
-<segment>
-<pinref part="U2" gate="G$1" pin="FB"/>
-<wire x1="154.94" y1="63.5" x2="170.18" y2="63.5" width="0.1524" layer="91"/>
-<pinref part="R1" gate="G$1" pin="A"/>
-<wire x1="170.18" y1="63.5" x2="170.18" y2="68.58" width="0.1524" layer="91"/>
-<pinref part="R2" gate="G$1" pin="2"/>
-<wire x1="170.18" y1="63.5" x2="170.18" y2="58.42" width="0.1524" layer="91"/>
-<junction x="170.18" y="63.5"/>
-</segment>
-</net>
-<net name="N$14" class="0">
-<segment>
-<pinref part="R1" gate="G$1" pin="E"/>
-<wire x1="170.18" y1="78.74" x2="170.18" y2="88.9" width="0.1524" layer="91"/>
-<pinref part="D4" gate="A" pin="C"/>
-<wire x1="170.18" y1="88.9" x2="165.1" y2="88.9" width="0.1524" layer="91"/>
-<pinref part="C2" gate="G$1" pin="2"/>
-<wire x1="170.18" y1="88.9" x2="185.42" y2="88.9" width="0.1524" layer="91"/>
-<wire x1="185.42" y1="88.9" x2="185.42" y2="68.58" width="0.1524" layer="91"/>
-<junction x="170.18" y="88.9"/>
-</segment>
-</net>
+<wire x1="210.82" y1="99.06" x2="121.92" y2="99.06" width="0.1524" layer="91"/>
+<wire x1="121.92" y1="99.06" x2="121.92" y2="81.28" width="0.1524" layer="91"/>
+<junction x="121.92" y="81.28"/>
+</segment>
+</net>
+<net name="N$26" class="0">
+<segment>
+<pinref part="U3" gate="A" pin="VOUT"/>
+<pinref part="C4" gate="G$1" pin="1"/>
+<wire x1="294.64" y1="60.96" x2="307.34" y2="60.96" width="0.1524" layer="91"/>
+</segment>
+</net>

Commit message: Update motherBoard_Power.sch
Connections:
- net N$12: now also R1.S; no longer R1.A
Changed lines of the file:
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@@
 <setting verticaltext="up"/>
 </settings>
-<grid distance="0.1" unitdist="inch" unit="inch" style="lines" multiple="1" display="yes" altdistance="0.01" altunitdist="inch" altunit="inch"/>
+<grid distance="0.1" unitdist="inch" unit="inch" style="lines" multiple="1" display="no" altdistance="0.01" altunitdist="inch" altunit="inch"/>
 <layers>
 <layer number="1" name="Top" color="4" fill="1" visible="no" active="no"/>
@@
 <pinref part="U2" gate="G$1" pin="FB"/>
 <wire x1="154.94" y1="63.5" x2="170.18" y2="63.5" width="0.1524" layer="91"/>
-<pinref part="R1" gate="G$1" pin="A"/>
-<wire x1="170.18" y1="63.5" x2="170.18" y2="68.58" width="0.1524" layer="91"/>
 <pinref part="R2" gate="G$1" pin="2"/>
 <wire x1="170.18" y1="63.5" x2="170.18" y2="58.42" width="0.1524" layer="91"/>
+<wire x1="170.18" y1="63.5" x2="170.18" y2="66.04" width="0.1524" layer="91"/>
 <junction x="170.18" y="63.5"/>
+<wire x1="170.18" y1="66.04" x2="162.56" y2="66.04" width="0.1524" layer="91"/>
+<wire x1="162.56" y1="66.04" x2="162.56" y2="73.66" width="0.1524" layer="91"/>
+<pinref part="R1" gate="G$1" pin="S"/>
+<wire x1="162.56" y1="73.66" x2="165.1" y2="73.66" width="0.1524" layer="91"/>
 </segment>
 </net>
 <net name="N$14" class="0">
 <segment>
-<pinref part="R1" gate="G$1" pin="E"/>
-<wire x1="170.18" y1="78.74" x2="170.18" y2="88.9" width="0.1524" layer="91"/>
 <pinref part="D4" gate="A" pin="C"/>
-<wire x1="170.18" y1="88.9" x2="165.1" y2="88.9" width="0.1524" layer="91"/>
 <pinref part="C2" gate="G$1" pin="2"/>
+<wire x1="165.1" y1="88.9" x2="170.18" y2="88.9" width="0.1524" layer="91"/>
 <wire x1="170.18" y1="88.9" x2="185.42" y2="88.9" width="0.1524" layer="91"/>
 <wire x1="185.42" y1="88.9" x2="185.42" y2="68.58" width="0.1524" layer="91"/>
+<pinref part="R1" gate="G$1" pin="E"/>
+<wire x1="170.18" y1="88.9" x2="170.18" y2="78.74" width="0.1524" layer="91"/>
 <junction x="170.18" y="88.9"/>
 </segment>

Commit message: Update motherBoard_Power.sch
Parts:
- removed 0.1: RL1220S-R10-F, RL1220S-R10-F:RL1220S-R10-F
- added 0.1U1, 0.UF1: C0805C104K4RACTU, C0805C104K4RACTU:C0805C104K4RACTU
- added 1: ERJP6WF3300V, ERJP6WF3300V:ERJP6WF3300V
- added 100K1: CRGH0805J100K, CRGH0805J100K:CRGH0805J100K
- added 10U1, 10UF1: GRM21BC81C106KE15L, GRM21BC81C106KE15L:GRM21BC81C106KE15L
- added 10UH1: MLZ2012N100LT000, MLZ2012N100LT000:MLZ2012N100LT000
- added 2.7K1: ERA-6AEB272V, ERA-6AEB272V:ERA-6AEB272V
- added 3.6V_LI-ION1: SL-160AA/PR, battery:SL-160AA/PR
- added C5, C6: 22uF, SparkFun-Capacitors:22NF/22,000PF-0603-50V-10%
- added C7: 2.2uF, SparkFun-Capacitors:2.2UF-0603-10V-20%
- added C8: 10uF, SparkFun-Capacitors:10UF-0603-6.3V-20%
- added D1: LTST-C191KGKT, LTST-C191KGKT:LTST-C191KGKT
- added D2, D6: SS34, SS34:SS34
- added J1: 10118193-0001LF, 10118193-0001LF:10118193-0001LF
- added R3, R6: 0.1, SparkFun-Resistors:RESISTOR0805
- added R4: (no value), rcl:R-TRIMM3296P
- added R5: 1k, SparkFun-Resistors:1KOHM-0603-1/10W-1%
- added S2: JS102011SAQN, JS102011SAQN:JS102011SAQN
- added U$10: CDRH104R, CDRH104R:CDRH104R
- added U$2: NDS8434, NDS8434:NDS8434
- added U$7: AP9101C, AP910C:AP9101C
- added U$8, U$9: ZXM61N02F, ZXM61N02F:ZXM61N02F
- added U4: MCP7384XX, SparkFun-IC-Power:MCP7384XX
- added U5: MT3608, MT3608:MT3608
- added U6: LTC3531ES6-3_3, LTC3531ES6-3_3:LTC3531ES6-3_3
Connections:
- new net N$1: 100K1.2, 10UF1.1, D1.A2, D6.C, R6.1, U4.VDD
- new net N$13: D1.K2, U4.STAT1
- new net N$15: 100K1.1, U4.EN
- new net N$16: R6.2, U$2.D@1, U4.SENSE
- new net N$27: 0.UF1.1, U4.TIMER
- new net N$28: 10U1.1, U4.VBAT
- new net N$29: 1.1, 3.6V_LI-ION1.+, S2.1, U$2.S@3
- new net N$30: U$2.G, U4.DRV
- new net N$31: 0.1U1.1, 1.2, U$7.VDD
- new net N$32: U$8.D, U$9.D
- new net N$33: U$7.DO, U$8.G
- new net N$34: U$7.CO, U$9.G
- new net N$35: 2.7K1.R1, U$7.VM
- new net N$36: 2.7K1.R2, C5.1, C6.1, C7.2, C8.2, R5.1, U$9.S, U5.GND, U6.GND/PGND
- new net N$37: D6.A, J1.VUSB
- new net N$38: D2.A, U$10.2, U5.SW
- new net N$39: R4.S, R5.2, U5.FB
- new net N$40: C6.2, D2.C, R4.E
- new net N$41: 10UH1.1, U6.SW1
- new net N$42: 10UH1.2, U6.SW2
- new net N$43: C5.2, C7.1, S2.2, U$10.1, U5.EN, U5.IN, U6.*SHDN, U6.VIN
- new net N$44: C8.1, U6.VOUT
- net GND: now also 0.1U1.2, 0.UF1.2, 10U1.2, 10UF1.2, 3.6V_LI-ION1.-, J1.GND, U$7.VSS, U$8.S, U4.VSS
- net N$5: now also R3.1; no longer 0.1.R2
- net N$9: now also R3.2; no longer 0.1.R1
