File: eagle/projects/smartBobber Mother Board/motherBoard/motherBoard_Power.sch (EAGLE design)
At the start: 58 parts, among them J1 10118193-0001LF, J4 10118193-0001LF, U1 MCP7384XX, U2 MT3608, U3 LTC3531ES6-3_3, U4 MCP7384XX, U5 MT3608, U6 LTC3531ES6-3_3

Commit message: Update motherBoard_Power.sch
Parts:
- removed 0.1U, 0.UF: C0805C104K4RACTU, C0805C104K4RACTU:C0805C104K4RACTU
- removed 100K: CRGH0805J100K, CRGH0805J100K:CRGH0805J100K
- removed 10U, 10UF: GRM21BC81C106KE15L, GRM21BC81C106KE15L:GRM21BC81C106KE15L
- removed 2.7K: ERA-6AEB272V, ERA-6AEB272V:ERA-6AEB272V
- removed 330: ERJP6WF3300V, ERJP6WF3300V:ERJP6WF3300V
- removed C4: 10uF, SparkFun-Capacitors:10UF-0603-6.3V-20%
- removed R2: 1k, SparkFun-Resistors:1KOHM-0603-1/10W-1%
- added C10, C9: 10uF, SparkFun-Capacitors:10UF-0603-6.3V-20%
- added C11, C12: 0.1uF, SparkFun-Capacitors:0.1UF-0603-25V-(+80/-20%)
- added C13: 2.2uF, SparkFun-Capacitors:2.2UF-0603-10V-20%
- added R10: 1.5K, SparkFun-Resistors:RESISTOR0603
- added R7: 100K, SparkFun-Resistors:RESISTOR0603
- added R8: 330, SparkFun-Resistors:RESISTOR0603
- added R9: 2.7K, SparkFun-Resistors:RESISTOR0603
- C1, C2: device SparkFun-Capacitors:22NF/22,000PF-0603-50V-10% -> SparkFun-Capacitors:10UF-0603-6.3V-20%
- C3: value 2.2uF -> 10uF; device SparkFun-Capacitors:2.2UF-0603-10V-20% -> SparkFun-Capacitors:10UF-0603-6.3V-20%
Connections:
- removed net N$14: C2.2, D4.C, R1.E
- removed net N$26: C4.1, U3.VOUT
- new net 12V: C2.1, D4.C, R1.E
- new net 3.3V: C3.1, U3.VOUT
- net GND: now also C10.2, C11.2, C12.2, C9.2; no longer 0.1U.2, 0.UF.2, 10U.2, 10UF.2
- net N$11: now also C1.1, C13.1; no longer C1.2, C3.1
- net N$12: now also R10.2; no longer R2.2
- net N$17: now also C11.1; no longer 0.UF.1
- net N$18: now also C10.1; no longer 10U.1
- net N$19: now also R8.1; no longer 330.1
- net N$20: now also C12.1, R8.2; no longer 0.1U.1, 330.2
- net N$24: now also R9.2; no longer 2.7K.R1
- net N$25: now also C1.2, C13.2, C2.2, R10.1, R9.1; no longer 2.7K.R2, C1.1, C2.1, C4.2, R2.1
- net N$5: now also C9.1, R7.1; no longer 100K.2, 10UF.1
- net N$8: now also R7.2; no longer 100K.1
Other:
- moved on the sheet: C1, C2, C3
