File: eagle/projects/smartBobber Mother Board/motherBoard/motherBoard_Power.sch (EAGLE design)
At the start: 58 parts, among them J1 10118193-0001LF, J4 10118193-0001LF, U1 MCP7384XX, U2 MT3608, U3 LTC3531ES6-3_3, U4 MCP7384XX, U5 MT3608, U6 LTC3531ES6-3_3

Commit message: Update motherBoard_Power.sch
Connections:
- removed net N$25: C1.2, C13.2, C2.2, C3.2, R10.1, R9.1, U$6.S, U2.GND, U3.GND/PGND
- net GND: now also C1.2, C13.2, C2.2, C3.2, R10.1, R9.1, U$6.S, U2.GND, U3.GND/PGND
