File: eagle/projects/smartBobber Mother Board/motherBoard/motherBoard.sch (EAGLE design)
At the start: 46 parts, among them J4 10118193-0001LF, Q1 2A/20V/150mΩ, Q2 MMBT3904, U1 MCP7384XX, U2 MT3608, Y1 ECS-40-S-4X

Commit message: Update motherBoard.sch
Parts:
- removed 0.1: RL1220S-R10-F, RL1220S-R10-F:RL1220S-R10-F
- removed 0.1U, 0.UF: C0805C104K4RACTU, C0805C104K4RACTU:C0805C104K4RACTU
- removed 100K: CRGH0805J100K, CRGH0805J100K:CRGH0805J100K
- removed 10U, 10UF: GRM21BC81C106KE15L, GRM21BC81C106KE15L:GRM21BC81C106KE15L
- removed 2.7K: ERA-6AEB272V, ERA-6AEB272V:ERA-6AEB272V
- removed 3.6V_LI-ION: SL-160AA/PR, battery:SL-160AA/PR
- removed 330: ERJP6WF3300V, ERJP6WF3300V:ERJP6WF3300V
- added 10UH: MLZ2012N100LT000, MLZ2012N100LT000:MLZ2012N100LT000
- added C10, C7, C9: 10uF, SparkFun-Capacitors:10UF-0603-6.3V-20%
- added C11, C12: 0.1uF, SparkFun-Capacitors:0.1UF-0603-25V-(+80/-20%)
- added C13: 2.2uF, SparkFun-Capacitors:2.2UF-0603-10V-20%
- added C3, C5: 22uF, SparkFun-Capacitors:10UF-0603-6.3V-20%
- added C6: 0.1uF, SparkFun-Capacitors:0.1UF-0603-25V-5%
- added J5: (no value), SparkFun-Connectors:CONN_02
- added J6: 1053131202, 1053131202:1053131202
- added R1, R9: 10K, SparkFun-Resistors:RESISTOR0603
- added R10: 10k, SparkFun-Resistors:RESISTOR0603
- added R11: 100k, SparkFun-Resistors:RESISTOR0603
- added R12: (no value), rcl:R-TRIMM3296P
- added R13: 0.1, SparkFun-Resistors:RESISTOR0805
- added R14: 100K, SparkFun-Resistors:RESISTOR0603
- added R15: 330, SparkFun-Resistors:RESISTOR0603
- added R16: 2.7K, SparkFun-Resistors:RESISTOR0603
- added R17: 1.5K, SparkFun-Resistors:RESISTOR0603
- added S2: Button, SparkFun-Switches:MOMENTARY-SWITCH-SPST-SMD-5.2MM
- added U$2: CDRH104R, CDRH104R:CDRH104R
- added U3: LTC3531ES6-3_3, LTC3531ES6-3_3:LTC3531ES6-3_3
- J1: value (none) -> 10118193-0001LF; device SparkFun-Connectors:CONN_06POLAR -> 10118193-0001LF:10118193-0001LF
- J2: device SparkFun-Connectors:CONN_06POLAR -> SparkFun-Connectors:CONN_05JST-VERT
- J4: value 10118193-0001LF -> (none); device 10118193-0001LF:10118193-0001LF -> SparkFun-Connectors:CONN_06SILK_FEMALE_PTH
Connections:
- removed net N$18: 10U.1, U1.VBAT
- removed net N$25: 2.7K.R2, U$6.S
- removed net TEMP_SENS: U$1.RC3/SCK/SCL
- removed net VDD: J1.2
- new net 3.3V: C6.1, C7.1, J2.4, J4.2, R1.2, U$1.VDD, U3.VOUT
- new net BLUETOOTH_ON/OFF: J2.1, R10.2, U$1.RB0/INT
- new net TEMP_DQ: J3.2, R9.2, U$1.RC3/SCK/SCL
- new net VCC: J3.3, J5.2, Q1G1.S, R4.1, R9.1
- net 12V: now also C5.1, D4.C, R12.E; no longer Q1G1.S, R4.1
- net ADC: now also R11.1, R11.2
- net GND: now also C10.2, C11.2, C12.2, C13.2, C3.2, C5.2, C6.2, C7.2, C9.2, J1.GND, J2.5, J3.1, J4.3, J5.1, J6.2, R10.1, R16.1, R17.1, S2.1, U$1.VSS, U$1.VSS_2, U$6.S, U2.GND, U3.GND/PGND; no longer 0.1U.2, 0.UF.2, 10U.2, 10UF.2, 3.6V_LI-ION.-, J1.3, J4.GND
- net LVP: now also J4.6; no longer J1.6
- net MCLR: now also J4.1; no longer J1.1
- net N$11: now also D5.A, J1.VUSB; no longer J2.6
- net N$12: now also D4.A, U$2.2, U2.SW; no longer J2.5
- net N$13: now also R12.S, R17.2, U2.FB; no longer J2.4
- net N$14: now also 10UH.1, U3.SW1; no longer J2.3
- net N$15: now also 10UH.2, U3.SW2; no longer J2.2
- net N$16: now also C13.1, C3.1, S1.2, U$2.1, U2.EN, U2.IN, U3.*SHDN, U3.VIN; no longer J2.1
- net N$17: now also C11.1; no longer 0.UF.1
- net N$19: now also C10.1, J6.1, R15.1, U1.VBAT; no longer 3.6V_LI-ION.+, 330.1
- net N$2: now also C9.1, D3.A2, D5.C, R13.1, R14.1, U1.VDD; no longer D5.A, J4.VUSB
- net N$20: now also C12.1, R15.2; no longer 0.1U.1, 330.2
- net N$24: now also R16.2; no longer 2.7K.R1
- net N$5: now also R1.1, S2.2, U$1.~MCLR/VPP; no longer 0.1.R2, 100K.2, 10UF.1, D3.A2, D5.C, U1.VDD
- net N$8: now also R14.2; no longer 100K.1
- net N$9: now also R13.2; no longer 0.1.R1
- net PGC: now also J4.5; no longer J1.5
- net PGD: now also J4.4; no longer J1.4
- net RX: now also J2.3
- net TX: now also J2.2
Other:
- note added: "12V Supply Circuit"
- note added: "3.3V Supply Circuit"
- note added: "Charging Circuit"
- note added: "EXTERNAL CLOCK"
- note added: "HEADERS"
- note added: "LED ARRAYS"
- note added: "MICROCONTROLLER"
- note added: "Protection Circuit"
- note added: "SOLENOID DETECTOR"
- note added: "SOLENOID DRIVER"
- note added: "TEST POWER SUPPLY"
- moved on the sheet: BLED1, BLED2, BLED3, C1, C2, C4, D1, D2, D3, D4, D5, J3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

Commit message: MCP73831
Parts:
- removed C10: 10uF, SparkFun-Capacitors:10UF-0603-6.3V-20%
- removed D5: SS34, SS34:SS34
- removed U$3: NDS8434, NDS8434:NDS8434
- C11: value 0.1uF -> 4.7uF
- C9: value 10uF -> 4.7uF
- R13: value 0.1 -> 2k
- R14: value 100K -> 470
- U1: value MCP7384XX -> MCP73831; device SparkFun-IC-Power:MCP7384XX -> SparkFun-IC-Power:MCP73831
Connections:
- removed net N$10: U$3.G, U1.DRV
- removed net N$17: C11.1, U1.TIMER
- removed net N$19: C10.1, J6.1, R15.1, S1.1, U$3.S@3, U1.VBAT
- net GND: now also R13.1; no longer C10.2
- net N$11: now also C9.1, D3.A2, U1.VIN; no longer D5.A
- net N$2: now also D3.K2, R14.2; no longer C9.1, D3.A2, D5.C, R13.1, R14.1, U1.VDD
- net N$7: now also R14.1, U1.STAT; no longer D3.K2, U1.STAT1
- net N$8: now also C11.1, J6.1, R15.1, S1.1, U1.VBAT; no longer R14.2, U1.EN
- net N$9: now also U1.PROG; no longer U$3.D@1, U1.SENSE
Other:
- moved on the sheet: C11, C9, D3, R13, R14

Commit message: Update motherBoard.sch
Parts:
- removed U$4: AP9101C, AP910C:AP9101C
- removed U$5, U$6: ZXM61N02F, ZXM61N02F:ZXM61N02F
- added U$3: FS312F-G, FS312F-G:FS312F-G
- R15: value 330 -> 100
Connections:
- removed net N$21: U$5.D, U$6.D
- removed net N$22: U$4.DO, U$5.G
- removed net N$23: U$4.CO, U$6.G
- removed net N$24: R16.2, U$4.VM
- net GND: now also U$3.GND; no longer U$4.VSS, U$5.S, U$6.S
- net N$20: now also U$3.VCC; no longer U$4.VDD
Changed lines of the file:
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@@
 <part name="SUPPLY4" library="supply2" library_urn="urn:adsk.eagle:library:372" deviceset="GND" device="" value="GND1"/>
 <part name="SUPPLY5" library="supply2" library_urn="urn:adsk.eagle:library:372" deviceset="GND" device="" value="GND1"/>
-<part name="U$4" library="AP910C" deviceset="AP9101C" device=""/>
 <part name="S1" library="JS102011SAQN" deviceset="JS102011SAQN" device=""/>
-<part name="U$5" library="ZXM61N02F" deviceset="ZXM61N02F" device=""/>
-<part name="U$6" library="ZXM61N02F" deviceset="ZXM61N02F" device=""/>
 <part name="U2" library="MT3608" deviceset="MT3608" device=""/>
 <part name="D4" library="SS34" deviceset="SS34" device=""/>
@@
 <part name="R13" library="SparkFun-Resistors" deviceset="RESISTOR" device="0805" value="2k"/>
 <part name="R14" library="SparkFun-Resistors" deviceset="RESISTOR" device="0603" value="470"/>
-<part name="R15" library="SparkFun-Resistors" deviceset="RESISTOR" device="0603" value="330"/>
+<part name="R15" library="SparkFun-Resistors" deviceset="RESISTOR" device="0603" value="100"/>
 <part name="R16" library="SparkFun-Resistors" deviceset="RESISTOR" device="0603" value=" 2.7K"/>
 <part name="R17" library="SparkFun-Resistors" deviceset="RESISTOR" device="0603" value=" 1.5K"/>
@@
 <part name="GND11" library="SparkFun-PowerSymbols" deviceset="GND" device=""/>
 <part name="U1" library="SparkFun-IC-Power" deviceset="MCP73831" device=""/>
+<part name="U$3" library="FS312F-G" deviceset="FS312F-G" device=""/>
 </parts>
 <sheets>
@@
 <attribute name="VALUE" x="142.875" y="12.065" size="1.778" layer="96"/>
 </instance>
-<instance part="U$4" gate="G$1" x="195.58" y="48.26" smashed="yes"/>
 <instance part="S1" gate="G$1" x="193.04" y="66.04" smashed="yes">
 <attribute name="NAME" x="185.417090625" y="71.121940625" size="1.270490625" layer="95"/>
 <attribute name="VALUE" x="185.411440625" y="60.954290625" size="1.27143125" layer="96"/>
-</instance>
-<instance part="U$5" gate="G$1" x="195.58" y="25.4" smashed="yes" rot="R270">
-<attribute name="VALUE" x="190.5" y="21.5754" size="1.78026875" layer="96" rot="R90"/>
-</instance>
-<instance part="U$6" gate="G$1" x="205.74" y="25.4" smashed="yes" rot="MR270">
-<attribute name="VALUE" x="210.82" y="21.5754" size="1.78026875" layer="96" rot="MR90"/>
 </instance>
 <instance part="U2" gate="G$1" x="274.32" y="53.34" smashed="yes" rot="MR0">
@@
 <attribute name="VALUE" x="83.82" y="30.48" size="1.778" layer="96"/>
 </instance>
+<instance part="U$3" gate="G$1" x="185.42" y="53.34" smashed="yes" rot="R180"/>
 </instances>
 <busses>
@@
 <segment>
 <pinref part="SUPPLY5" gate="GND" pin="GND"/>
-<pinref part="U$5" gate="G$1" pin="S"/>
 <wire x1="144.78" y1="20.32" x2="144.78" y2="17.78" width="0.1524" layer="91"/>
 <wire x1="144.78" y1="20.32" x2="167.64" y2="20.32" width="0.1524" layer="91"/>
-<wire x1="167.64" y1="20.32" x2="175.26" y2="20.32" width="0.1524" layer="91"/>
-<wire x1="175.26" y1="20.32" x2="193.04" y2="20.32" width="0.1524" layer="91"/>
-<pinref part="U$4" gate="G$1" pin="VSS"/>
-<wire x1="177.8" y1="43.18" x2="175.26" y2="43.18" width="0.1524" layer="91"/>
-<wire x1="175.26" y1="43.18" x2="175.26" y2="20.32" width="0.1524" layer="91"/>
-<junction x="175.26" y="20.32"/>
+<wire x1="167.64" y1="20.32" x2="193.04" y2="20.32" width="0.1524" layer="91"/>
 <pinref part="C12" gate="G$1" pin="2"/>
-<wire x1="167.64" y1="33.02" x2="167.64" y2="20.32" width="0.1524" layer="91"/>
+<wire x1="167.64" y1="33.02" x2="167.64" y2="27.94" width="0.1524" layer="91"/>
 <junction x="167.64" y="20.32"/>
 <pinref part="J6" gate="G$1" pin="2"/>
+<wire x1="167.64" y1="27.94" x2="167.64" y2="20.32" width="0.1524" layer="91"/>
 <wire x1="144.78" y1="38.1" x2="144.78" y2="20.32" width="0.1524" layer="91"/>
 <junction x="144.78" y="20.32"/>
-</segment>
-<segment>
-<pinref part="U$6" gate="G$1" pin="S"/>
+<wire x1="167.64" y1="27.94" x2="175.26" y2="27.94" width="0.1524" layer="91"/>
+<junction x="167.64" y="27.94"/>
+<pinref part="U$3" gate="G$1" pin="GND"/>
+<wire x1="175.26" y1="27.94" x2="175.26" y2="45.72" width="0.1524" layer="91"/>
+</segment>
+<segment>
 <pinref part="U2" gate="G$1" pin="GND"/>
 <wire x1="220.98" y1="20.32" x2="208.28" y2="20.32" width="0.1524" layer="91"/>
@@
 <net name="N$20" class="0">
 <segment>
-<pinref part="U$4" gate="G$1" pin="VDD"/>
 <wire x1="165.1" y1="50.8" x2="167.64" y2="50.8" width="0.1524" layer="91"/>
 <pinref part="R15" gate="G$1" pin="2"/>
 <pinref part="C12" gate="G$1" pin="1"/>
-<wire x1="167.64" y1="50.8" x2="177.8" y2="50.8" width="0.1524" layer="91"/>
 <wire x1="167.64" y1="50.8" x2="167.64" y2="40.64" width="0.1524" layer="91"/>
+<pinref part="U$3" gate="G$1" pin="VCC"/>
+<wire x1="167.64" y1="50.8" x2="175.26" y2="50.8" width="0.1524" layer="91"/>
 <junction x="167.64" y="50.8"/>
 </segment>
 </net>
-<net name="N$21" class="0">
-<segment>
-<pinref part="U$5" gate="G$1" pin="D"/>
-<pinref part="U$6" gate="G$1" pin="D"/>
-<wire x1="198.12" y1="20.32" x2="203.2" y2="20.32" width="0.1524" layer="91"/>
-</segment>
-</net>
-<net name="N$22" class="0">
-<segment>
-<pinref part="U$5" gate="G$1" pin="G"/>
-<pinref part="U$4" gate="G$1" pin="DO"/>
-<wire x1="193.04" y1="30.48" x2="193.04" y2="35.56" width="0.1524" layer="91"/>
-</segment>
-</net>
-<net name="N$23" class="0">
-<segment>
-<pinref part="U$4" gate="G$1" pin="CO"/>
-<wire x1="200.66" y1="35.56" x2="200.66" y2="33.02" width="0.1524" layer="91"/>
-<wire x1="200.66" y1="33.02" x2="208.28" y2="33.02" width="0.1524" layer="91"/>
-<pinref part="U$6" gate="G$1" pin="G"/>
-<wire x1="208.28" y1="33.02" x2="208.28" y2="30.48" width="0.1524" layer="91"/>
-</segment>
-</net>
-<net name="N$24" class="0">
-<segment>
-<pinref part="U$4" gate="G$1" pin="VM"/>
-<wire x1="210.82" y1="50.8" x2="220.98" y2="50.8" width="0.1524" layer="91"/>
-<pinref part="R16" gate="G$1" pin="2"/>
-<wire x1="220.98" y1="50.8" x2="220.98" y2="40.64" width="0.1524" layer="91"/>
-</segment>
-</net>

Commit message: FS8205
Parts:
- added U$4: FS8205, FS8205:FS8205
Other:
- moved on the sheet: S1
Changed lines of the file:
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@@
 <part name="U1" library="SparkFun-IC-Power" deviceset="MCP73831" device=""/>
 <part name="U$3" library="FS312F-G" deviceset="FS312F-G" device=""/>
+<part name="U$4" library="FS8205" deviceset="FS8205" device=""/>
 </parts>
 <sheets>
@@
 <attribute name="VALUE" x="142.875" y="12.065" size="1.778" layer="96"/>
 </instance>
-<instance part="S1" gate="G$1" x="193.04" y="66.04" smashed="yes">
-<attribute name="NAME" x="185.417090625" y="71.121940625" size="1.270490625" layer="95"/>
-<attribute name="VALUE" x="185.411440625" y="60.954290625" size="1.27143125" layer="96"/>
+<instance part="S1" gate="G$1" x="193.04" y="104.14" smashed="yes">
+<attribute name="NAME" x="185.417090625" y="109.221940625" size="1.270490625" layer="95"/>
+<attribute name="VALUE" x="185.411440625" y="99.054290625" size="1.27143125" layer="96"/>
 </instance>
 <instance part="U2" gate="G$1" x="274.32" y="53.34" smashed="yes" rot="MR0">
@@
 </instance>
 <instance part="U$3" gate="G$1" x="185.42" y="53.34" smashed="yes" rot="R180"/>
+<instance part="U$4" gate="G$1" x="210.82" y="76.2" smashed="yes"/>
 </instances>
 <busses>
@@
 <junction x="246.38" y="50.8"/>
 <wire x1="241.3" y1="50.8" x2="246.38" y2="50.8" width="0.1524" layer="91"/>
-<wire x1="241.3" y1="50.8" x2="241.3" y2="66.04" width="0.1524" layer="91"/>
-<pinref part="S1" gate="G$1" pin="2"/>
-<wire x1="241.3" y1="66.04" x2="200.66" y2="66.04" width="0.1524" layer="91"/>
+<wire x1="241.3" y1="50.8" x2="241.3" y2="83.82" width="0.1524" layer="91"/>
 <wire x1="330.2" y1="83.82" x2="241.3" y2="83.82" width="0.1524" layer="91"/>
-<wire x1="241.3" y1="83.82" x2="241.3" y2="66.04" width="0.1524" layer="91"/>
-<junction x="241.3" y="66.04"/>
 <pinref part="C3" gate="G$1" pin="1"/>
 <wire x1="241.3" y1="50.8" x2="241.3" y2="38.1" width="0.1524" layer="91"/>
@@
 <wire x1="330.2" y1="48.26" x2="330.2" y2="38.1" width="0.1524" layer="91"/>
 <junction x="330.2" y="48.26"/>
+<pinref part="S1" gate="G$1" pin="2"/>
+<wire x1="200.66" y1="104.14" x2="241.3" y2="104.14" width="0.1524" layer="91"/>
+<wire x1="241.3" y1="104.14" x2="241.3" y2="83.82" width="0.1524" layer="91"/>
+<junction x="241.3" y="83.82"/>
 </segment>
 </net>
@@
 <pinref part="S1" gate="G$1" pin="1"/>
 <wire x1="134.62" y1="50.8" x2="144.78" y2="50.8" width="0.1524" layer="91"/>
-<wire x1="144.78" y1="50.8" x2="144.78" y2="68.58" width="0.1524" layer="91"/>
-<wire x1="144.78" y1="68.58" x2="185.42" y2="68.58" width="0.1524" layer="91"/>
+<wire x1="144.78" y1="50.8" x2="144.78" y2="106.68" width="0.1524" layer="91"/>
+<wire x1="144.78" y1="106.68" x2="185.42" y2="106.68" width="0.1524" layer="91"/>
 <pinref part="R15" gate="G$1" pin="1"/>
 <wire x1="144.78" y1="50.8" x2="154.94" y2="50.8" width="0.1524" layer="91"/>

Commit message: Update motherBoard.sch
Parts:
- R16: value 2.7K -> 1k
Connections:
- new net N$10: R16.2, U$3.CS
- new net N$17: U$3.OD, U$4.G1
- new net N$18: U$3.OC, U$4.G2
- net GND: now also U$4.S1, U$4.S2
Changed lines of the file:
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@@
 <part name="R14" library="SparkFun-Resistors" deviceset="RESISTOR" device="0603" value="470"/>
 <part name="R15" library="SparkFun-Resistors" deviceset="RESISTOR" device="0603" value="100"/>
-<part name="R16" library="SparkFun-Resistors" deviceset="RESISTOR" device="0603" value=" 2.7K"/>
+<part name="R16" library="SparkFun-Resistors" deviceset="RESISTOR" device="0603" value="1k"/>
 <part name="R17" library="SparkFun-Resistors" deviceset="RESISTOR" device="0603" value=" 1.5K"/>
 <part name="C9" library="SparkFun-Capacitors" deviceset="10UF" device="-0603-6.3V-20%" value="4.7uF"/>
@@
 <attribute name="VALUE" x="83.82" y="30.48" size="1.778" layer="96"/>
 </instance>
-<instance part="U$3" gate="G$1" x="185.42" y="53.34" smashed="yes" rot="R180"/>
-<instance part="U$4" gate="G$1" x="210.82" y="76.2" smashed="yes"/>
+<instance part="U$3" gate="G$1" x="195.58" y="60.96" smashed="yes" rot="R180"/>
+<instance part="U$4" gate="G$1" x="195.58" y="33.02" smashed="yes"/>
 </instances>
 <busses>
@@
 <wire x1="144.78" y1="20.32" x2="144.78" y2="17.78" width="0.1524" layer="91"/>
 <wire x1="144.78" y1="20.32" x2="167.64" y2="20.32" width="0.1524" layer="91"/>
-<wire x1="167.64" y1="20.32" x2="193.04" y2="20.32" width="0.1524" layer="91"/>
 <pinref part="C12" gate="G$1" pin="2"/>
-<wire x1="167.64" y1="33.02" x2="167.64" y2="27.94" width="0.1524" layer="91"/>
-<junction x="167.64" y="20.32"/>
 <pinref part="J6" gate="G$1" pin="2"/>
-<wire x1="167.64" y1="27.94" x2="167.64" y2="20.32" width="0.1524" layer="91"/>
+<wire x1="167.64" y1="33.02" x2="167.64" y2="25.4" width="0.1524" layer="91"/>
+<wire x1="167.64" y1="25.4" x2="167.64" y2="20.32" width="0.1524" layer="91"/>
 <wire x1="144.78" y1="38.1" x2="144.78" y2="20.32" width="0.1524" layer="91"/>
 <junction x="144.78" y="20.32"/>
-<wire x1="167.64" y1="27.94" x2="175.26" y2="27.94" width="0.1524" layer="91"/>
-<junction x="167.64" y="27.94"/>
 <pinref part="U$3" gate="G$1" pin="GND"/>
-<wire x1="175.26" y1="27.94" x2="175.26" y2="45.72" width="0.1524" layer="91"/>
+<wire x1="185.42" y1="53.34" x2="175.26" y2="53.34" width="0.1524" layer="91"/>
+<wire x1="175.26" y1="53.34" x2="175.26" y2="25.4" width="0.1524" layer="91"/>
+<wire x1="175.26" y1="25.4" x2="167.64" y2="25.4" width="0.1524" layer="91"/>
+<junction x="167.64" y="25.4"/>
+<wire x1="167.64" y1="20.32" x2="180.34" y2="20.32" width="0.1524" layer="91"/>
+<junction x="167.64" y="20.32"/>
+<wire x1="180.34" y1="20.32" x2="180.34" y2="38.1" width="0.1524" layer="91"/>
+<pinref part="U$4" gate="G$1" pin="S1"/>
+<wire x1="180.34" y1="38.1" x2="185.42" y2="38.1" width="0.1524" layer="91"/>
 </segment>
 <segment>
 <pinref part="U2" gate="G$1" pin="GND"/>
-<wire x1="220.98" y1="20.32" x2="208.28" y2="20.32" width="0.1524" layer="91"/>
 <wire x1="274.32" y1="50.8" x2="276.86" y2="50.8" width="0.1524" layer="91"/>
 <wire x1="276.86" y1="50.8" x2="276.86" y2="20.32" width="0.1524" layer="91"/>
@@
 <pinref part="SUPPLY15" gate="GND" pin="GND"/>
 <wire x1="289.56" y1="20.32" x2="289.56" y2="17.78" width="0.1524" layer="91" style="dashdot"/>
+<pinref part="U$4" gate="G$1" pin="S2"/>
+<wire x1="185.42" y1="27.94" x2="185.42" y2="20.32" width="0.1524" layer="91"/>
+<wire x1="185.42" y1="20.32" x2="220.98" y2="20.32" width="0.1524" layer="91"/>
 </segment>
 <segment>
@@
 <pinref part="C12" gate="G$1" pin="1"/>
 <wire x1="167.64" y1="50.8" x2="167.64" y2="40.64" width="0.1524" layer="91"/>
+<wire x1="167.64" y1="50.8" x2="167.64" y2="58.42" width="0.1524" layer="91"/>
+<junction x="167.64" y="50.8"/>
 <pinref part="U$3" gate="G$1" pin="VCC"/>
-<wire x1="167.64" y1="50.8" x2="175.26" y2="50.8" width="0.1524" layer="91"/>
-<junction x="167.64" y="50.8"/>
+<wire x1="167.64" y1="58.42" x2="185.42" y2="58.42" width="0.1524" layer="91"/>
 </segment>
 </net>
@@
 </segment>
 </net>
+<net name="N$10" class="0">
+<segment>
+<pinref part="U$3" gate="G$1" pin="CS"/>
+<pinref part="R16" gate="G$1" pin="2"/>
+<wire x1="210.82" y1="58.42" x2="220.98" y2="58.42" width="0.1524" layer="91"/>
+<wire x1="220.98" y1="58.42" x2="220.98" y2="40.64" width="0.1524" layer="91"/>
+</segment>
+</net>
+<net name="N$17" class="0">
+<segment>
+<pinref part="U$3" gate="G$1" pin="OD"/>
+<wire x1="210.82" y1="53.34" x2="210.82" y2="38.1" width="0.1524" layer="91"/>
+<pinref part="U$4" gate="G$1" pin="G1"/>
+<wire x1="210.82" y1="38.1" x2="208.28" y2="38.1" width="0.1524" layer="91"/>
+</segment>
+</net>
+<net name="N$18" class="0">
+<segment>
+<pinref part="U$3" gate="G$1" pin="OC"/>
+<wire x1="210.82" y1="63.5" x2="215.9" y2="63.5" width="0.1524" layer="91"/>
+<pinref part="U$4" gate="G$1" pin="G2"/>
+<wire x1="215.9" y1="63.5" x2="215.9" y2="27.94" width="0.1524" layer="91"/>
+<wire x1="215.9" y1="27.94" x2="208.28" y2="27.94" width="0.1524" layer="91"/>
+</segment>
+</net>
