File: eagle/projects/smartBobber Mother Board/motherBoard/motherBoard.sch (EAGLE design)
At the start: 58 parts, among them J1 10118193-0001LF, J6 1053131202, Q1 2A/20V/150mΩ, Q2 MMBT3904, U1 MCP73831, U2 MT3608, U3 LTC3531ES6-3_3, Y1 ECS-40-S-4X

Commit message: Update motherBoard.sch
Parts:
- removed D3: LTST-C191KGKT, LTST-C191KGKT:LTST-C191KGKT
- added GLED: (no value), led:LED5MM
Connections:
- net N$11: now also GLED.A; no longer D3.A2
- net N$2: now also GLED.C; no longer D3.K2
Other:
- moved on the sheet: S1
Changed lines of the file:
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@@
 <part name="SUPPLY1" library="supply2" library_urn="urn:adsk.eagle:library:372" deviceset="GND" device="" value="GND1"/>
 <part name="SUPPLY2" library="supply2" library_urn="urn:adsk.eagle:library:372" deviceset="GND" device="" value="GND1"/>
-<part name="D3" library="LTST-C191KGKT" deviceset="LTST-C191KGKT" device=""/>
 <part name="SUPPLY3" library="supply2" library_urn="urn:adsk.eagle:library:372" deviceset="GND" device="" value="GND1"/>
 <part name="SUPPLY4" library="supply2" library_urn="urn:adsk.eagle:library:372" deviceset="GND" device="" value="GND1"/>
@@
 <part name="U$3" library="FS312F-G" deviceset="FS312F-G" device=""/>
 <part name="U$4" library="FS8205" deviceset="FS8205" device=""/>
+<part name="GLED" library="led" library_urn="urn:adsk.eagle:library:259" deviceset="LED" device="5MM" package3d_urn="urn:adsk.eagle:package:15799/2"/>
 </parts>
 <sheets>
@@
 <attribute name="VALUE" x="43.815" y="12.065" size="1.778" layer="96"/>
 </instance>
-<instance part="D3" gate="G$1" x="63.5" y="33.02" smashed="yes">
-<attribute name="NAME" x="60.95498125" y="27.94501875" size="1.78151875" layer="95" rot="R90"/>
-</instance>
 <instance part="SUPPLY3" gate="GND" x="121.92" y="15.24" smashed="yes">
 <attribute name="VALUE" x="120.015" y="12.065" size="1.778" layer="96"/>
@@
 <attribute name="VALUE" x="142.875" y="12.065" size="1.778" layer="96"/>
 </instance>
-<instance part="S1" gate="G$1" x="193.04" y="104.14" smashed="yes">
-<attribute name="NAME" x="185.417090625" y="109.221940625" size="1.270490625" layer="95"/>
-<attribute name="VALUE" x="185.411440625" y="99.054290625" size="1.27143125" layer="96"/>
+<instance part="S1" gate="G$1" x="195.58" y="78.74" smashed="yes">
+<attribute name="NAME" x="187.957090625" y="83.821940625" size="1.270490625" layer="95"/>
+<attribute name="VALUE" x="187.951440625" y="73.654290625" size="1.27143125" layer="96"/>
 </instance>
 <instance part="U2" gate="G$1" x="274.32" y="53.34" smashed="yes" rot="MR0">
@@
 <instance part="U$3" gate="G$1" x="195.58" y="60.96" smashed="yes" rot="R180"/>
 <instance part="U$4" gate="G$1" x="195.58" y="33.02" smashed="yes"/>
+<instance part="GLED" gate="G$1" x="63.5" y="35.56" smashed="yes">
+<attribute name="NAME" x="67.056" y="30.988" size="1.778" layer="95" rot="R90"/>
+<attribute name="VALUE" x="69.215" y="30.988" size="1.778" layer="96" rot="R90"/>
+</instance>
 </instances>
 <busses>
@@
 <pinref part="C12" gate="G$1" pin="2"/>
 <pinref part="J6" gate="G$1" pin="2"/>
-<wire x1="167.64" y1="33.02" x2="167.64" y2="25.4" width="0.1524" layer="91"/>
-<wire x1="167.64" y1="25.4" x2="167.64" y2="20.32" width="0.1524" layer="91"/>
+<wire x1="167.64" y1="33.02" x2="167.64" y2="20.32" width="0.1524" layer="91"/>
 <wire x1="144.78" y1="38.1" x2="144.78" y2="20.32" width="0.1524" layer="91"/>
 <junction x="144.78" y="20.32"/>
-<pinref part="U$3" gate="G$1" pin="GND"/>
-<wire x1="185.42" y1="53.34" x2="175.26" y2="53.34" width="0.1524" layer="91"/>
-<wire x1="175.26" y1="53.34" x2="175.26" y2="25.4" width="0.1524" layer="91"/>
-<wire x1="175.26" y1="25.4" x2="167.64" y2="25.4" width="0.1524" layer="91"/>
-<junction x="167.64" y="25.4"/>
-<wire x1="167.64" y1="20.32" x2="180.34" y2="20.32" width="0.1524" layer="91"/>
+<wire x1="167.64" y1="20.32" x2="175.26" y2="20.32" width="0.1524" layer="91"/>
 <junction x="167.64" y="20.32"/>
+<wire x1="175.26" y1="20.32" x2="180.34" y2="20.32" width="0.1524" layer="91"/>
 <wire x1="180.34" y1="20.32" x2="180.34" y2="38.1" width="0.1524" layer="91"/>
 <pinref part="U$4" gate="G$1" pin="S1"/>
 <wire x1="180.34" y1="38.1" x2="185.42" y2="38.1" width="0.1524" layer="91"/>
+<pinref part="U$3" gate="G$1" pin="GND"/>
+<wire x1="185.42" y1="53.34" x2="175.26" y2="53.34" width="0.1524" layer="91"/>
+<wire x1="175.26" y1="53.34" x2="175.26" y2="20.32" width="0.1524" layer="91"/>
+<junction x="175.26" y="20.32"/>
 </segment>
 <segment>
@@
 <pinref part="C9" gate="G$1" pin="1"/>
 <wire x1="45.72" y1="40.64" x2="45.72" y2="35.56" width="0.1524" layer="91"/>
-<pinref part="D3" gate="G$1" pin="A2"/>
-<wire x1="45.72" y1="40.64" x2="63.5" y2="40.64" width="0.1524" layer="91"/>
-<wire x1="63.5" y1="40.64" x2="63.5" y2="38.1" width="0.1524" layer="91"/>
 <junction x="45.72" y="40.64"/>
 <pinref part="U1" gate="G$1" pin="VIN"/>
+<wire x1="45.72" y1="40.64" x2="63.5" y2="40.64" width="0.1524" layer="91"/>
+<pinref part="GLED" gate="G$1" pin="A"/>
 <wire x1="63.5" y1="40.64" x2="81.28" y2="40.64" width="0.1524" layer="91"/>
+<wire x1="63.5" y1="40.64" x2="63.5" y2="38.1" width="0.1524" layer="91"/>
 <junction x="63.5" y="40.64"/>
 </segment>
@@
 <junction x="330.2" y="48.26"/>
 <pinref part="S1" gate="G$1" pin="2"/>
-<wire x1="200.66" y1="104.14" x2="241.3" y2="104.14" width="0.1524" layer="91"/>
-<wire x1="241.3" y1="104.14" x2="241.3" y2="83.82" width="0.1524" layer="91"/>
+<wire x1="203.2" y1="78.74" x2="233.68" y2="78.74" width="0.1524" layer="91"/>
+<wire x1="233.68" y1="78.74" x2="233.68" y2="83.82" width="0.1524" layer="91"/>
+<wire x1="233.68" y1="83.82" x2="241.3" y2="83.82" width="0.1524" layer="91"/>
 <junction x="241.3" y="83.82"/>
 </segment>
@@
 </segment>
 </net>
-<net name="N$2" class="0">
-<segment>
-<pinref part="D3" gate="G$1" pin="K2"/>
-<pinref part="R14" gate="G$1" pin="2"/>
-<wire x1="63.5" y1="30.48" x2="63.5" y2="27.94" width="0.1524" layer="91"/>
-</segment>
-</net>
 <net name="N$7" class="0">
 <segment>
@@
 <pinref part="S1" gate="G$1" pin="1"/>
 <wire x1="134.62" y1="50.8" x2="144.78" y2="50.8" width="0.1524" layer="91"/>
-<wire x1="144.78" y1="50.8" x2="144.78" y2="106.68" width="0.1524" layer="91"/>
-<wire x1="144.78" y1="106.68" x2="185.42" y2="106.68" width="0.1524" layer="91"/>
+<wire x1="144.78" y1="50.8" x2="144.78" y2="81.28" width="0.1524" layer="91"/>
+<wire x1="144.78" y1="81.28" x2="187.96" y2="81.28" width="0.1524" layer="91"/>
 <pinref part="R15" gate="G$1" pin="1"/>
 <wire x1="144.78" y1="50.8" x2="154.94" y2="50.8" width="0.1524" layer="91"/>
@@
 </segment>
 </net>
+<net name="N$2" class="0">
+<segment>
+<pinref part="GLED" gate="G$1" pin="C"/>
+<pinref part="R14" gate="G$1" pin="2"/>
+<wire x1="63.5" y1="30.48" x2="63.5" y2="27.94" width="0.1524" layer="91"/>
+</segment>
+</net>

Commit message: Update motherBoard.sch
Parts:
- added U$5, U$6: SCMR18G604SRBA0, SCMRCapacitor:SCMR18G604SRBA0
Connections:
- removed net GND: C1.2, C11.2, C12.2, C13.2, C2.2, C3.2, C4.2, C5.2, C6.2, C7.2, C9.2, D2.A, J1.GND, J2.5, J3.1, J4.3, J5.1, J6.2, Q2.E, R10.1, R13.1, R16.1, R17.1, R3.2, R5.1, R7.1, R8.1, S2.1, SOLENOID.2, U$1.VSS, U$1.VSS_2, U$3.GND, U$4.S1, U$4.S2, U1.VSS, U2.GND, U3.GND/PGND
- new net N$19: U$5.-, U$6.+
- new net _12V: C1.2, C11.2, C12.2, C13.2, C2.2, C3.2, C4.2, C5.2, C6.2, C7.2, C9.2, D2.A, J1.GND, J2.5, J3.1, J4.3, J5.1, J6.2, Q2.E, R10.1, R13.1, R16.1, R17.1, R3.2, R5.1, R7.1, R8.1, S2.1, SOLENOID.2, U$1.VSS, U$1.VSS_2, U$3.GND, U$4.S1, U$4.S2, U$6.-, U1.VSS, U2.GND, U3.GND/PGND
- net 12V: now also U$5.+
Changed lines of the file:
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@@
 <part name="U$4" library="FS8205" deviceset="FS8205" device=""/>
 <part name="GLED" library="led" library_urn="urn:adsk.eagle:library:259" deviceset="LED" device="5MM" package3d_urn="urn:adsk.eagle:package:15799/2"/>
+<part name="U$5" library="SCMRCapacitor" deviceset="SCMR18G604SRBA0" device=""/>
+<part name="U$6" library="SCMRCapacitor" deviceset="SCMR18G604SRBA0" device=""/>
 </parts>
 <sheets>
@@
 </segment>
 </net>
-<net name="GND" class="0">
+<net name="_12V" class="0">
 <segment>
 <pinref part="D2" gate="G$1" pin="A"/>
@@
 <attribute name="VALUE" x="69.215" y="30.988" size="1.778" layer="96" rot="R90"/>
 </instance>
+<instance part="U$5" gate="G$1" x="294.64" y="88.9" smashed="yes"/>
+<instance part="U$6" gate="G$1" x="320.04" y="88.9" smashed="yes"/>
 </instances>
 <busses>
 </busses>
 <nets>
-<net name="GND" class="0">
+<net name="_12V" class="0">
 <segment>
 <wire x1="20.32" y1="30.48" x2="33.02" y2="30.48" width="0.1524" layer="91"/>
@@
 <wire x1="416.56" y1="48.26" x2="416.56" y2="20.32" width="0.1524" layer="91"/>
 <wire x1="416.56" y1="20.32" x2="330.2" y2="20.32" width="0.1524" layer="91"/>
-<wire x1="330.2" y1="20.32" x2="304.8" y2="20.32" width="0.1524" layer="91"/>
+<wire x1="330.2" y1="20.32" x2="314.96" y2="20.32" width="0.1524" layer="91"/>
+<wire x1="314.96" y1="20.32" x2="304.8" y2="20.32" width="0.1524" layer="91"/>
 <wire x1="426.72" y1="20.32" x2="416.56" y2="20.32" width="0.1524" layer="91"/>
 <junction x="416.56" y="20.32"/>
@@
 <wire x1="185.42" y1="27.94" x2="185.42" y2="20.32" width="0.1524" layer="91"/>
 <wire x1="185.42" y1="20.32" x2="220.98" y2="20.32" width="0.1524" layer="91"/>
+<pinref part="U$6" gate="G$1" pin="-"/>
+<wire x1="330.2" y1="88.9" x2="335.28" y2="88.9" width="0.1524" layer="91"/>
+<wire x1="335.28" y1="88.9" x2="335.28" y2="73.66" width="0.1524" layer="91"/>
+<wire x1="335.28" y1="73.66" x2="314.96" y2="73.66" width="0.1524" layer="91"/>
+<wire x1="314.96" y1="73.66" x2="314.96" y2="20.32" width="0.1524" layer="91"/>
+<junction x="314.96" y="20.32"/>
+<wire x1="335.28" y1="88.9" x2="342.9" y2="88.9" width="0.1524" layer="91"/>
+<junction x="335.28" y="88.9"/>
+<label x="342.9" y="88.9" size="1.778" layer="95"/>
 </segment>
 <segment>
@@
 <net name="12V" class="0">
 <segment>
+<wire x1="304.8" y1="81.28" x2="279.4" y2="81.28" width="0.1524" layer="91"/>
+<wire x1="279.4" y1="81.28" x2="279.4" y2="88.9" width="0.1524" layer="91"/>
+<pinref part="U$5" gate="G$1" pin="+"/>
+<wire x1="279.4" y1="88.9" x2="284.48" y2="88.9" width="0.1524" layer="91"/>
+<pinref part="R12" gate="G$1" pin="E"/>
 <pinref part="D4" gate="A" pin="C"/>
 <wire x1="284.48" y1="73.66" x2="289.56" y2="73.66" width="0.1524" layer="91"/>
+<wire x1="289.56" y1="73.66" x2="289.56" y2="63.5" width="0.1524" layer="91"/>
 <wire x1="289.56" y1="73.66" x2="304.8" y2="73.66" width="0.1524" layer="91"/>
-<pinref part="R12" gate="G$1" pin="E"/>
-<wire x1="289.56" y1="73.66" x2="289.56" y2="63.5" width="0.1524" layer="91"/>
 <junction x="289.56" y="73.66"/>
 <pinref part="C5" gate="G$1" pin="1"/>
 <wire x1="304.8" y1="73.66" x2="304.8" y2="50.8" width="0.1524" layer="91"/>
-<wire x1="304.8" y1="73.66" x2="312.42" y2="73.66" width="0.1524" layer="91"/>
+<wire x1="304.8" y1="73.66" x2="304.8" y2="81.28" width="0.1524" layer="91"/>
 <junction x="304.8" y="73.66"/>
-<label x="312.42" y="73.66" size="1.778" layer="95"/>
 </segment>
 </net>
@@
 </segment>
 </net>
+<net name="N$19" class="0">
+<segment>
+<pinref part="U$5" gate="G$1" pin="-"/>
+<pinref part="U$6" gate="G$1" pin="+"/>
+<wire x1="304.8" y1="88.9" x2="309.88" y2="88.9" width="0.1524" layer="91"/>
+</segment>
+</net>

Commit message: WNER50FET Resistor
Connections:
- new net N$21: C3.1, U$2.1, U2.EN, U2.IN
- net N$16: no longer C3.1, U$2.1, U2.EN, U2.IN
Changed lines of the file:
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@@
 <junction x="337.82" y="48.26"/>
 <wire x1="330.2" y1="48.26" x2="330.2" y2="83.82" width="0.1524" layer="91"/>
-<pinref part="U2" gate="G$1" pin="IN"/>
-<wire x1="248.92" y1="50.8" x2="246.38" y2="50.8" width="0.1524" layer="91"/>
-<pinref part="U$2" gate="G$1" pin="1"/>
-<wire x1="246.38" y1="50.8" x2="246.38" y2="63.5" width="0.1524" layer="91"/>
-<wire x1="246.38" y1="63.5" x2="254" y2="63.5" width="0.1524" layer="91"/>
-<pinref part="U2" gate="G$1" pin="EN"/>
-<wire x1="248.92" y1="48.26" x2="246.38" y2="48.26" width="0.1524" layer="91"/>
-<wire x1="246.38" y1="48.26" x2="246.38" y2="50.8" width="0.1524" layer="91"/>
-<junction x="246.38" y="50.8"/>
-<wire x1="241.3" y1="50.8" x2="246.38" y2="50.8" width="0.1524" layer="91"/>
-<wire x1="241.3" y1="50.8" x2="241.3" y2="83.82" width="0.1524" layer="91"/>
-<wire x1="330.2" y1="83.82" x2="241.3" y2="83.82" width="0.1524" layer="91"/>
-<pinref part="C3" gate="G$1" pin="1"/>
-<wire x1="241.3" y1="50.8" x2="241.3" y2="38.1" width="0.1524" layer="91"/>
-<junction x="241.3" y="50.8"/>
+<wire x1="330.2" y1="83.82" x2="233.68" y2="83.82" width="0.1524" layer="91"/>
 <pinref part="C13" gate="G$1" pin="1"/>
 <wire x1="330.2" y1="48.26" x2="330.2" y2="38.1" width="0.1524" layer="91"/>
@@
 <wire x1="203.2" y1="78.74" x2="233.68" y2="78.74" width="0.1524" layer="91"/>
 <wire x1="233.68" y1="78.74" x2="233.68" y2="83.82" width="0.1524" layer="91"/>
-<wire x1="233.68" y1="83.82" x2="241.3" y2="83.82" width="0.1524" layer="91"/>
-<junction x="241.3" y="83.82"/>
 </segment>
 </net>
@@
 </segment>
 </net>
+<net name="N$21" class="0">
+<segment>
+<pinref part="C3" gate="G$1" pin="1"/>
+<pinref part="U$2" gate="G$1" pin="1"/>
+<wire x1="246.38" y1="63.5" x2="254" y2="63.5" width="0.1524" layer="91"/>
+<pinref part="U2" gate="G$1" pin="IN"/>
+<wire x1="248.92" y1="50.8" x2="246.38" y2="50.8" width="0.1524" layer="91"/>
+<wire x1="246.38" y1="50.8" x2="246.38" y2="63.5" width="0.1524" layer="91"/>
+<pinref part="U2" gate="G$1" pin="EN"/>
+<wire x1="248.92" y1="48.26" x2="246.38" y2="48.26" width="0.1524" layer="91"/>
+<wire x1="246.38" y1="48.26" x2="246.38" y2="50.8" width="0.1524" layer="91"/>
+<junction x="246.38" y="50.8"/>
+<wire x1="241.3" y1="50.8" x2="246.38" y2="50.8" width="0.1524" layer="91"/>
+<wire x1="241.3" y1="50.8" x2="241.3" y2="38.1" width="0.1524" layer="91"/>
+</segment>
+</net>
