File: eagle/projects/smartBobber Mother Board/motherBoard/motherBoard.sch (EAGLE design)
At the start: 61 parts, among them J1 10118193-0001LF, J6 1053131202, Q1 2A/20V/150mΩ, Q2 MMBT3904, U1 MCP73831, U2 MT3608, U3 LTC3531ES6-3_3, Y1 ECS-40-S-4X

Commit message: I'm going through changes
Parts:
- J6: value 1053131202 -> 640456-2; device 1053131202:1053131202 -> 640456-2:640456-2
Connections:
- net N$8: now also J6.P1; no longer J6.1
- net _12V: now also J6.P2; no longer J6.2
Other:
- moved on the sheet: J6
Changed lines of the file:
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@@
 <part name="SUPPLY14" library="supply2" library_urn="urn:adsk.eagle:library:372" deviceset="GND" device=""/>
 <part name="SUPPLY15" library="supply2" library_urn="urn:adsk.eagle:library:372" deviceset="GND" device=""/>
-<part name="J6" library="1053131202" deviceset="1053131202" device=""/>
 <part name="U$1" library="PIC16LF876A-I_SS" deviceset="PIC16LF876A-I/SS" device=""/>
 <part name="Y1" library="ECS-40-S-4X" deviceset="ECS-40-S-4X" device=""/>
@@
 <part name="U$6" library="SCMRCapacitor" deviceset="SCMR18G604SRBA0" device=""/>
 <part name="U$7" library="WNER50FET" deviceset="WNER50FET" device=""/>
+<part name="J6" library="640456-2" deviceset="640456-2" device=""/>
 </parts>
 <sheets>
@@
 <attribute name="VALUE" x="287.655" y="12.065" size="1.778" layer="96"/>
 </instance>
-<instance part="J6" gate="G$1" x="149.86" y="40.64" smashed="yes">
-<attribute name="NAME" x="147.312" y="43.6976" size="1.783609375" layer="95"/>
-<attribute name="VALUE" x="147.313540625" y="33.000609375" size="1.78251875" layer="96"/>
-</instance>
 <instance part="U1" gate="G$1" x="91.44" y="38.1" smashed="yes">
 <attribute name="NAME" x="83.82" y="43.688" size="1.778" layer="95"/>
@@
 <instance part="U$6" gate="G$1" x="320.04" y="88.9" smashed="yes"/>
 <instance part="U$7" gate="G$1" x="241.3" y="66.04" smashed="yes" rot="R90"/>
+<instance part="J6" gate="G$1" x="149.86" y="35.56" smashed="yes">
+<attribute name="NAME" x="144.77536875" y="41.661559375" size="1.271159375" layer="95"/>
+<attribute name="VALUE" x="144.772140625" y="27.928209375" size="1.271959375" layer="96"/>
+</instance>
 </instances>
 <busses>
@@
 <wire x1="144.78" y1="20.32" x2="167.64" y2="20.32" width="0.1524" layer="91"/>
 <pinref part="C12" gate="G$1" pin="2"/>
-<pinref part="J6" gate="G$1" pin="2"/>
 <wire x1="167.64" y1="33.02" x2="167.64" y2="20.32" width="0.1524" layer="91"/>
-<wire x1="144.78" y1="38.1" x2="144.78" y2="20.32" width="0.1524" layer="91"/>
-<junction x="144.78" y="20.32"/>
 <wire x1="167.64" y1="20.32" x2="175.26" y2="20.32" width="0.1524" layer="91"/>
 <junction x="167.64" y="20.32"/>
@@
 <wire x1="175.26" y1="53.34" x2="175.26" y2="20.32" width="0.1524" layer="91"/>
 <junction x="175.26" y="20.32"/>
+<pinref part="J6" gate="G$1" pin="P2"/>
+<wire x1="142.24" y1="33.02" x2="142.24" y2="20.32" width="0.1524" layer="91"/>
+<wire x1="142.24" y1="20.32" x2="144.78" y2="20.32" width="0.1524" layer="91"/>
+<junction x="144.78" y="20.32"/>
 </segment>
 <segment>
@@
 <wire x1="134.62" y1="50.8" x2="134.62" y2="40.64" width="0.1524" layer="91"/>
 <junction x="144.78" y="50.8"/>
-<pinref part="J6" gate="G$1" pin="1"/>
-<wire x1="144.78" y1="50.8" x2="144.78" y2="40.64" width="0.1524" layer="91"/>
 <wire x1="121.92" y1="40.64" x2="134.62" y2="40.64" width="0.1524" layer="91"/>
 <junction x="121.92" y="40.64"/>
-</segment>
-</net>
+<wire x1="144.78" y1="50.8" x2="144.78" y2="43.18" width="0.1524" layer="91"/>
+<wire x1="144.78" y1="43.18" x2="142.24" y2="43.18" width="0.1524" layer="91"/>
+<pinref part="J6" gate="G$1" pin="P1"/>
+<wire x1="142.24" y1="43.18" x2="142.24" y2="38.1" width="0.1524" layer="91"/>
+</segment>
+</net>

Commit message: Update motherBoard.sch
Parts:
- removed J2: (no value), SparkFun-Connectors:CONN_05JST-VERT
- removed J3: (no value), SparkFun-Connectors:CONN_03POLAR
- removed J4: (no value), SparkFun-Connectors:CONN_06SILK_FEMALE_PTH
- removed J5, SOLENOID: (no value), SparkFun-Connectors:CONN_02
- added J10: 640456-5, 640456-5:640456-5
- added J11, J8: 640456-2, 640456-2:640456-2
- added J7: (no value), SparkFun-Connectors:CONN_06SILK_FEMALE_PTH
- added J9: 640456-3, 640456-3:640456-3
- renumbered BLED1 to BLED4, BLED2 to BLED5, BLED3 to BLED6, C1 to C8, C2 to C10, C4 to C14, C6 to C15, D1 to D5, D2 to D3, Q1 to Q3, Q2 to Q4, R1 to R25, R10 to R27, R11 to R28, R2 to R18, R3 to R19, R4 to R20, R5 to R21, R6 to R22, R7 to R23, R8 to R24, R9 to R26, RLED1 to RLED4, RLED2 to RLED5, RLED3 to RLED6, S2 to S3, U$1 to U$8, Y1 to Y2
Connections:
- new net GND: C10.2, C14.2, C15.2, C8.2, D3.A, J10.1, J11.P1, J7.3, J8.P2, J9.1, Q4.E, R19.2, R21.1, R23.1, R24.1, R27.1, S3.1, U$8.VSS, U$8.VSS_2
- net 3.3V: now also J10.2, J7.2; no longer J2.4, J4.2
- net BLUETOOTH_ON/OFF: now also J10.5; no longer J2.1
- net DRIVER: now also J8.P1; no longer SOLENOID.1
- net LVP: now also J7.6; no longer J4.6
- net MCLR: now also J7.1; no longer J4.1
- net PGC: now also J7.5; no longer J4.5
- net PGD: now also J7.4; no longer J4.4
- net RX: now also J10.3; no longer J2.3
- net TEMP_DQ: now also J9.2; no longer J3.2
- net TX: now also J10.4; no longer J2.2
- net VCC: now also J11.P2, J9.3; no longer J3.3, J5.2
- net _12V: no longer C10.2, C14.2, C15.2, C8.2, D3.A, J2.5, J3.1, J4.3, J5.1, Q4.E, R19.2, R21.1, R23.1, R24.1, R27.1, S3.1, SOLENOID.2, U$8.VSS, U$8.VSS_2

Commit message: Board make
Parts:
- renumbered J6 to BATT
Changed lines of the file:
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@@
 <part name="U$6" library="SCMRCapacitor" deviceset="SCMR18G604SRBA0" device=""/>
 <part name="U$7" library="WNER50FET" deviceset="WNER50FET" device=""/>
-<part name="J6" library="640456-2" deviceset="640456-2" device=""/>
+<part name="BATT" library="640456-2" deviceset="640456-2" device=""/>
 <part name="U$8" library="PIC16LF876A-I_SS" deviceset="PIC16LF876A-I/SS" device=""/>
 <part name="Y2" library="ECS-40-S-4X" deviceset="ECS-40-S-4X" device=""/>
@@
 <instance part="U$6" gate="G$1" x="320.04" y="88.9" smashed="yes"/>
 <instance part="U$7" gate="G$1" x="241.3" y="66.04" smashed="yes" rot="R90"/>
-<instance part="J6" gate="G$1" x="149.86" y="35.56" smashed="yes">
+<instance part="BATT" gate="G$1" x="149.86" y="35.56" smashed="yes">
 <attribute name="NAME" x="144.77536875" y="41.661559375" size="1.271159375" layer="95"/>
 <attribute name="VALUE" x="144.772140625" y="27.928209375" size="1.271959375" layer="96"/>
@@
 <wire x1="175.26" y1="53.34" x2="175.26" y2="20.32" width="0.1524" layer="91"/>
 <junction x="175.26" y="20.32"/>
-<pinref part="J6" gate="G$1" pin="P2"/>
+<pinref part="BATT" gate="G$1" pin="P2"/>
 <wire x1="142.24" y1="33.02" x2="142.24" y2="20.32" width="0.1524" layer="91"/>
 <wire x1="142.24" y1="20.32" x2="144.78" y2="20.32" width="0.1524" layer="91"/>
@@
 <wire x1="144.78" y1="50.8" x2="144.78" y2="43.18" width="0.1524" layer="91"/>
 <wire x1="144.78" y1="43.18" x2="142.24" y2="43.18" width="0.1524" layer="91"/>
-<pinref part="J6" gate="G$1" pin="P1"/>
+<pinref part="BATT" gate="G$1" pin="P1"/>
 <wire x1="142.24" y1="43.18" x2="142.24" y2="38.1" width="0.1524" layer="91"/>
 </segment>

Commit message: Update motherBoard.sch
Parts:
- removed U2: MT3608, MT3608:MT3608
- renumbered BATT to J6
Connections:
- net N$12: no longer U2.SW
- net N$13: no longer U2.FB
- net N$21: no longer U2.EN, U2.IN
- net _12V: no longer U2.GND
Changed lines of the file:
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@@
 <part name="SUPPLY5" library="supply2" library_urn="urn:adsk.eagle:library:372" deviceset="GND" device="" value="GND1"/>
 <part name="S1" library="JS102011SAQN" deviceset="JS102011SAQN" device=""/>
-<part name="U2" library="MT3608" deviceset="MT3608" device=""/>
 <part name="D4" library="SS34" deviceset="SS34" device=""/>
 <part name="J1" library="10118193-0001LF" deviceset="10118193-0001LF" device=""/>
@@
 <part name="U$6" library="SCMRCapacitor" deviceset="SCMR18G604SRBA0" device=""/>
 <part name="U$7" library="WNER50FET" deviceset="WNER50FET" device=""/>
-<part name="BATT" library="640456-2" deviceset="640456-2" device=""/>
+<part name="J6" library="640456-2" deviceset="640456-2" device=""/>
 <part name="U$8" library="PIC16LF876A-I_SS" deviceset="PIC16LF876A-I/SS" device=""/>
 <part name="Y2" library="ECS-40-S-4X" deviceset="ECS-40-S-4X" device=""/>
@@
 <attribute name="VALUE" x="187.951440625" y="73.654290625" size="1.27143125" layer="96"/>
 </instance>
-<instance part="U2" gate="G$1" x="274.32" y="53.34" smashed="yes" rot="MR0">
-<attribute name="NAME" x="252.73" y="60.96" size="1.778" layer="95" rot="MR0" align="center-left"/>
-<attribute name="VALUE" x="252.73" y="58.42" size="1.778" layer="96" rot="MR0" align="center-left"/>
-</instance>
 <instance part="D4" gate="A" x="281.94" y="73.66" smashed="yes">
 <attribute name="NAME" x="279.654" y="75.565" size="1.778" layer="95"/>
@@
 <instance part="U$6" gate="G$1" x="320.04" y="88.9" smashed="yes"/>
 <instance part="U$7" gate="G$1" x="241.3" y="66.04" smashed="yes" rot="R90"/>
-<instance part="BATT" gate="G$1" x="149.86" y="35.56" smashed="yes">
+<instance part="J6" gate="G$1" x="149.86" y="35.56" smashed="yes">
 <attribute name="NAME" x="144.77536875" y="41.661559375" size="1.271159375" layer="95"/>
 <attribute name="VALUE" x="144.772140625" y="27.928209375" size="1.271959375" layer="96"/>
@@
 <wire x1="175.26" y1="53.34" x2="175.26" y2="20.32" width="0.1524" layer="91"/>
 <junction x="175.26" y="20.32"/>
-<pinref part="BATT" gate="G$1" pin="P2"/>
+<pinref part="J6" gate="G$1" pin="P2"/>
 <wire x1="142.24" y1="33.02" x2="142.24" y2="20.32" width="0.1524" layer="91"/>
 <wire x1="142.24" y1="20.32" x2="144.78" y2="20.32" width="0.1524" layer="91"/>
@@
 </segment>
 <segment>
-<pinref part="U2" gate="G$1" pin="GND"/>
 <wire x1="274.32" y1="50.8" x2="276.86" y2="50.8" width="0.1524" layer="91"/>
 <wire x1="276.86" y1="50.8" x2="276.86" y2="20.32" width="0.1524" layer="91"/>
@@
 <wire x1="269.24" y1="63.5" x2="276.86" y2="63.5" width="0.1524" layer="91"/>
 <wire x1="276.86" y1="63.5" x2="276.86" y2="53.34" width="0.1524" layer="91"/>
-<pinref part="U2" gate="G$1" pin="SW"/>
 <wire x1="276.86" y1="53.34" x2="274.32" y2="53.34" width="0.1524" layer="91"/>
 <pinref part="D4" gate="A" pin="A"/>
@@
 <net name="N$13" class="0">
 <segment>
-<pinref part="U2" gate="G$1" pin="FB"/>
 <wire x1="274.32" y1="48.26" x2="289.56" y2="48.26" width="0.1524" layer="91"/>
 <wire x1="289.56" y1="48.26" x2="289.56" y2="50.8" width="0.1524" layer="91"/>
@@
 <wire x1="144.78" y1="50.8" x2="144.78" y2="43.18" width="0.1524" layer="91"/>
 <wire x1="144.78" y1="43.18" x2="142.24" y2="43.18" width="0.1524" layer="91"/>
-<pinref part="BATT" gate="G$1" pin="P1"/>
+<pinref part="J6" gate="G$1" pin="P1"/>
 <wire x1="142.24" y1="43.18" x2="142.24" y2="38.1" width="0.1524" layer="91"/>
 </segment>
@@
 <pinref part="U$2" gate="G$1" pin="1"/>
 <wire x1="246.38" y1="63.5" x2="254" y2="63.5" width="0.1524" layer="91"/>
-<pinref part="U2" gate="G$1" pin="IN"/>
 <wire x1="248.92" y1="50.8" x2="246.38" y2="50.8" width="0.1524" layer="91"/>
 <wire x1="246.38" y1="50.8" x2="246.38" y2="63.5" width="0.1524" layer="91"/>
-<pinref part="U2" gate="G$1" pin="EN"/>
 <wire x1="248.92" y1="48.26" x2="246.38" y2="48.26" width="0.1524" layer="91"/>
 <wire x1="246.38" y1="48.26" x2="246.38" y2="50.8" width="0.1524" layer="91"/>

Commit message: Update motherBoard.sch
Parts:
- added U2: MT3608, MT3608:MT3608
Connections:
- net N$12: now also U2.SW
- net N$13: now also U2.FB
- net N$21: now also U2.EN, U2.IN
- net _12V: now also U2.GND
Changed lines of the file:
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@@
 <part name="D5" library="1N4002" deviceset="1N4002" device=""/>
 <part name="J11" library="640456-2" deviceset="640456-2" device=""/>
+<part name="U2" library="MT3608" deviceset="MT3608" device=""/>
 </parts>
 <sheets>
@@
 <attribute name="VALUE" x="144.772140625" y="27.928209375" size="1.271959375" layer="96"/>
 </instance>
+<instance part="U2" gate="G$1" x="274.32" y="53.34" smashed="yes" rot="MR0">
+<attribute name="NAME" x="252.73" y="60.96" size="1.778" layer="95" rot="MR0" align="center-left"/>
+<attribute name="VALUE" x="252.73" y="58.42" size="1.778" layer="96" rot="MR0" align="center-left"/>
+</instance>
 </instances>
 <busses>
@@
 </segment>
 <segment>
-<wire x1="274.32" y1="50.8" x2="276.86" y2="50.8" width="0.1524" layer="91"/>
 <wire x1="276.86" y1="50.8" x2="276.86" y2="20.32" width="0.1524" layer="91"/>
 <wire x1="276.86" y1="20.32" x2="241.3" y2="20.32" width="0.1524" layer="91"/>
@@
 <junction x="335.28" y="88.9"/>
 <label x="342.9" y="88.9" size="1.778" layer="95"/>
+<pinref part="U2" gate="G$1" pin="GND"/>
+<wire x1="276.86" y1="50.8" x2="274.32" y2="50.8" width="0.1524" layer="91"/>
 </segment>
 <segment>
@@
 <wire x1="269.24" y1="63.5" x2="276.86" y2="63.5" width="0.1524" layer="91"/>
 <wire x1="276.86" y1="63.5" x2="276.86" y2="53.34" width="0.1524" layer="91"/>
-<wire x1="276.86" y1="53.34" x2="274.32" y2="53.34" width="0.1524" layer="91"/>
 <pinref part="D4" gate="A" pin="A"/>
 <wire x1="279.4" y1="73.66" x2="276.86" y2="73.66" width="0.1524" layer="91"/>
 <wire x1="276.86" y1="73.66" x2="276.86" y2="63.5" width="0.1524" layer="91"/>
 <junction x="276.86" y="63.5"/>
+<pinref part="U2" gate="G$1" pin="SW"/>
+<wire x1="276.86" y1="53.34" x2="274.32" y2="53.34" width="0.1524" layer="91"/>
 </segment>
 </net>
 <net name="N$13" class="0">
 <segment>
-<wire x1="274.32" y1="48.26" x2="289.56" y2="48.26" width="0.1524" layer="91"/>
-<wire x1="289.56" y1="48.26" x2="289.56" y2="50.8" width="0.1524" layer="91"/>
 <wire x1="289.56" y1="50.8" x2="281.94" y2="50.8" width="0.1524" layer="91"/>
 <wire x1="281.94" y1="50.8" x2="281.94" y2="58.42" width="0.1524" layer="91"/>
@@
 <wire x1="281.94" y1="58.42" x2="284.48" y2="58.42" width="0.1524" layer="91"/>
 <pinref part="R17" gate="G$1" pin="2"/>
+<wire x1="289.56" y1="50.8" x2="289.56" y2="48.26" width="0.1524" layer="91"/>
+<pinref part="U2" gate="G$1" pin="FB"/>
 <wire x1="289.56" y1="48.26" x2="289.56" y2="40.64" width="0.1524" layer="91"/>
+<wire x1="274.32" y1="48.26" x2="289.56" y2="48.26" width="0.1524" layer="91"/>
 <junction x="289.56" y="48.26"/>
 </segment>
@@
 <pinref part="U$2" gate="G$1" pin="1"/>
 <wire x1="246.38" y1="63.5" x2="254" y2="63.5" width="0.1524" layer="91"/>
-<wire x1="248.92" y1="50.8" x2="246.38" y2="50.8" width="0.1524" layer="91"/>
 <wire x1="246.38" y1="50.8" x2="246.38" y2="63.5" width="0.1524" layer="91"/>
-<wire x1="248.92" y1="48.26" x2="246.38" y2="48.26" width="0.1524" layer="91"/>
 <wire x1="246.38" y1="48.26" x2="246.38" y2="50.8" width="0.1524" layer="91"/>
 <junction x="246.38" y="50.8"/>
@@
 <wire x1="241.3" y1="55.88" x2="241.3" y2="50.8" width="0.1524" layer="91"/>
 <junction x="241.3" y="50.8"/>
-</segment>
-</net>
+<pinref part="U2" gate="G$1" pin="IN"/>
+<wire x1="246.38" y1="50.8" x2="248.92" y2="50.8" width="0.1524" layer="91"/>
+<pinref part="U2" gate="G$1" pin="EN"/>
+<wire x1="246.38" y1="48.26" x2="248.92" y2="48.26" width="0.1524" layer="91"/>
+</segment>
+</net>

Commit message: Update motherBoard.sch
Parts:
- renumbered J6 to BATT
Changed lines of the file:
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@@
 <part name="U$6" library="SCMRCapacitor" deviceset="SCMR18G604SRBA0" device=""/>
 <part name="U$7" library="WNER50FET" deviceset="WNER50FET" device=""/>
-<part name="J6" library="640456-2" deviceset="640456-2" device=""/>
+<part name="BATT" library="640456-2" deviceset="640456-2" device=""/>
 <part name="U$8" library="PIC16LF876A-I_SS" deviceset="PIC16LF876A-I/SS" device=""/>
 <part name="Y2" library="ECS-40-S-4X" deviceset="ECS-40-S-4X" device=""/>
@@
 <instance part="U$6" gate="G$1" x="320.04" y="88.9" smashed="yes"/>
 <instance part="U$7" gate="G$1" x="241.3" y="66.04" smashed="yes" rot="R90"/>
-<instance part="J6" gate="G$1" x="149.86" y="35.56" smashed="yes">
+<instance part="BATT" gate="G$1" x="149.86" y="35.56" smashed="yes">
 <attribute name="NAME" x="144.77536875" y="41.661559375" size="1.271159375" layer="95"/>
 <attribute name="VALUE" x="144.772140625" y="27.928209375" size="1.271959375" layer="96"/>
@@
 <wire x1="175.26" y1="53.34" x2="175.26" y2="20.32" width="0.1524" layer="91"/>
 <junction x="175.26" y="20.32"/>
-<pinref part="J6" gate="G$1" pin="P2"/>
+<pinref part="BATT" gate="G$1" pin="P2"/>
 <wire x1="142.24" y1="33.02" x2="142.24" y2="20.32" width="0.1524" layer="91"/>
 <wire x1="142.24" y1="20.32" x2="144.78" y2="20.32" width="0.1524" layer="91"/>
@@
 <wire x1="144.78" y1="50.8" x2="144.78" y2="43.18" width="0.1524" layer="91"/>
 <wire x1="144.78" y1="43.18" x2="142.24" y2="43.18" width="0.1524" layer="91"/>
-<pinref part="J6" gate="G$1" pin="P1"/>
+<pinref part="BATT" gate="G$1" pin="P1"/>
 <wire x1="142.24" y1="43.18" x2="142.24" y2="38.1" width="0.1524" layer="91"/>
 </segment>

Commit message: Error Fix
Connections:
- net 3.3V: no longer U3.VOUT
Changed lines of the file:
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@@
 <part name="GND17" library="SparkFun-PowerSymbols" deviceset="GND" device=""/>
 <part name="R25" library="SparkFun-Resistors" deviceset="RESISTOR" device="0603" value=" 10K"/>
-<part name="3.3V3" library="supply1" library_urn="urn:adsk.eagle:library:371" deviceset="VCC" device="" value="3.3V"/>
 <part name="GND18" library="SparkFun-PowerSymbols" deviceset="GND" device=""/>
 <part name="R26" library="SparkFun-Resistors" deviceset="RESISTOR" device="0603" value=" 10K"/>
@@
 <attribute name="VALUE" x="133.604" y="91.44" size="1.778" layer="96" font="vector" rot="R90" align="top-center"/>
 </instance>
-<instance part="3.3V3" gate="VCC" x="132.08" y="106.68" smashed="yes"/>
 <instance part="GND18" gate="1" x="58.42" y="30.48" smashed="yes">
 <attribute name="VALUE" x="58.42" y="30.226" size="1.778" layer="96" align="top-center"/>
@@
 <pinref part="R25" gate="G$1" pin="2"/>
 <wire x1="142.24" y1="96.52" x2="132.08" y2="96.52" width="0.1524" layer="91"/>
-<wire x1="132.08" y1="96.52" x2="132.08" y2="104.14" width="0.1524" layer="91"/>
-<junction x="132.08" y="96.52"/>
-<pinref part="3.3V3" gate="VCC" pin="VCC"/>
-<label x="134.62" y="101.6" size="1.778" layer="95"/>
 </segment>
 <segment>
@@
 <junction x="335.28" y="88.9"/>
 <label x="342.9" y="88.9" size="1.778" layer="95"/>
+<wire x1="276.86" y1="50.8" x2="274.32" y2="50.8" width="0.1524" layer="91"/>
 <pinref part="U2" gate="G$1" pin="GND"/>
-<wire x1="276.86" y1="50.8" x2="274.32" y2="50.8" width="0.1524" layer="91"/>
 </segment>
 <segment>
@@
 <wire x1="276.86" y1="73.66" x2="276.86" y2="63.5" width="0.1524" layer="91"/>
 <junction x="276.86" y="63.5"/>
+<wire x1="276.86" y1="53.34" x2="274.32" y2="53.34" width="0.1524" layer="91"/>
 <pinref part="U2" gate="G$1" pin="SW"/>
-<wire x1="276.86" y1="53.34" x2="274.32" y2="53.34" width="0.1524" layer="91"/>
 </segment>
 </net>
@@
 <pinref part="R17" gate="G$1" pin="2"/>
 <wire x1="289.56" y1="50.8" x2="289.56" y2="48.26" width="0.1524" layer="91"/>
-<pinref part="U2" gate="G$1" pin="FB"/>
 <wire x1="289.56" y1="48.26" x2="289.56" y2="40.64" width="0.1524" layer="91"/>
 <wire x1="274.32" y1="48.26" x2="289.56" y2="48.26" width="0.1524" layer="91"/>
 <junction x="289.56" y="48.26"/>
+<pinref part="U2" gate="G$1" pin="FB"/>
 </segment>
 </net>
@@
 <net name="3.3V" class="0">
 <segment>
-<pinref part="U3" gate="A" pin="VOUT"/>
-<wire x1="414.02" y1="45.72" x2="426.72" y2="45.72" width="0.1524" layer="91"/>
 <pinref part="C7" gate="G$1" pin="1"/>
 <wire x1="426.72" y1="45.72" x2="426.72" y2="38.1" width="0.1524" layer="91"/>
 <wire x1="426.72" y1="45.72" x2="434.34" y2="45.72" width="0.1524" layer="91"/>
-<junction x="426.72" y="45.72"/>
-<label x="434.34" y="45.72" size="1.778" layer="95"/>
 </segment>
 </net>
@@
 <wire x1="241.3" y1="55.88" x2="241.3" y2="50.8" width="0.1524" layer="91"/>
 <junction x="241.3" y="50.8"/>
+<wire x1="246.38" y1="50.8" x2="248.92" y2="50.8" width="0.1524" layer="91"/>
+<wire x1="246.38" y1="48.26" x2="248.92" y2="48.26" width="0.1524" layer="91"/>
 <pinref part="U2" gate="G$1" pin="IN"/>
-<wire x1="246.38" y1="50.8" x2="248.92" y2="50.8" width="0.1524" layer="91"/>
 <pinref part="U2" gate="G$1" pin="EN"/>
-<wire x1="246.38" y1="48.26" x2="248.92" y2="48.26" width="0.1524" layer="91"/>
-</segment>
-</net>
+</segment>
+</net>
