File: eagle/projects/smartBobber Mother Board/motherBoard/motherBoard.sch (EAGLE design)
At the start: 61 parts, among them J1 10118193-0001LF, Q3 2A/20V/150mΩ, Q4 MMBT3904, U1 MCP73831, U2 MT3608, U3 LTC3531ES6-3_3, Y2 ECS-40-S-4X

Commit message: motherBoard
Parts:
- removed GLED: (no value), led:LED5MM
- added D2: Green, SparkFun:LED0603
Connections:
- removed net N$2: GLED.C, R14.2
- new net N$1: D2.C, R14.2
- net N$11: now also D2.A; no longer GLED.A
Changed lines of the file:
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@@
 <part name="U$3" library="FS312F-G" deviceset="FS312F-G" device=""/>
 <part name="U$4" library="FS8205" deviceset="FS8205" device=""/>
-<part name="GLED" library="led" library_urn="urn:adsk.eagle:library:259" deviceset="LED" device="5MM" package3d_urn="urn:adsk.eagle:package:15799/2"/>
 <part name="U$5" library="SCMRCapacitor" deviceset="SCMR18G604SRBA0" device=""/>
 <part name="U$6" library="SCMRCapacitor" deviceset="SCMR18G604SRBA0" device=""/>
@@
 <part name="U2" library="MT3608" deviceset="MT3608" device=""/>
 <part name="3.3V1" library="supply1" library_urn="urn:adsk.eagle:library:371" deviceset="VCC" device="" value="3.3V"/>
+<part name="D2" library="SparkFun" deviceset="LED" device="0603" value="Green"/>
 </parts>
 <sheets>
@@
 <instance part="U$3" gate="G$1" x="195.58" y="60.96" smashed="yes" rot="R180"/>
 <instance part="U$4" gate="G$1" x="195.58" y="33.02" smashed="yes"/>
-<instance part="GLED" gate="G$1" x="63.5" y="35.56" smashed="yes">
-<attribute name="NAME" x="67.056" y="30.988" size="1.778" layer="95" rot="R90"/>
-<attribute name="VALUE" x="69.215" y="30.988" size="1.778" layer="96" rot="R90"/>
-</instance>
 <instance part="U$5" gate="G$1" x="294.64" y="88.9" smashed="yes"/>
 <instance part="U$6" gate="G$1" x="320.04" y="88.9" smashed="yes"/>
@@
 <attribute name="NAME" x="252.73" y="60.96" size="1.778" layer="95" rot="MR0" align="center-left"/>
 <attribute name="VALUE" x="252.73" y="58.42" size="1.778" layer="96" rot="MR0" align="center-left"/>
+</instance>
+<instance part="D2" gate="G$1" x="63.5" y="35.56" smashed="yes">
+<attribute name="NAME" x="67.056" y="30.988" size="1.778" layer="95" rot="R90"/>
+<attribute name="VALUE" x="69.215" y="30.988" size="1.778" layer="96" rot="R90"/>
 </instance>
 </instances>
@@
 <pinref part="U1" gate="G$1" pin="VIN"/>
 <wire x1="45.72" y1="40.64" x2="63.5" y2="40.64" width="0.1524" layer="91"/>
-<pinref part="GLED" gate="G$1" pin="A"/>
+<pinref part="D2" gate="G$1" pin="A"/>
 <wire x1="63.5" y1="40.64" x2="81.28" y2="40.64" width="0.1524" layer="91"/>
 <wire x1="63.5" y1="40.64" x2="63.5" y2="38.1" width="0.1524" layer="91"/>
@@
 </segment>
 </net>
-<net name="N$2" class="0">
-<segment>
-<pinref part="GLED" gate="G$1" pin="C"/>
-<pinref part="R14" gate="G$1" pin="2"/>
-<wire x1="63.5" y1="30.48" x2="63.5" y2="27.94" width="0.1524" layer="91"/>
-</segment>
-</net>
 <net name="N$19" class="0">
 <segment>
@@
 </segment>
 </net>
+<net name="N$1" class="0">
+<segment>
+<pinref part="D2" gate="G$1" pin="C"/>
+<pinref part="R14" gate="G$1" pin="2"/>
+<wire x1="63.5" y1="30.48" x2="63.5" y2="27.94" width="0.1524" layer="91"/>
+</segment>
+</net>

Commit message: motherBoard
Connections:
- removed net LVP: PIC.6
- removed net N$26: R25.1, S3.2, U$8.~MCLR/VPP
- net 3.3V: now also U3.VOUT
- net MCLR: now also R25.1, S3.2, U$8.~MCLR/VPP
- net PGC: now also U$8.RB6/PGC
- net PGD: now also U$8.RB7/PGD
Changed lines of the file:
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@@
 <label x="22.86" y="10.16" size="1.778" layer="95"/>
+</segment>
+<segment>
+<pinref part="U$8" gate="A" pin="~MCLR/VPP"/>
+<wire x1="124.46" y1="86.36" x2="132.08" y2="86.36" width="0.1524" layer="91"/>
+<pinref part="R25" gate="G$1" pin="1"/>
+<wire x1="132.08" y1="86.36" x2="149.86" y2="86.36" width="0.1524" layer="91"/>
+<junction x="132.08" y="86.36"/>
+<pinref part="S3" gate="G$1" pin="2"/>
+<label x="139.7" y="86.36" size="1.778" layer="95"/>
 </segment>
 </net>
@@
 <label x="22.86" y="17.78" size="1.778" layer="95"/>
 </segment>
+<segment>
+<pinref part="U$8" gate="A" pin="RB7/PGD"/>
+<wire x1="149.86" y1="43.18" x2="139.7" y2="43.18" width="0.1524" layer="91"/>
+<label x="139.7" y="43.18" size="1.778" layer="95"/>
+</segment>
 </net>
 <net name="PGC" class="0">
@@
 <label x="22.86" y="20.32" size="1.778" layer="95"/>
 </segment>
-</net>
-<net name="LVP" class="0">
-<segment>
-<pinref part="PIC" gate="G$1" pin="6"/>
-<wire x1="17.78" y1="22.86" x2="27.94" y2="22.86" width="0.1524" layer="91"/>
-<label x="22.86" y="22.86" size="1.778" layer="95"/>
+<segment>
+<pinref part="U$8" gate="A" pin="RB6/PGC"/>
+<wire x1="149.86" y1="45.72" x2="139.7" y2="45.72" width="0.1524" layer="91"/>
+<label x="139.7" y="45.72" size="1.778" layer="95"/>
 </segment>
 </net>
@@
 <pinref part="R23" gate="G$1" pin="2"/>
 <wire x1="238.76" y1="160.02" x2="236.22" y2="160.02" width="0.1524" layer="91"/>
-</segment>
-</net>
-<net name="N$26" class="0">
-<segment>
-<pinref part="U$8" gate="A" pin="~MCLR/VPP"/>
-<wire x1="124.46" y1="86.36" x2="132.08" y2="86.36" width="0.1524" layer="91"/>
-<pinref part="R25" gate="G$1" pin="1"/>
-<wire x1="132.08" y1="86.36" x2="149.86" y2="86.36" width="0.1524" layer="91"/>
-<junction x="132.08" y="86.36"/>
-<pinref part="S3" gate="G$1" pin="2"/>
 </segment>
 </net>
@@
 <wire x1="426.72" y1="45.72" x2="426.72" y2="38.1" width="0.1524" layer="91"/>
 <wire x1="426.72" y1="45.72" x2="434.34" y2="45.72" width="0.1524" layer="91"/>
-</segment>
-</net>
+<pinref part="U3" gate="A" pin="VOUT"/>
+<wire x1="414.02" y1="45.72" x2="426.72" y2="45.72" width="0.1524" layer="91"/>
+<junction x="426.72" y="45.72"/>
+<label x="431.8" y="48.26" size="1.778" layer="95"/>
+</segment>
+</net>

Commit message: motherBoard
Parts:
- removed R13: 2k, SparkFun-Resistors:RESISTOR0805
- added R1: 2k, SparkFun-Resistors:RESISTOR0603
Connections:
- net N$9: now also R1.2; no longer R13.2
- net _12V: now also R1.1; no longer R13.1
Changed lines of the file:
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@@
 <part name="U3" library="LTC3531ES6-3_3" deviceset="LTC3531ES6-3_3" device=""/>
 <part name="10UH" library="MLZ2012N100LT000" deviceset="MLZ2012N100LT000" device=""/>
-<part name="R13" library="SparkFun-Resistors" deviceset="RESISTOR" device="0805" value="2k"/>
 <part name="R14" library="SparkFun-Resistors" deviceset="RESISTOR" device="0603" value="470"/>
 <part name="R15" library="SparkFun-Resistors" deviceset="RESISTOR" device="0603" value="100"/>
@@
 <part name="3.3V1" library="supply1" library_urn="urn:adsk.eagle:library:371" deviceset="VCC" device="" value="3.3V"/>
 <part name="D2" library="SparkFun" deviceset="LED" device="0603" value="Green"/>
+<part name="R1" library="SparkFun-Resistors" deviceset="RESISTOR" device="0603" value="2k"/>
 </parts>
 <sheets>
@@
 <attribute name="VALUE" x="368.295609375" y="63.497809375" size="1.77953125" layer="96"/>
 </instance>
-<instance part="R13" gate="G$1" x="111.76" y="27.94" smashed="yes" rot="R90">
-<attribute name="NAME" x="110.236" y="27.94" size="1.778" layer="95" font="vector" rot="R90" align="bottom-center"/>
-<attribute name="VALUE" x="113.284" y="27.94" size="1.778" layer="96" font="vector" rot="R90" align="top-center"/>
-</instance>
 <instance part="R14" gate="G$1" x="63.5" y="22.86" smashed="yes" rot="R90">
 <attribute name="NAME" x="61.976" y="22.86" size="1.778" layer="95" font="vector" rot="R90" align="bottom-center"/>
@@
 <attribute name="NAME" x="67.056" y="30.988" size="1.778" layer="95" rot="R90"/>
 <attribute name="VALUE" x="69.215" y="30.988" size="1.778" layer="96" rot="R90"/>
+</instance>
+<instance part="R1" gate="G$1" x="111.76" y="27.94" smashed="yes" rot="R90">
+<attribute name="NAME" x="110.236" y="27.94" size="1.778" layer="95" font="vector" rot="R90" align="bottom-center"/>
+<attribute name="VALUE" x="113.284" y="27.94" size="1.778" layer="96" font="vector" rot="R90" align="top-center"/>
 </instance>
 </instances>
@@
 </segment>
 <segment>
-<pinref part="R13" gate="G$1" pin="1"/>
 <pinref part="SUPPLY4" gate="GND" pin="GND"/>
 <wire x1="111.76" y1="22.86" x2="111.76" y2="20.32" width="0.1524" layer="91"/>
@@
 <pinref part="U1" gate="G$1" pin="VSS"/>
 <wire x1="104.14" y1="35.56" x2="101.6" y2="35.56" width="0.1524" layer="91"/>
+<pinref part="R1" gate="G$1" pin="1"/>
 </segment>
 </net>
@@
 <pinref part="U1" gate="G$1" pin="PROG"/>
 <wire x1="101.6" y1="38.1" x2="111.76" y2="38.1" width="0.1524" layer="91"/>
-<pinref part="R13" gate="G$1" pin="2"/>
 <wire x1="111.76" y1="38.1" x2="111.76" y2="33.02" width="0.1524" layer="91"/>
-</segment>
-</net>
+<pinref part="R1" gate="G$1" pin="2"/>
+</segment>
+</net>

Commit message: motherBoard V1
Parts:
- removed BLED4, BLED5, BLED6, RLED4, RLED5, RLED6: (no value), led:LED5MM
- added D1, D6: CLX6F-FKC-CKNNQDGBB7A363, CLX6F-LED:CLX6F-FKC-CKNNQDGBB7A363
- R23: value 47 -> 20
- R24: value 1 -> 5
Connections:
- net BLUE_LEDS: now also D6.4, D6.5, D6.6; no longer BLED4.A, BLED5.A, BLED6.A
- net N$24: now also D6.1, D6.2, D6.3; no longer BLED4.C, BLED5.C, BLED6.C
- net N$25: now also D1.1, D1.2, D1.3; no longer RLED4.C, RLED5.C, RLED6.C
- net RED_LEDS: now also D1.4, D1.5, D1.6; no longer RLED4.A, RLED5.A, RLED6.A

Commit message: Bullshit
Parts:
- added U$1: 12V-BOARD, 12V-Board:12V-BOARD
Connections:
- removed net N$21: C3.1, U$2.1, U$7.1, U2.EN, U2.IN
- new net N$2: C3.1, U$1.VIN+, U$2.1, U$7.1, U2.EN, U2.IN
- net 12V: now also U$1.VOUT+
- net GND: now also C13.2, C3.2, C5.2, C7.2, R16.1, R17.1, U$1.VIN-, U$1.VOUT-, U$4.S2, U$6.-, U2.GND, U3.GND/PGND
- net _12V: no longer C13.2, C3.2, C5.2, C7.2, R16.1, R17.1, U$4.S2, U$6.-, U2.GND, U3.GND/PGND

Commit message: Led Part and Board Update
Parts:
- removed D1, D6: CLX6F-FKC-CKNNQDGBB7A363, CLX6F-LED:CLX6F-FKC-CKNNQDGBB7A363
- removed R23: 20, SparkFun-Resistors:RESISTOR0603
- added R2: 5, SparkFun-Resistors:RESISTOR0603
- added R3, R4: 20, SparkFun-Resistors:RESISTOR0603
- added U$10, U$9: CLX6F-BKB-CPR453, CLX6F-LED:CLX6F-BKB-CPR453
- added U$11, U$12: CLX6F-RKB-CSTBB3, CLX6F-LED:CLX6F-RKB-CSTBB3
Connections:
- removed net BLUE_LEDS: D6.4, D6.5, D6.6, U$8.RC4/SDI/SDA
- removed net N$24: D6.1, D6.2, D6.3, R24.2
- removed net RED_LEDS: D1.4, D1.5, D1.6, U$8.RC5/SDO
- new net BLUE_LEDS_1: U$8.RC4/SDI/SDA, U$9.4, U$9.5, U$9.6
- new net BLUE_LEDS_2: U$10.4, U$10.5, U$10.6, U$8.RA1/AN1
- new net N$21: R24.2, U$10.1, U$10.2, U$10.3
- new net N$3: R2.2, U$9.1, U$9.2, U$9.3
- new net N$5: R3.2, U$12.1, U$12.2, U$12.3
- new net RED_LEDS_1: U$12.4, U$12.5, U$12.6, U$8.RC5/SDO
- new net RED_LEDS_2: U$11.4, U$11.5, U$11.6, U$8.RA2/AN2/VREF-/CVREF
- net GND: now also R2.1, R3.1, R4.1; no longer R23.1
- net N$25: now also R4.2, U$11.1, U$11.2, U$11.3; no longer D1.1, D1.2, D1.3, R23.2
Other:
- moved on the sheet: R24

Commit message: Schematic Update
Connections:
- net N$16 renamed LOAD
- net N$8 renamed BATT+
- new net N$4: U$1.VIN-, U$1.VOUT-
- net GND: no longer U$1.VIN-, U$1.VOUT-
Other:
- note added: "Zachary L. Hutson"
- moved on the sheet: 10UH, BATT, C11, C12, C13, C3, C5, C7, C9, D2, D4, R1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

Commit message: update schematic and board
Connections:
- new net GND1: BATT.P2, C12.2, U$3.GND, U$4.S1
- net _12V: no longer BATT.P2, C12.2, U$3.GND, U$4.S1
Changed lines of the file:
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@@
 <parts>
 <part name="SUPPLY1" library="supply2" library_urn="urn:adsk.eagle:library:372" deviceset="GND" device="" value="GND1"/>
-<part name="SUPPLY2" library="supply2" library_urn="urn:adsk.eagle:library:372" deviceset="GND" device="" value="GND1"/>
-<part name="SUPPLY3" library="supply2" library_urn="urn:adsk.eagle:library:372" deviceset="GND" device="" value="GND1"/>
-<part name="SUPPLY4" library="supply2" library_urn="urn:adsk.eagle:library:372" deviceset="GND" device="" value="GND1"/>
 <part name="SUPPLY5" library="supply2" library_urn="urn:adsk.eagle:library:372" deviceset="GND" device="" value="GND1"/>
 <part name="S1" library="JS102011SAQN" deviceset="JS102011SAQN" device=""/>
@@
 <plain>
 <wire x1="0" y1="48.26" x2="0" y2="5.08" width="0.1524" layer="94" style="dashdot"/>
-<text x="5.08" y="58.42" size="1.778" layer="95">Charging Circuit </text>
+<text x="7.62" y="76.2" size="1.778" layer="95">Charging Circuit </text>
 <text x="7.62" y="170.18" size="1.778" layer="95">Protection Circuit </text>
 <text x="134.62" y="76.2" size="1.778" layer="95">3.3V Supply Circuit </text>
@@
 <attribute name="VALUE" x="26.035" y="12.065" size="1.778" layer="96"/>
 </instance>
-<instance part="SUPPLY2" gate="GND" x="35.56" y="15.24" smashed="yes">
-<attribute name="VALUE" x="33.655" y="12.065" size="1.778" layer="96"/>
-</instance>
-<instance part="SUPPLY3" gate="GND" x="106.68" y="15.24" smashed="yes">
-<attribute name="VALUE" x="104.775" y="12.065" size="1.778" layer="96"/>
-</instance>
-<instance part="SUPPLY4" gate="GND" x="99.06" y="15.24" smashed="yes">
-<attribute name="VALUE" x="97.155" y="12.065" size="1.778" layer="96"/>
-</instance>
-<instance part="SUPPLY5" gate="GND" x="20.32" y="93.98" smashed="yes">
-<attribute name="VALUE" x="18.415" y="90.805" size="1.778" layer="96"/>
+<instance part="SUPPLY5" gate="GND" x="22.86" y="93.98" smashed="yes">
+<attribute name="VALUE" x="20.955" y="90.805" size="1.778" layer="96"/>
 </instance>
 <instance part="S1" gate="G$1" x="63.5" y="157.48" smashed="yes">
@@
 </instance>
 <instance part="D2" gate="G$1" x="45.72" y="35.56" smashed="yes" rot="R90">
-<attribute name="NAME" x="50.292" y="39.116" size="1.778" layer="95" rot="R180"/>
-<attribute name="VALUE" x="50.292" y="41.275" size="1.778" layer="96" rot="R180"/>
+<attribute name="NAME" x="48.768" y="39.116" size="1.778" layer="95" rot="R180"/>
+<attribute name="VALUE" x="50.8" y="32.385" size="1.778" layer="96" rot="R180"/>
 </instance>
 <instance part="R1" gate="G$1" x="99.06" y="27.94" smashed="yes" rot="R90">
@@
 <net name="_12V" class="0">
 <segment>
+<pinref part="C11" gate="G$1" pin="2"/>
+<wire x1="106.68" y1="25.4" x2="106.68" y2="17.78" width="0.1524" layer="91"/>
+<wire x1="99.06" y1="22.86" x2="99.06" y2="17.78" width="0.1524" layer="91"/>
+<pinref part="R1" gate="G$1" pin="1"/>
 <wire x1="20.32" y1="30.48" x2="27.94" y2="30.48" width="0.1524" layer="91"/>
 <pinref part="SUPPLY1" gate="GND" pin="GND"/>
 <wire x1="27.94" y1="30.48" x2="27.94" y2="17.78" width="0.1524" layer="91"/>
 <pinref part="J1" gate="G$1" pin="GND"/>
-</segment>
-<segment>
-<pinref part="SUPPLY5" gate="GND" pin="GND"/>
-<wire x1="20.32" y1="99.06" x2="20.32" y2="96.52" width="0.1524" layer="91"/>
-<wire x1="20.32" y1="99.06" x2="43.18" y2="99.06" width="0.1524" layer="91"/>
-<pinref part="C12" gate="G$1" pin="2"/>
-<wire x1="43.18" y1="111.76" x2="43.18" y2="99.06" width="0.1524" layer="91"/>
-<wire x1="43.18" y1="99.06" x2="50.8" y2="99.06" width="0.1524" layer="91"/>
-<junction x="43.18" y="99.06"/>
-<wire x1="50.8" y1="99.06" x2="55.88" y2="99.06" width="0.1524" layer="91"/>
-<wire x1="55.88" y1="99.06" x2="55.88" y2="116.84" width="0.1524" layer="91"/>
-<pinref part="U$4" gate="G$1" pin="S1"/>
-<wire x1="55.88" y1="116.84" x2="60.96" y2="116.84" width="0.1524" layer="91"/>
-<pinref part="U$3" gate="G$1" pin="GND"/>
-<wire x1="60.96" y1="132.08" x2="50.8" y2="132.08" width="0.1524" layer="91"/>
-<wire x1="50.8" y1="132.08" x2="50.8" y2="99.06" width="0.1524" layer="91"/>
-<junction x="50.8" y="99.06"/>
-<pinref part="BATT" gate="G$1" pin="P2"/>
-<wire x1="15.24" y1="109.22" x2="20.32" y2="109.22" width="0.1524" layer="91"/>
-<wire x1="20.32" y1="109.22" x2="20.32" y2="99.06" width="0.1524" layer="91"/>
-<junction x="20.32" y="99.06"/>
-</segment>
-<segment>
 <pinref part="C9" gate="G$1" pin="2"/>
-<pinref part="SUPPLY2" gate="GND" pin="GND"/>
 <wire x1="35.56" y1="27.94" x2="35.56" y2="17.78" width="0.1524" layer="91"/>
-</segment>
-<segment>
-<pinref part="C11" gate="G$1" pin="2"/>
-<pinref part="SUPPLY3" gate="GND" pin="GND"/>
-<wire x1="106.68" y1="25.4" x2="106.68" y2="17.78" width="0.1524" layer="91"/>
-</segment>
-<segment>
-<pinref part="SUPPLY4" gate="GND" pin="GND"/>
-<wire x1="99.06" y1="22.86" x2="99.06" y2="20.32" width="0.1524" layer="91"/>
-<wire x1="99.06" y1="20.32" x2="99.06" y2="17.78" width="0.1524" layer="91"/>
-<wire x1="99.06" y1="20.32" x2="93.98" y2="20.32" width="0.1524" layer="91"/>
-<junction x="99.06" y="20.32"/>
-<wire x1="93.98" y1="20.32" x2="93.98" y2="35.56" width="0.1524" layer="91"/>
+<wire x1="27.94" y1="17.78" x2="35.56" y2="17.78" width="0.1524" layer="91"/>
+<junction x="27.94" y="17.78"/>
+<junction x="35.56" y="17.78"/>
+<wire x1="99.06" y1="17.78" x2="93.98" y2="17.78" width="0.1524" layer="91"/>
+<junction x="99.06" y="17.78"/>
+<wire x1="93.98" y1="17.78" x2="35.56" y2="17.78" width="0.1524" layer="91"/>
+<wire x1="106.68" y1="17.78" x2="99.06" y2="17.78" width="0.1524" layer="91"/>
 <pinref part="U1" gate="G$1" pin="VSS"/>
 <wire x1="93.98" y1="35.56" x2="88.9" y2="35.56" width="0.1524" layer="91"/>
-<pinref part="R1" gate="G$1" pin="1"/>
+<wire x1="93.98" y1="17.78" x2="93.98" y2="35.56" width="0.1524" layer="91"/>
+<junction x="93.98" y="17.78"/>
 </segment>
 </net>
@@
 <segment>
 <pinref part="S1" gate="G$1" pin="1"/>
-<wire x1="20.32" y1="129.54" x2="20.32" y2="160.02" width="0.1524" layer="91"/>
-<wire x1="20.32" y1="160.02" x2="55.88" y2="160.02" width="0.1524" layer="91"/>
+<wire x1="22.86" y1="129.54" x2="22.86" y2="160.02" width="0.1524" layer="91"/>
+<wire x1="22.86" y1="160.02" x2="55.88" y2="160.02" width="0.1524" layer="91"/>
 <pinref part="R15" gate="G$1" pin="1"/>
-<wire x1="20.32" y1="129.54" x2="25.4" y2="129.54" width="0.1524" layer="91"/>
+<wire x1="22.86" y1="129.54" x2="25.4" y2="129.54" width="0.1524" layer="91"/>
 <pinref part="BATT" gate="G$1" pin="P1"/>
-<wire x1="15.24" y1="114.3" x2="20.32" y2="114.3" width="0.1524" layer="91"/>
-<wire x1="20.32" y1="114.3" x2="20.32" y2="129.54" width="0.1524" layer="91"/>
-<junction x="20.32" y="129.54"/>
-<label x="20.32" y="119.38" size="1.778" layer="95" rot="R90"/>
+<wire x1="15.24" y1="114.3" x2="22.86" y2="114.3" width="0.1524" layer="91"/>
+<wire x1="22.86" y1="114.3" x2="22.86" y2="129.54" width="0.1524" layer="91"/>
+<junction x="22.86" y="129.54"/>
+<label x="22.86" y="116.84" size="1.778" layer="95" rot="R180"/>
 </segment>
 </net>
@@
 <segment>
 <pinref part="U$1" gate="G$1" pin="VOUT-"/>
-<wire x1="202.2" y1="152.4" x2="208.28" y2="152.4" width="0.1524" layer="91"/>
-<wire x1="208.28" y1="152.4" x2="208.28" y2="147.32" width="0.1524" layer="91"/>
-<wire x1="208.28" y1="147.32" x2="170.18" y2="147.32" width="0.1524" layer="91"/>
-<wire x1="170.18" y1="147.32" x2="170.18" y2="152.4" width="0.1524" layer="91"/>
+<wire x1="202.2" y1="152.4" x2="205.74" y2="152.4" width="0.1524" layer="91"/>
+<wire x1="205.74" y1="152.4" x2="205.74" y2="147.32" width="0.1524" layer="91"/>
+<wire x1="205.74" y1="147.32" x2="172.72" y2="147.32" width="0.1524" layer="91"/>
+<wire x1="172.72" y1="147.32" x2="172.72" y2="152.4" width="0.1524" layer="91"/>
 <pinref part="U$1" gate="G$1" pin="VIN-"/>
-<wire x1="170.18" y1="152.4" x2="174.72" y2="152.4" width="0.1524" layer="91"/>
-</segment>
-</net>
+<wire x1="172.72" y1="152.4" x2="174.72" y2="152.4" width="0.1524" layer="91"/>
+</segment>
+</net>
+<net name="GND1" class="0">
+<segment>
+<pinref part="SUPPLY5" gate="GND" pin="GND"/>
+<wire x1="22.86" y1="99.06" x2="22.86" y2="96.52" width="0.1524" layer="91"/>
+<wire x1="22.86" y1="99.06" x2="43.18" y2="99.06" width="0.1524" layer="91"/>
+<pinref part="C12" gate="G$1" pin="2"/>
+<wire x1="43.18" y1="111.76" x2="43.18" y2="99.06" width="0.1524" layer="91"/>
+<wire x1="43.18" y1="99.06" x2="50.8" y2="99.06" width="0.1524" layer="91"/>
+<junction x="43.18" y="99.06"/>
+<wire x1="50.8" y1="99.06" x2="55.88" y2="99.06" width="0.1524" layer="91"/>
+<wire x1="55.88" y1="99.06" x2="55.88" y2="116.84" width="0.1524" layer="91"/>
+<pinref part="U$4" gate="G$1" pin="S1"/>
+<wire x1="55.88" y1="116.84" x2="60.96" y2="116.84" width="0.1524" layer="91"/>
+<pinref part="U$3" gate="G$1" pin="GND"/>
+<wire x1="60.96" y1="132.08" x2="50.8" y2="132.08" width="0.1524" layer="91"/>
+<wire x1="50.8" y1="132.08" x2="50.8" y2="99.06" width="0.1524" layer="91"/>
+<junction x="50.8" y="99.06"/>
+<pinref part="BATT" gate="G$1" pin="P2"/>
+<wire x1="15.24" y1="109.22" x2="22.86" y2="109.22" width="0.1524" layer="91"/>
+<wire x1="22.86" y1="109.22" x2="22.86" y2="99.06" width="0.1524" layer="91"/>
+<junction x="22.86" y="99.06"/>
+<label x="15.24" y="109.22" size="1.778" layer="95"/>
+</segment>
+</net>
