File: eagle/projects/smartBobber Mother Board/motherBoard/motherBoard.brd (EAGLE design)
At the start: 160 x 100 mm, 61 parts, among them J1 10118193-0001LF, J10 640456-5, J11 640456-2, J8 640456-2, J9 640456-3, Q3 2A/20V/150mΩ, Q4 MMBT3904, U1 MCP73831, U2 MT3608, U3 LTC3531ES6-3_3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

Commit message: Error Fix
Parts:
- moved U2 111.2 mm to (68.6, 64.8)
Connections:
- net 3.3V: no longer U3.3
Changed lines of the file:
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@@
 <attribute name="VALUE" x="14.9225" y="94.1705" size="0.4064" layer="27" rot="R180"/>
-</element>
-<element name="U2" library="MT3608" package="SOT95P280X145-6N" value="MT3608" x="-41.91" y="77.47" smashed="yes">
-<attribute name="ARROW_PART_NUMBER" value="MT3608" x="0" y="0" size="1.778" layer="27" display="off"/>
-<attribute name="ARROW_PRICE-STOCK" value="" x="0" y="0" size="1.778" layer="27" display="off"/>
-<attribute name="DESCRIPTION" value="High Efficiency 1.2MHz 2A Step Up Converter" x="0" y="0" size="1.778" layer="27" display="off"/>
-<attribute name="HEIGHT" value="1.45mm" x="0" y="0" size="1.778" layer="27" display="off"/>
-<attribute name="MANUFACTURER_NAME" value="Aerosemi" x="0" y="0" size="1.778" layer="27" display="off"/>
-<attribute name="MANUFACTURER_PART_NUMBER" value="MT3608" x="0" y="0" size="1.778" layer="27" display="off"/>
-<attribute name="NAME" x="-41.91" y="77.47" size="1.27" layer="25" align="center"/>
-<attribute name="RS_PART_NUMBER" value="" x="0" y="0" size="1.778" layer="27" display="off"/>
-<attribute name="RS_PRICE-STOCK" value="" x="0" y="0" size="1.778" layer="27" display="off"/>
-<attribute name="VALUE" x="-41.91" y="77.47" size="1.27" layer="27" align="center"/>
 </element>
 <element name="U3" library="LTC3531ES6-3_3" package="TSOT-23_S6" value="LTC3531ES6-3_3" x="-62.23" y="69.85" smashed="yes">
@@
 <attribute name="VALUE" x="-34.99111875" y="31.17456875" size="1.27245" layer="27"/>
 </element>
+<element name="U2" library="MT3608" package="SOT95P280X145-6N" value="MT3608" x="68.58" y="64.77" smashed="yes">
+<attribute name="ARROW_PART_NUMBER" value="MT3608" x="68.58" y="64.77" size="1.778" layer="27" display="off"/>
+<attribute name="ARROW_PRICE-STOCK" value="" x="68.58" y="64.77" size="1.778" layer="27" display="off"/>
+<attribute name="DESCRIPTION" value="High Efficiency 1.2MHz 2A Step Up Converter" x="68.58" y="64.77" size="1.778" layer="27" display="off"/>
+<attribute name="HEIGHT" value="1.45mm" x="68.58" y="64.77" size="1.778" layer="27" display="off"/>
+<attribute name="MANUFACTURER_NAME" value="Aerosemi" x="68.58" y="64.77" size="1.778" layer="27" display="off"/>
+<attribute name="MANUFACTURER_PART_NUMBER" value="MT3608" x="68.58" y="64.77" size="1.778" layer="27" display="off"/>
+<attribute name="RS_PART_NUMBER" value="" x="68.58" y="64.77" size="1.778" layer="27" display="off"/>
+<attribute name="RS_PRICE-STOCK" value="" x="68.58" y="64.77" size="1.778" layer="27" display="off"/>
+</element>
 </elements>
 <signals>
@@
 <contactref element="R25" pad="2"/>
 <contactref element="C15" pad="1"/>
-<contactref element="U3" pad="3"/>
 <contactref element="C7" pad="1"/>
 <wire x1="81.28" y1="51.22" x2="91.2114" y2="48.5648" width="0" layer="19" extent="1-1"/>
@@
 <wire x1="-33.02" y1="77.47" x2="-22.86" y2="24.13" width="0" layer="19" extent="1-1"/>
 <wire x1="-60.54" y1="77.47" x2="-33.02" y2="77.47" width="0" layer="19" extent="1-1"/>
-<wire x1="-63.373" y1="68.9" x2="-60.54" y2="77.47" width="0" layer="19" extent="1-1"/>
 </signal>
 <signal name="PGD">
@@
 <contactref element="U$3" pad="6"/>
 <contactref element="BATT" pad="2"/>
-<contactref element="U2" pad="2"/>
 <contactref element="U3" pad="2"/>
 <contactref element="R16" pad="1"/>
@@
 <contactref element="R13" pad="1"/>
 <contactref element="U1" pad="2"/>
+<contactref element="U2" pad="2"/>
 <wire x1="56.73" y1="86.36" x2="128.72" y2="71.12" width="0" layer="19" extent="1-1"/>
 <wire x1="52.92" y1="86.36" x2="56.73" y2="86.36" width="0" layer="19" extent="1-1"/>
@@
 <wire x1="-8.04" y1="85.09" x2="5.08" y2="81.28" width="0" layer="19" extent="1-1"/>
 <wire x1="-38.95" y1="82.55" x2="-8.04" y2="85.09" width="0" layer="19" extent="1-1"/>
-<wire x1="-43.16" y1="77.47" x2="-38.95" y2="82.55" width="0" layer="19" extent="1-1"/>
-<wire x1="-58.84" y1="77.47" x2="-43.16" y2="77.47" width="0" layer="19" extent="1-1"/>
+<wire x1="-58.84" y1="77.47" x2="-38.95" y2="82.55" width="0" layer="19" extent="1-1"/>
 <wire x1="-63.373" y1="69.85" x2="-58.84" y2="77.47" width="0" layer="19" extent="1-1"/>
+<wire x1="67.33" y1="64.77" x2="-63.373" y2="69.85" width="0" layer="19" extent="1-1"/>
 </signal>
 <signal name="N$20">
@@
 <signal name="N$12">
 <contactref element="U$2" pad="2"/>
+<contactref element="D4" pad="A"/>
 <contactref element="U2" pad="1"/>
-<contactref element="D4" pad="A"/>
-<wire x1="-43.16" y1="78.42" x2="88.9" y2="85.72" width="0" layer="19" extent="1-1"/>
-<wire x1="-49.87" y1="55.88" x2="-43.16" y2="78.42" width="0" layer="19" extent="1-1"/>
+<wire x1="-49.87" y1="55.88" x2="88.9" y2="85.72" width="0" layer="19" extent="1-1"/>
+<wire x1="67.33" y1="65.72" x2="-49.87" y2="55.88" width="0" layer="19" extent="1-1"/>
 </signal>
 <signal name="N$13">
-<contactref element="U2" pad="3"/>
 <contactref element="R12" pad="2"/>
 <contactref element="R17" pad="2"/>
-<wire x1="-43.16" y1="76.52" x2="55.46" y2="82.55" width="0" layer="19" extent="1-1"/>
-<wire x1="-41.91" y1="45.72" x2="-43.16" y2="76.52" width="0" layer="19" extent="1-1"/>
+<contactref element="U2" pad="3"/>
+<wire x1="-41.91" y1="45.72" x2="55.46" y2="82.55" width="0" layer="19" extent="1-1"/>
+<wire x1="67.33" y1="63.82" x2="-41.91" y2="45.72" width="0" layer="19" extent="1-1"/>
 </signal>
 <signal name="12V">
@@
 <contactref element="C3" pad="1"/>
 <contactref element="U$2" pad="1"/>
+<contactref element="U$7" pad="1"/>
 <contactref element="U2" pad="5"/>
 <contactref element="U2" pad="4"/>
-<contactref element="U$7" pad="1"/>
 <wire x1="74.67" y1="95.25" x2="88.9" y2="94.62" width="0" layer="19" extent="1-1"/>
 <wire x1="55.03" y1="86.36" x2="74.67" y2="95.25" width="0" layer="19" extent="1-1"/>
-<wire x1="-40.66" y1="77.47" x2="55.03" y2="86.36" width="0" layer="19" extent="1-1"/>
-<wire x1="-40.66" y1="76.52" x2="-40.66" y2="77.47" width="0" layer="19" extent="1-1"/>
+<wire x1="69.83" y1="64.77" x2="55.03" y2="86.36" width="0" layer="19" extent="1-1"/>
+<wire x1="69.83" y1="63.82" x2="69.83" y2="64.77" width="0" layer="19" extent="1-1"/>
 </signal>
 </signals>

Commit message: motherBoard
Parts:
- removed J10: 640456-5, 640456-5:TE_640456-5
- removed J11, J8: 640456-2, 640456-2:TE_640456-2
- removed J7: (no value), SparkFun-Connectors:1X06
- removed J9: 640456-3, 640456-3:CONN_640456-3
- added BLUE: 640456-5, 640456-5:TE_640456-5
- added PIC: (no value), SparkFun-Connectors:1X06
- added SOLENOID, TSTSPPLY: 640456-2, 640456-2:TE_640456-2
- added TEMP: 640456-3, 640456-3:CONN_640456-3
- moved R18 147.0 mm to (97.8, 50.8), turned to 270 degrees
- moved R22 144.5 mm to (78.7, 45.7)
- moved C10 141.2 mm to (68.6, 57.1)
- moved D4 141.2 mm to (87.6, 76.2)
- moved C7 139.7 mm to (78.7, 58.4), turned to 90 degrees
- moved C8 137.5 mm to (68.6, 39.4)
- moved R21 123.3 mm to (54.6, 30.5)
- moved D3 121.3 mm to (40.6, 35.6)
- moved U3 116.6 mm to (53.3, 54.6)
- moved R26 115.2 mm to (21.6, 21.6)
- moved R19 113.1 mm to (49.5, 27.9), turned to 90 degrees
- moved 10UH 111.1 mm to (53.3, 59.7), turned to 180 degrees
- moved D5 110.8 mm to (52.1, 36.8)
- moved Q4 105.4 mm to (41.9, 27.9)
- moved R12 102.9 mm to (54.6, 73.7)
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Connections:
- net 3.3V: now also BLUE.2, PIC.2; no longer J10.2, J7.2
- net BLUETOOTH_ON/OFF: now also BLUE.5; no longer J10.5
- net DRIVER: now also SOLENOID.1; no longer J8.1
- net GND: now also BLUE.1, PIC.3, SOLENOID.2, TEMP.3, TSTSPPLY.1; no longer J10.1, J11.1, J7.3, J8.2, J9.3
- net LVP: now also PIC.6; no longer J7.6
- net MCLR: now also PIC.1; no longer J7.1
- net PGC: now also PIC.5; no longer J7.5
- net PGD: now also PIC.4; no longer J7.4
- net RX: now also BLUE.3; no longer J10.3
- net TEMP_DQ: now also TEMP.2; no longer J9.2
- net TX: now also BLUE.4; no longer J10.4
- net VCC: now also TEMP.1, TSTSPPLY.2; no longer J11.2, J9.1
Other:
- board size 160 x 100 mm -> 158.7 x 100 mm

Commit message: Update motherBoard.brd
Parts:
- moved U$6 115.6 mm to (15.2, 26.7)
- moved U$5 114.9 mm to (15.2, 36.8)
- moved R22 80.7 mm to (2.54, 19.1)
- moved PIC 70.9 mm to (57.1, 5.08), turned to 180 degrees
- moved TSTSPPLY 61.0 mm to (72.4, 43.2), turned to 270 degrees
- moved BLUE 60.2 mm to (72.4, 24.1)
- moved R27 58.4 mm to (53.3, 14.0)
- moved R18 57.5 mm to (48.3, 21.6), turned to 180 degrees
- moved U$7 56.9 mm to (35.6, 43.2), turned to 270 degrees
- moved C10 47.8 mm to (59.7, 10.2)
- moved C9 44.5 mm to (15.2, 53.3)
- moved R13 44.5 mm to (19.1, 49.5), turned to 0 degrees
- moved U$2 44.5 mm to (62.2, 54.6), turned to 180 degrees
- moved U1 44.5 mm to (14.0, 49.5)
- moved C3 44.4 mm to (45.7, 43.2), turned to 270 degrees
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Other:
- board size 158.7 x 100 mm -> 78.7 x 61.9 mm

Commit message: motherBoard
Parts:
- removed GLED: (no value), led:LED5MM
- added D2: Green, SparkFun:LED-0603
- moved C12 1.27 mm to (8.89, 48.3)
- moved R13 1.27 mm to (19.1, 48.3)
- moved R14 1.27 mm to (20.3, 52.1)
- moved S1 1.27 mm to (14.0, 59.7)
Connections:
- removed net N$2: GLED.K, R14.2
- new net N$1: D2.C, R14.2
- net N$11: now also D2.A; no longer GLED.A

Commit message: Update motherBoard.brd
Parts:
- moved Q3 31.4 mm to (7.62, 2.54)
- moved U$2 26.7 mm to (38.1, 43.2), turned to 270 degrees
- moved C3 19.9 mm to (63.5, 34.3)
- moved C5 19.9 mm to (59.7, 34.3)
- moved R12 19.2 mm to (63.5, 54.6)
- moved TSTSPPLY 18.8 mm to (63.5, 26.7)
- moved R17 17.6 mm to (57.1, 39.4)
- moved BLUE 17.6 mm to (63.5, 8.89)
- moved U2 17.6 mm to (62.2, 39.4)
- moved D4 15.5 mm to (50.8, 41.9)
- moved R19 14.2 mm to (29.2, 27.9)
- moved S3 12.5 mm to (48.3, 34.3)
- moved U$7 12.5 mm to (40.6, 54.6), turned to 0 degrees
- moved C13 11.7 mm to (41.9, 22.9)
- moved C15 11.7 mm to (41.9, 15.2)
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Other:
- board size 78.7 x 61.9 mm -> 68.6 x 59.4 mm

Commit message: motherBoard
Parts:
- moved Q3 44.1 mm to (36.8, 35.6), turned to 180 degrees
- moved C3 43.8 mm to (25.4, 55.9)
- moved U2 36.9 mm to (29.2, 55.9)
- moved C5 34.3 mm to (33.0, 55.9)
- moved R20 33.4 mm to (31.8, 40.6), turned to 90 degrees
- moved C7 33.0 mm to (21.6, 31.8), flipped to the bottom
- moved C13 31.4 mm to (11.4, 30.5), flipped to the bottom, turned to 90 degrees
- moved Y2 29.6 mm to (34.3, 19.1), flipped to the bottom
- moved R17 26.2 mm to (36.8, 55.9), turned to 270 degrees
- moved U3 25.4 mm to (16.5, 30.5), flipped to the bottom
- moved 10UH 24.5 mm to (16.5, 26.7), flipped to the bottom
- moved R16 22.6 mm to (24.1, 40.6), turned to 0 degrees
- moved D4 21.7 mm to (30.5, 49.5), turned to 180 degrees
- moved C10 18.2 mm to (31.8, 15.2), turned to 270 degrees
- moved U$8 17.3 mm to (34.3, 27.9)
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Connections:
- removed net LVP: PIC.6
- removed net N$26: R25.1, S3.3, U$8.1
- net 3.3V: now also U3.3
- net MCLR: now also R25.1, S3.3, U$8.1
- net PGC: now also U$8.27
- net PGD: now also U$8.28
Other:
- board size 68.6 x 59.4 mm -> 59.7 x 59.4 mm

Commit message: motherBoard
Parts:
- removed R13: 2k, SparkFun-Resistors:0805
- added R1: 2k, SparkFun-Resistors:0603
- moved R27 20.1 mm to (45.6, 28.7)
- moved R19 16.7 mm to (45.7, 43.2), turned to 90 degrees
- moved R14 13.3 mm to (7.62, 40.6), turned to 180 degrees
- moved C14 12.7 mm to (12.7, 14.0), flipped to the bottom, turned to 180 degrees
- moved R28 11.7 mm to (17.8, 14.0), flipped to the bottom, turned to 180 degrees
- moved Q3 11.7 mm to (27.9, 43.2), turned to 0 degrees
- moved R21 11.5 mm to (17.8, 17.8), flipped to the bottom, turned to 0 degrees
- moved D5 9.25 mm to (20.3, 8.89)
- moved R22 9.16 mm to (12.7, 17.8), flipped to the bottom, turned to 180 degrees
- moved C12 8.52 mm to (2.54, 36.8)
- moved R16 8.52 mm to (16.5, 44.5)
- moved R18 7.73 mm to (45.7, 38.1)
- moved C9 7.18 mm to (11.4, 44.5)
- moved C10 5.68 mm to (34.3, 10.2), flipped to the bottom
- moved C8 5.68 mm to (39.4, 10.2), flipped to the bottom
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Connections:
- net N$9: now also R1.2; no longer R13.2
- net _12V: now also R1.1; no longer R13.1

Commit message: motherBoard V1
Parts:
- removed BLED4, BLED5, BLED6, RLED4, RLED5, RLED6: (no value), led:LED5MM
- added D1, D6: CLX6F-FKC-CKNNQDGBB7A363, CLX6F-LED:SOJ100P350X290-6N
- R23: value 47 -> 20
- R24: value 1 -> 5
- moved R24 111.4 mm to (40.6, 30.5), turned to 90 degrees
- moved R23 78.5 mm to (19.1, 30.5), turned to 90 degrees
- moved D3 16.5 mm to (21.6, 2.54)
- moved C11 7.73 mm to (19.1, 49.5), turned to 90 degrees
- moved C12 7.41 mm to (8.89, 40.6), turned to 90 degrees
- moved C15 6.48 mm to (41.9, 20.3)
- moved U$8 6.35 mm to (34.3, 20.3)
- moved D2 6.35 mm to (15.2, 44.5), turned to 0 degrees
- moved R14 5.39 mm to (11.4, 44.5), turned to 90 degrees
- moved U$4 5.24 mm to (20.3, 39.4), turned to 0 degrees
- moved C9 5.08 mm to (11.4, 49.5), turned to 270 degrees
- moved TEMP 4.02 mm to (2.54, 12.7)
- moved BATT 3.81 mm to (3.81, 35.6)
- moved U$5 3.81 mm to (15.2, 22.9)
- moved S1 3.59 mm to (16.5, 57.1)
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Connections:
- net BLUE_LEDS: now also D6.4, D6.5, D6.6; no longer BLED4.A, BLED5.A, BLED6.A
- net N$24: now also D6.1, D6.2, D6.3; no longer BLED4.K, BLED5.K, BLED6.K
- net N$25: now also D1.1, D1.2, D1.3; no longer RLED4.K, RLED5.K, RLED6.K
- net RED_LEDS: now also D1.4, D1.5, D1.6; no longer RLED4.A, RLED5.A, RLED6.A
Other:
- board size 59.7 x 59.4 mm -> 60 x 60 mm
