File: eagle/projects/smartBobber Mother Board/motherBoard/motherBoard.brd (EAGLE design)
At the start: 60 x 60 mm, 57 parts, among them J1 10118193-0001LF, Q3 2A/20V/150mΩ, Q4 MMBT3904, U1 MCP73831, U2 MT3608, U3 LTC3531ES6-3_3, Y2 ECS-40-S-4X

Commit message: Update motherBoard.brd
Parts:
- moved R19 76.0 mm to (-25.4, 16.5), turned to 270 degrees
- moved R18 73.3 mm to (-25.4, 20.3), turned to 0 degrees
- moved R27 70.8 mm to (-20.4, 3.30)
- moved C15 70.8 mm to (-24.1, -5.08)
- moved R25 70.8 mm to (-20.3, 7.62)
- moved R26 70.8 mm to (-20.3, -1.27)
- moved Q4 64.2 mm to (-19.1, 16.5), turned to 270 degrees
- moved C14 63.5 mm to (76.2, 14.0), flipped to the top
- moved R21 63.5 mm to (81.3, 19.1), flipped to the top
- moved R22 63.5 mm to (76.2, 19.1), flipped to the top
- moved R28 63.5 mm to (81.3, 14.0), flipped to the top
- moved D5 55.9 mm to (78.7, 8.89)
- moved D3 54.6 mm to (76.2, 3.81)
- moved R20 52.9 mm to (-12.7, 16.5), turned to 90 degrees
- moved 10UH 50.4 mm to (57.1, 49.5), flipped to the top, turned to 270 degrees
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
Commit message: Bullshit
Parts:
- added U$1: 12V-BOARD, 12V-Board:PERF_BOARD
Connections:
- removed net N$21: C3.1, U$2.1, U$7.1, U2.4, U2.5
- new net N$2: C3.1, U$1.VIN+, U$2.1, U$7.1, U2.4, U2.5
- net 12V: now also U$1.VOUT+
- net GND: now also C13.2, C3.2, C5.2, C7.2, R16.1, R17.1, U$1.VIN-, U$1.VOUT-, U$4.3, U$6.-, U2.2, U3.2
- net _12V: no longer C13.2, C3.2, C5.2, C7.2, R16.1, R17.1, U$4.3, U$6.-, U2.2, U3.2

Commit message: Update motherBoard.brd
Parts:
- moved C15 69.6 mm to (43.2, 12.7), turned to 270 degrees
- moved R18 66.7 mm to (38.1, 40.6), flipped to the bottom, turned to 90 degrees
- moved D3 64.1 mm to (26.7, 44.5), turned to 270 degrees
- moved R19 62.5 mm to (31.8, 41.9), flipped to the bottom, turned to 180 degrees
- moved Q4 61.4 mm to (34.3, 47.0), flipped to the bottom, turned to 0 degrees
- moved TEMP 61.3 mm to (57.1, 40.6), flipped to the top
- moved SOLENOID 59.6 mm to (57.1, 50.8), flipped to the top, turned to 270 degrees
- moved R20 58.9 mm to (34.3, 52.1), flipped to the bottom
- moved D5 57.4 mm to (26.7, 33.0), turned to 90 degrees
- moved C14 53.6 mm to (44.5, 57.1), flipped to the bottom
- moved R22 53.0 mm to (39.4, 57.1), flipped to the bottom
- moved C3 52.8 mm to (2.54, 8.89), turned to 0 degrees
- moved R21 52.6 mm to (31.8, 36.8), flipped to the bottom
- moved R28 52.6 mm to (31.8, 31.8), flipped to the bottom
- moved U2 51.4 mm to (2.54, 12.7), turned to 90 degrees
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
Commit message: Led Part and Board Update
Parts:
- removed D1, D6: CLX6F-FKC-CKNNQDGBB7A363, CLX6F-LED:SOJ100P350X290-6N
- removed R23: 20, SparkFun-Resistors:0603
- added R2: 5, SparkFun-Resistors:0603
- added R3, R4: 20, SparkFun-Resistors:0603
- added U$10, U$9: CLX6F-BKB-CPR453, CLX6F-LED:SOJ100P350X290-6N
- added U$11, U$12: CLX6F-RKB-CSTBB3, CLX6F-LED:SOJ100P350X290-6N
- moved R24 23.2 mm to (53.3, 31.8), turned to 90 degrees
- moved S3 5.68 mm to (45.7, 19.1)
- moved C15 1.27 mm to (41.9, 12.7)
- moved U$1 1.27 mm to (15.2, 17.8)
- moved C12 1.27 mm to (8.89, 40.6)
- moved BATT 0.74 mm to (3.17, 37.7)
- turned D2 to 180 degrees
- turned D5 to 270 degrees
- turned R16 to 90 degrees
Connections:
- removed net BLUE_LEDS: D6.4, D6.5, D6.6, U$8.15
- removed net N$24: D6.1, D6.2, D6.3, R24.2
- removed net RED_LEDS: D1.4, D1.5, D1.6, U$8.16
- new net BLUE_LEDS_1: U$8.15, U$9.4, U$9.5, U$9.6
- new net BLUE_LEDS_2: U$10.4, U$10.5, U$10.6, U$8.3
- new net N$21: R24.2, U$10.1, U$10.2, U$10.3
- new net N$3: R2.2, U$9.1, U$9.2, U$9.3
- new net N$5: R3.2, U$12.1, U$12.2, U$12.3
- new net RED_LEDS_1: U$12.4, U$12.5, U$12.6, U$8.16
- new net RED_LEDS_2: U$11.4, U$11.5, U$11.6, U$8.4
- net GND: now also R2.1, R3.1, R4.1; no longer R23.1
- net N$25: now also R4.2, U$11.1, U$11.2, U$11.3; no longer D1.1, D1.2, D1.3, R23.2

Commit message: Schematic Update
Connections:
- net N$16 renamed LOAD
- net N$8 renamed BATT+
- new net N$4: U$1.VIN-, U$1.VOUT-
- net GND: no longer U$1.VIN-, U$1.VOUT-

Commit message: update schematic and board
Parts:
- moved S1 16.6 mm to (2.41, 48.4), turned to 270 degrees
- moved U$3 14.2 mm to (10.2, 39.4), turned to 0 degrees
- moved J1 13.9 mm to (16.4, 56.4), turned to 180 degrees
- moved C12 6.84 mm to (11.4, 47.0)
- moved R1 6.48 mm to (10.2, 50.8), turned to 180 degrees
- moved R15 6.35 mm to (19.1, 45.7), turned to 90 degrees
- moved C9 4.58 mm to (8.89, 54.6)
- moved C11 3.81 mm to (17.8, 50.8), turned to 180 degrees
- moved R16 2.84 mm to (16.5, 47.0)
- moved R14 2.54 mm to (8.89, 45.7)
- moved U$4 2.54 mm to (21.6, 40.6), turned to 90 degrees
- moved U1 1.80 mm to (15.2, 39.4), turned to 180 degrees
- moved R4 1.27 mm to (33.0, 2.54)
- moved D2 1.27 mm to (14.0, 45.7)
- moved U$11 1.27 mm to (27.9, 3.81)
Connections:
- new net GND1: BATT.2, C12.2, U$3.6, U$4.1
- net _12V: no longer BATT.2, C12.2, U$3.6, U$4.1

Commit message: Update motherBoard.brd
Parts:
- moved D3 23.6 mm to (45.1, 29.7), turned to 0 degrees
- moved D5 17.9 mm to (44.6, 32.8), turned to 0 degrees
- moved R1 15.5 mm to (19.1, 38.1)
- moved Y2 12.5 mm to (46.4, 19.4)
- moved U$3 10.5 mm to (20.3, 41.9)
- moved S3 10.3 mm to (47.5, 8.89)
- moved C11 7.18 mm to (22.9, 55.9), turned to 90 degrees
- moved U1 5.08 mm to (10.2, 39.4), turned to 270 degrees
- moved U$8 4.58 mm to (30.0, 16.2)
- moved R16 4.58 mm to (19.1, 50.8)
- moved C8 4.10 mm to (43.9, 23.1)
- moved R15 4.02 mm to (22.9, 47.0)
- moved C12 3.81 mm to (11.4, 50.8)
- moved C10 3.75 mm to (48.8, 23.4)
- moved U$4 2.54 mm to (24.1, 40.6)
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