File: eagle/projects/smartBobber Mother Board/motherBoard/motherBoard.brd (EAGLE design)
At the start: 60 x 60 mm, 62 parts, among them J1 10118193-0001LF, Q3 2A/20V/150mΩ, Q4 MMBT3904, U1 MCP73831, U2 MT3608, U3 LTC3531ES6-3_3, Y2 ECS-40-S-4X

Commit message: Update motherBoard.brd
Parts:
- moved R28 7.18 mm to (26.7, 36.8)
Changed lines of the file:
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@@
 <?xml version="1.0" encoding="utf-8"?>
 <!DOCTYPE eagle SYSTEM "eagle.dtd">
-<eagle version="9.3.1">
+<eagle version="9.3.0">
 <drawing>
 <settings>
-<setting alwaysvectorfont="yes"/>
+<setting alwaysvectorfont="no"/>
 <setting verticaltext="up"/>
 </settings>
-<grid distance="50" unitdist="mil" unit="mil" style="lines" multiple="1" display="yes" altdistance="0.5" altunitdist="mm" altunit="mm"/>
+<grid distance="50" unitdist="mil" unit="mm" style="lines" multiple="1" display="yes" altdistance="0.5" altunitdist="mm" altunit="mm"/>
 <layers>
 <layer number="1" name="Top" color="4" fill="1" visible="yes" active="yes"/>
@@
 <attribute name="VALUE" x="17.653" y="11.684" size="0.6096" layer="27" font="vector" ratio="20" rot="R180" align="top-center"/>
 </element>
-<element name="R28" library="SparkFun-Resistors" package="0603" value=" 100k" x="31.75" y="31.75" smashed="yes" rot="MR180">
-<attribute name="NAME" x="31.75" y="30.988" size="0.6096" layer="26" font="vector" ratio="20" rot="MR180" align="bottom-center"/>
-<attribute name="PROD_ID" value=" " x="50.8" y="118.11" size="1.778" layer="28" rot="MR180" display="off"/>
-<attribute name="VALUE" x="31.75" y="32.512" size="0.6096" layer="28" font="vector" ratio="20" rot="MR180" align="top-center"/>
+<element name="R28" library="SparkFun-Resistors" package="0603" value=" 100k" x="26.67" y="36.83" smashed="yes" rot="MR180">
+<attribute name="NAME" x="26.67" y="36.068" size="0.6096" layer="26" font="vector" ratio="20" rot="MR180" align="bottom-center"/>
+<attribute name="PROD_ID" value=" " x="45.72" y="123.19" size="1.778" layer="28" rot="MR180" display="off"/>
+<attribute name="VALUE" x="26.67" y="37.592" size="0.6096" layer="28" font="vector" ratio="20" rot="MR180" align="top-center"/>
 </element>
 <element name="S1" library="JS102011SAQN" package="SW_JS102011SAQN" value="JS102011SAQN" x="2.413" y="48.387" smashed="yes" rot="R270">
@@
 <contactref element="R28" pad="2"/>
 <wire x1="30.9" y1="36.83" x2="43.6" y2="57.15" width="0" layer="19" extent="16-16"/>
-<wire x1="30.9" y1="31.75" x2="30.9" y2="36.83" width="0" layer="19" extent="16-16"/>
-<wire x1="32.6" y1="31.75" x2="30.9" y2="31.75" width="0" layer="19" extent="16-16"/>
-<wire x1="40.767" y1="32.766" x2="32.6" y2="31.75" width="0" layer="19" extent="16-16"/>
-<wire x1="26.4186" y1="19.7714" x2="30.9" y2="31.75" width="0" layer="19" extent="1-16"/>
+<wire x1="25.82" y1="36.83" x2="30.9" y2="36.83" width="0" layer="19" extent="16-16"/>
+<wire x1="27.52" y1="36.83" x2="25.82" y2="36.83" width="0" layer="19" extent="16-16"/>
+<wire x1="40.767" y1="32.766" x2="27.52" y2="36.83" width="0" layer="19" extent="16-16"/>
+<wire x1="26.4186" y1="19.7714" x2="25.82" y2="36.83" width="0" layer="19" extent="1-16"/>
 </signal>
 <signal name="SOLENOID_ON/OFF">

Commit message: Update motherBoard.brd
Parts:
- moved C12 12.0 mm to (22.9, 47.0)
- moved C9 10.2 mm to (11.4, 45.7)
- moved R16 7.41 mm to (15.2, 44.5), turned to 0 degrees
- moved R14 5.08 mm to (8.89, 52.1)
- moved D2 4.58 mm to (11.4, 49.5), turned to 0 degrees
- moved C11 3.81 mm to (22.9, 52.1)
- moved R15 3.81 mm to (19.1, 47.0), turned to 270 degrees
- moved U$2 1.95 mm to (11.4, 14.0)
- moved C3 1.27 mm to (3.81, 8.89)
- moved C5 1.27 mm to (3.81, 16.5), turned to 180 degrees
- moved R17 1.27 mm to (3.81, 19.1), turned to 180 degrees
- moved U2 1.27 mm to (3.81, 12.7), turned to 270 degrees
- moved R25 1.27 mm to (19.1, 15.2)
- moved R26 1.27 mm to (19.1, 6.35)
- moved R27 1.27 mm to (18.9, 10.9)
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Routing:
- net N$2: track 0.00 -> 66.6 mm
- net BATT+: track 0.00 -> 50.1 mm, vias 0 -> 2
- net LOAD: track 0.00 -> 44.7 mm, vias 0 -> 1
- net _12V: track 0.00 -> 40.1 mm
- net 12V: track 0.00 -> 20.9 mm
- net N$13: track 0.00 -> 14.3 mm
- net N$12: track 0.00 -> 13.8 mm, vias 0 -> 2
- net N$11: track 0.00 -> 13.0 mm, vias 0 -> 2
- net N$7: track 0.00 -> 10.9 mm
- net N$18: track 0.00 -> 10.6 mm
- net N$9: track 0.00 -> 9.36 mm
- net N$20: track 0.00 -> 8.78 mm
- net N$17: track 0.00 -> 6.45 mm
- net N$1: track 0.00 -> 4.68 mm
- net N$10: track 0.00 -> 4.68 mm

Commit message: boad update
Parts:
- added TP1, TP10, TP11, TP12, TP2, TP3, TP4, TP5, TP6, TP7, TP8, TP9: TEST-POINTPOGO_PTH, SparkFun-Connectors:1X01_NO_SILK
- moved R26 50.3 mm to (53.3, 43.2), flipped to the bottom, turned to 270 degrees
- moved R27 34.5 mm to (50.8, 24.1), flipped to the bottom, turned to 270 degrees
- moved C14 28.5 mm to (29.2, 33.0), turned to 270 degrees
- moved R25 21.9 mm to (40.6, 11.4), flipped to the bottom, turned to 90 degrees
- moved 10UH 8.89 mm to (45.7, 52.1)
- moved C15 4.02 mm to (40.6, 16.5), flipped to the bottom, turned to 180 degrees
- moved C10 1.93 mm to (47.0, 24.1)
- moved R22 1.80 mm to (38.1, 55.9), turned to 270 degrees
- moved R18 1.27 mm to (36.8, 40.6), turned to 180 degrees
- moved C8 1.27 mm to (43.2, 24.1)
- moved Y2 0.74 mm to (45.7, 19.1)
- moved D3 0.25 mm to (45.1, 30.0), turned to 180 degrees
- turned R3 to 180 degrees
- turned U$6 to 270 degrees
Connections:
- removed net N$4: U$1.VIN-, U$1.VOUT-
- removed net VCC: Q3.S1, R20.1, R26.1, TEMP.1, TSTSPPLY.2
- net 12V: now also Q3.S1, R20.1, TP4.1
- net 3.3V: now also R26.1, TEMP.1, TP6.1, TSTSPPLY.2
- net ADC: now also TP12.1
- net BATT+: now also TP1.1, TP9.1
- net GND: now also TP5.1, U$1.VIN-, U$1.VOUT-
- net GND1: now also TP2.1
- net LOAD: now also TP3.1
- net N$11: now also TP10.1
- net N$17: now also TP8.1
- net N$18: now also TP7.1
- net PWM: now also TP11.1
- net RX: now also BLUE.4; no longer BLUE.3
- net TX: now also BLUE.3; no longer BLUE.4
Routing:
- net 3.3V: track 0.00 -> 120.5 mm, vias 0 -> 1
- net 12V: track 20.9 -> 101.7 mm, vias 0 -> 3
- net PWM: track 0.00 -> 63.5 mm, vias 0 -> 3
- net DRIVER: track 0.00 -> 60.8 mm
- net TEMP_DQ: track 0.00 -> 60.5 mm, vias 0 -> 2
- net BLUE_LEDS_1: track 0.00 -> 56.2 mm, vias 0 -> 4
- net RED_LEDS_1: track 0.00 -> 54.1 mm, vias 0 -> 4
- net SOLENOID_ON/OFF: track 0.00 -> 52.7 mm, vias 0 -> 5
- net MCLR: track 0.00 -> 40.0 mm, vias 0 -> 2
- net BLUE_LEDS_2: track 0.00 -> 39.0 mm, vias 0 -> 2
- net OSC2: track 0.00 -> 33.8 mm
- net PGD: track 0.00 -> 32.2 mm
- net BLUETOOTH_ON/OFF: track 0.00 -> 31.2 mm
- net LOAD: track 44.7 -> 74.5 mm
- net ADC: track 0.00 -> 29.3 mm, vias 0 -> 1
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
Commit message: Update motherBoard.brd
Parts:
- moved TP10 92.7 mm to (22.9, 57.1)
- moved TP12 92.5 mm to (27.9, 23.3)
- moved TP11 77.1 mm to (19.1, 14.0)
- moved TP8 74.7 mm to (19.1, 45.7)
- moved TP9 72.6 mm to (14.0, 41.9)
- moved TP5 70.3 mm to (39.4, 26.7)
- moved TP6 69.5 mm to (37.5, 8.13)
- moved TP7 66.2 mm to (19.1, 38.1)
- moved TP3 59.1 mm to (36.8, 27.9)
- moved TP2 58.3 mm to (8.89, 57.1)
- moved TP4 53.9 mm to (15.2, 33.0)
- moved TP1 49.9 mm to (6.35, 54.6)
- moved R1 3.81 mm to (15.2, 38.1), turned to 90 degrees
- moved R15 2.54 mm to (19.1, 49.5)
Routing:
- net 12V: track 101.7 -> 114.7 mm
- net 3.3V: track 120.5 -> 133.3 mm
- net BATT+: track 50.1 -> 56.9 mm
- net N$11: track 13.0 -> 18.9 mm
- net N$9: track 9.36 -> 4.35 mm
- net _12V: track 40.1 -> 36.7 mm
- net MCLR: track 40.0 -> 43.1 mm
- net N$17: track 6.45 -> 9.35 mm
- net ADC: track 29.3 -> 32.0 mm
- net PWM: track 63.5 -> 66.1 mm
- net N$18: track 10.6 -> 13.1 mm
- net LOAD: track 74.5 -> 76.2 mm
- net N$20: track 8.78 -> 9.83 mm
- net PGC: track 23.3 -> 23.9 mm

Commit message: Update
Parts:
- moved R28 8.98 mm to (27.9, 45.7)
- moved R21 7.41 mm to (27.9, 43.2), turned to 180 degrees
- moved TP5 1.27 mm to (40.6, 26.7)
- renumbered BLUE to BLUETOOTH
Routing:
- net ADC: track 32.0 -> 45.9 mm

Commit message: CRAZY UPDATE
Parts:
- moved TP3 24.4 mm to (25.4, 49.5)
- moved R22 16.3 mm to (25.4, 45.7)
- moved R28 14.5 mm to (31.8, 31.8), turned to 270 degrees
- moved R21 14.5 mm to (36.8, 31.8), turned to 90 degrees
- moved TP5 12.6 mm to (49.5, 17.8)
- moved R20 11.4 mm to (29.2, 41.9), turned to 180 degrees
- moved Q3 6.48 mm to (29.2, 45.7)
- moved Q4 6.35 mm to (34.3, 40.6)
- moved TP9 5.39 mm to (10.2, 38.1)
- moved C14 5.24 mm to (34.3, 31.8)
- moved R18 5.08 mm to (36.8, 35.6), turned to 0 degrees
- moved R19 5.08 mm to (31.8, 35.6), turned to 0 degrees
- moved Y2 4.58 mm to (43.2, 22.9)
- moved C10 4.02 mm to (45.7, 27.9)
- moved C8 3.81 mm to (43.2, 27.9)
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- renumbered SOLENOID to DRIVER
Connections:
- new net N$4: C14.1, D5.C, R21.2, R28.1
- net ADC: no longer C14.1, D5.C, R21.2, R28.1
Routing:
- net ADC: track 45.9 -> 86.4 mm, vias 1 -> 0
- net N$2: track 80.0 -> 57.0 mm
- net LOAD: track 76.2 -> 56.9 mm
- net PWM: track 66.1 -> 53.0 mm, vias 3 -> 1
- net N$4: track 0.00 -> 8.94 mm
- net DRIVER: track 60.8 -> 68.3 mm
- net SOLENOID_ON/OFF: track 52.7 -> 46.3 mm, vias 5 -> 1
- net N$22: track 13.4 -> 7.67 mm
- net N$23: track 5.19 -> 10.5 mm
- net _12V: track 36.7 -> 32.2 mm
- net 3.3V: track 133.1 -> 128.8 mm
- net N$7: track 10.9 -> 7.10 mm
- net N$9: track 4.35 -> 7.59 mm
- net N$18: track 12.8 -> 10.5 mm
- net TEMP_DQ: track 60.5 -> 62.7 mm
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- added copper zone on layer 1, net GND
- added copper zone on layer 16, net GND
- added copper zone on layer 1, net GND1
- added copper zone on layer 16, net GND1
Other:
- board text added: "+"
- board text added: "+12V"
- board text added: "-"
- board text added: "3.3V"
- board text added: "DQ"
- board text added: "GND"
- board text added: "MCLR"
- board text added: "ON/OFF"
- board text added: "PGC"
- board text added: "PGD"
- board text added: "PICKIT"
- board text added: "RX"
- board text added: "TX"

Commit message: Update motherBoard.brd
Routing:
- net N$14: track 0.00 -> 2.97 mm
- net N$11: track 16.7 -> 17.9 mm
- net LOAD: track 56.9 -> 58.2 mm
- net ADC: track 86.4 -> 87.6 mm, vias 0 -> 1
Changed lines of the file:
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@@
 <wire x1="50.3428" y1="35.74938125" x2="50.3428" y2="29.39938125" width="0.3048" layer="1"/>
 <wire x1="50.3428" y1="29.39938125" x2="49.34061875" y2="28.3972" width="0.3048" layer="1"/>
-<wire x1="49.34061875" y1="28.3972" x2="33.8328" y2="28.3972" width="0.3048" layer="1"/>
-<wire x1="33.8328" y1="28.3972" x2="31.75" y2="30.48" width="0.3048" layer="1"/>
+<wire x1="49.34061875" y1="28.3972" x2="34.29" y2="28.3972" width="0.3048" layer="1"/>
+<wire x1="34.29" y1="28.3972" x2="33.8328" y2="28.3972" width="0.3048" layer="1"/>
 <wire x1="49.71938125" y1="27.4828" x2="51.2572" y2="29.02061875" width="0.3048" layer="1"/>
 <wire x1="36.3728" y1="27.4828" x2="49.71938125" y2="27.4828" width="0.3048" layer="1"/>
@@
 <wire x1="27.9146" y1="23.3426" x2="27.94" y2="23.3172" width="0.3048" layer="1"/>
 <wire x1="27.94" y1="23.3172" x2="27.94" y2="21.971" width="0.3048" layer="1"/>
-<wire x1="31.75" y1="30.48" x2="31.75" y2="30.9" width="0" layer="19" extent="1-16"/>
+<wire x1="33.8328" y1="28.3972" x2="32.5628" y2="28.3972" width="0.3048" layer="1"/>
+<wire x1="32.5628" y1="28.3972" x2="31.75" y2="29.21" width="0.3048" layer="1"/>
+<wire x1="31.75" y1="29.21" x2="31.75" y2="29.3243" width="0.3048" layer="1"/>
+<via x="31.75" y="29.3243" extent="1-16" drill="0.508"/>
+<wire x1="31.75" y1="29.3243" x2="31.75" y2="30.9" width="0.3048" layer="16"/>
 </signal>
 <signal name="SOLENOID_ON/OFF">
@@
 <wire x1="1.54" y1="34.57" x2="2.54" y2="34.57" width="0.3048" layer="1"/>
 <wire x1="2.54" y1="34.57" x2="3.54" y2="34.57" width="0.3048" layer="1"/>
-<wire x1="3.54" y1="34.57" x2="5.08" y2="35.56" width="0.3048" layer="1"/>
-<wire x1="5.08" y1="35.56" x2="22.86" y2="35.56" width="0.3048" layer="1"/>
-<wire x1="22.86" y1="35.56" x2="24.13" y2="34.29" width="0.3048" layer="1"/>
+<wire x1="3.54" y1="34.57" x2="4.52684375" y2="35.2044" width="0.3048" layer="1"/>
+<wire x1="4.52684375" y1="35.2044" x2="23.2156" y2="35.2044" width="0.3048" layer="1"/>
+<wire x1="23.2156" y1="35.2044" x2="24.13" y2="34.29" width="0.3048" layer="1"/>
 <via x="24.13" y="34.29" extent="1-16" drill="0.508"/>
 <via x="35.56" y="10.0432" extent="1-16" drill="0.508"/>
@@
 <wire x1="29.21" y1="55.87" x2="29.21" y2="49.53" width="0.3048" layer="1"/>
 <wire x1="29.21" y1="49.53" x2="27.94" y2="48.26" width="0.3048" layer="1"/>
-<wire x1="36.83" y1="27.94" x2="35.56" y2="29.21" width="0.3048" layer="16"/>
-<wire x1="35.56" y1="29.21" x2="30.48" y2="29.21" width="0.3048" layer="16"/>
+<wire x1="36.83" y1="27.94" x2="36.1315" y2="28.6385" width="0.3048" layer="16"/>
+<wire x1="36.1315" y1="28.6385" x2="31.0515" y2="28.6385" width="0.3048" layer="16"/>
 <wire x1="36.83" y1="12.5832" x2="36.83" y2="27.94" width="0.3048" layer="16"/>
-<wire x1="30.48" y1="29.21" x2="27.94" y2="31.75" width="0.3048" layer="16"/>
+<wire x1="31.0515" y1="28.6385" x2="27.94" y2="31.75" width="0.3048" layer="16"/>
 <wire x1="27.94" y1="31.75" x2="27.94" y2="36.83" width="0.3048" layer="16"/>
 <via x="27.94" y="36.83" extent="1-16" drill="0.508"/>
@@
 <contactref element="U1" pad="2"/>
 <wire x1="11.43" y1="47.41" x2="13.97" y2="49.95" width="0.6096" layer="1"/>
-<wire x1="13.97" y1="54.6" x2="14.1508" y2="54.7808" width="0.6096" layer="1"/>
-<wire x1="14.1508" y1="54.7808" x2="14.17238125" y2="54.7808" width="0.6096" layer="1"/>
-<wire x1="14.17238125" y1="54.7808" x2="15.0758" y2="55.68421875" width="0.6096" layer="1"/>
-<wire x1="15.0758" y1="55.68421875" x2="15.0758" y2="55.713" width="0.6096" layer="1"/>
 <wire x1="13.97" y1="49.95" x2="13.97" y2="52.07" width="0.6096" layer="1"/>
-<wire x1="13.97" y1="52.07" x2="13.97" y2="54.6" width="0.6096" layer="1"/>
 <wire x1="13.97" y1="52.07" x2="16.51" y2="52.07" width="0.6096" layer="1"/>
 <wire x1="16.51" y1="52.07" x2="17.78" y2="53.34" width="0.6096" layer="1"/>
@@
 <wire x1="9.9171" y1="44.2071" x2="9.9171" y2="42.69438125" width="0.6096" layer="1"/>
 <wire x1="11.43" y1="45.72" x2="9.9171" y2="44.2071" width="0.6096" layer="1"/>
-<wire x1="15.0758" y1="55.713" x2="15.083" y2="55.713" width="0" layer="19" extent="1-1"/>
+<wire x1="13.97" y1="52.07" x2="13.97" y2="54.61" width="0.6096" layer="1"/>
+<wire x1="13.98" y1="54.61" x2="14.00158125" y2="54.61" width="0.6096" layer="1"/>
+<wire x1="15.083" y1="55.713" x2="13.98" y2="54.61" width="0.6096" layer="1"/>
+<wire x1="13.98" y1="54.61" x2="13.97" y2="54.61" width="0.6096" layer="1"/>
 </signal>
 <signal name="N$20">
@@
 <wire x1="13.97" y1="53.34" x2="15.24" y2="53.34" width="0.6096" layer="16"/>
 <via x="15.24" y="53.34" extent="1-16" drill="0.35"/>
-<wire x1="17.6902" y1="54.84861875" x2="17.6902" y2="55.713" width="0.6096" layer="1"/>
-<wire x1="15.24" y1="53.34" x2="16.18158125" y2="53.34" width="0.6096" layer="1"/>
-<wire x1="16.18158125" y1="53.34" x2="17.6902" y2="54.84861875" width="0.6096" layer="1"/>
 <contactref element="TP10" pad="1"/>
-<wire x1="18.5036" y1="56.75373125" x2="18.66726875" y2="56.9174" width="0.254" layer="1"/>
-<wire x1="17.683" y1="55.713" x2="18.5036" y2="56.5336" width="0.254" layer="1"/>
-<wire x1="18.5036" y1="56.5336" x2="18.5036" y2="56.75373125" width="0.254" layer="1"/>
-<wire x1="22.6274" y1="56.9174" x2="22.86" y2="57.15" width="0.254" layer="1"/>
-<wire x1="18.66726875" y1="56.9174" x2="22.6274" y2="56.9174" width="0.254" layer="1"/>
-<wire x1="17.6902" y1="55.713" x2="17.683" y2="55.713" width="0" layer="19" extent="1-1"/>
+<wire x1="22.86" y1="57.15" x2="22.86" y2="55.88" width="0.3048" layer="1"/>
+<wire x1="22.86" y1="55.88" x2="21.59" y2="54.61" width="0.3048" layer="1"/>
+<wire x1="17.78" y1="54.61" x2="21.59" y2="54.61" width="0.3048" layer="1"/>
+<wire x1="16.51" y1="53.34" x2="17.78" y2="54.61" width="0.6096" layer="1"/>
+<wire x1="15.24" y1="53.34" x2="16.51" y2="53.34" width="0.6096" layer="1"/>
+<wire x1="17.683" y1="55.713" x2="17.78" y2="55.616" width="0.6096" layer="1"/>
+<wire x1="17.78" y1="55.616" x2="17.78" y2="54.61" width="0.6096" layer="1"/>
 <wire x1="11.4601" y1="42.23" x2="11.43" y2="49.11" width="0" layer="19" extent="1-1"/>
 </signal>
@@
 <contactref element="U3" pad="6"/>
 <contactref element="10UH" pad="1"/>
-<wire x1="44.577" y1="49.21" x2="44.845" y2="52.07" width="0" layer="19" extent="16-16"/>
+<wire x1="44.845" y1="52.07" x2="44.577" y2="51.802" width="0.6096" layer="16"/>
+<wire x1="44.577" y1="51.802" x2="44.577" y2="49.21" width="0.6096" layer="16"/>
 </signal>
 <signal name="N$15">
@@
 <wire x1="12.7" y1="48.26" x2="7.62" y2="48.26" width="0.6096" layer="16"/>
 <via x="7.62" y="48.26" extent="1-16" drill="0.508"/>
-<wire x1="7.62" y1="48.26" x2="6.35" y2="48.26" width="0.6096" layer="1"/>
 <wire x1="32.4993" y1="58.2997" x2="34.4103" y2="58.2997" width="0.6096" layer="16"/>
 <wire x1="34.4103" y1="58.2997" x2="38.1" y2="54.61" width="0.6096" layer="16"/>
@@
 <wire x1="24.13" y1="54.61" x2="24.13" y2="50.8" width="0.6096" layer="16"/>
 <wire x1="24.13" y1="50.8" x2="25.4" y2="49.53" width="0.6096" layer="16"/>
-<wire x1="6.35" y1="48.26" x2="5.163" y2="48.387" width="0" layer="19" extent="1-1"/>
+<wire x1="7.62" y1="48.26" x2="7.493" y2="48.387" width="0.6096" layer="1"/>
+<wire x1="7.493" y1="48.387" x2="5.163" y2="48.387" width="0.6096" layer="1"/>
 </signal>
 <signal name="N$7">
@@
 <vertex x="0" y="35.814"/>
 </polygon>
+<via x="10.16" y="54.61" extent="1-16" drill="0.508"/>
+<wire x1="21.42" y1="42.86" x2="22.86" y2="47.84" width="0" layer="19" extent="1-1"/>
+<wire x1="23.18" y1="37" x2="21.42" y2="42.86" width="0" layer="19" extent="1-1"/>
+<wire x1="10.16" y1="54.61" x2="22.86" y2="47.84" width="0" layer="19" extent="1-1"/>
+<wire x1="8.89" y1="57.15" x2="10.16" y2="54.61" width="0" layer="19" extent="1-1"/>
+<wire x1="3.175" y1="40.259" x2="10.16" y2="54.61" width="0" layer="19" extent="1-1"/>
 </signal>
 <signal name="N$4">

Commit message: fuck fuck fuck fuck fuck fuck
Parts:
- removed J1: 10118193-0001LF, 10118193-0001LF:FCI_10118193-0001LF
- added J2: 10118194-0001LF, 10118194-0001LF:AMPHENOL_10118194-0001LF
Connections:
- net N$11: now also J2.1; no longer J1.1
- net _12V: now also J2.5; no longer J1.5
Routing:
- net N$11: track 17.9 -> 18.9 mm
Changed lines of the file:
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@@
 <attribute name="VALUE" x="41.93868125" y="33.876090625" size="1.27166875" layer="27" ratio="10"/>
-</element>
-<element name="J1" library="10118193-0001LF" package="FCI_10118193-0001LF" value="10118193-0001LF" x="16.383" y="58.388" smashed="yes" rot="R180">
-<attribute name="DESCRIPTION" value=" Single Port 5 Contact Shielded SMT MICRO USB B-Type Receptacle " x="-33.147" y="81.248" size="1.778" layer="27" rot="R180" display="off"/>
-<attribute name="DIGI-KEY_PART_NUMBER" value="609-4616-1-ND" x="-33.147" y="81.248" size="1.778" layer="27" rot="R180" display="off"/>
-<attribute name="DIGI-KEY_PURCHASE_URL" value="https://www.digikey.com/product-detail/en/amphenol-icc-fci/10118193-0001LF/609-4616-1-ND/2785380?utm_source=snapeda&amp;utm_medium=aggregator&amp;utm_campaign=symbol" x="-33.147" y="81.248" size="1.778" layer="27" rot="R180" display="off"/>
-<attribute name="MF" value="Amphenol ICC" x="-33.147" y="81.248" size="1.778" layer="27" rot="R180" display="off"/>
-<attribute name="MP" value="10118193-0001LF" x="-33.147" y="81.248" size="1.778" layer="27" rot="R180" display="off"/>
-<attribute name="NAME" x="20.237409375" y="54.53408125" size="1.27" layer="25" rot="R180"/>
-<attribute name="PACKAGE" value="None" x="-33.147" y="81.248" size="1.778" layer="27" rot="R180" display="off"/>
-<attribute name="VALUE" x="20.26908125" y="62.79171875" size="1.27" layer="27" rot="R180"/>
 </element>
 <element name="BLUETOOTH" library="640456-5" package="TE_640456-5" value="640456-5" x="56.388" y="8.382" smashed="yes" rot="R90">
@@
 <element name="TP12" library="SparkFun-Connectors" package="1X01_NO_SILK" value="TEST-POINTPOGO_PTH" x="27.9146" y="23.3426" smashed="yes">
 <attribute name="NAME" x="26.6446" y="24.4856" size="0.6096" layer="25" font="vector" ratio="20"/>
+</element>
+<element name="J2" library="10118194-0001LF" package="AMPHENOL_10118194-0001LF" value="10118194-0001LF" x="15.24" y="58.42" smashed="yes" rot="R180">
+<attribute name="AVAILABILITY" value="Unavailable" x="15.24" y="58.42" size="1.016" layer="27" rot="R180" display="off"/>
+<attribute name="DESCRIPTION" value=" Micro Usb, 2.0 Type b, Rcpt, Smt " x="15.24" y="58.42" size="1.016" layer="27" rot="R180" display="off"/>
+<attribute name="MF" value="Amphenol ICC" x="15.24" y="58.42" size="1.016" layer="27" rot="R180" display="off"/>
+<attribute name="MP" value="10118194-0001LF" x="15.24" y="58.42" size="1.016" layer="27" rot="R180" display="off"/>
+<attribute name="NAME" x="19.28428125" y="54.030859375" size="1.271209375" layer="25" rot="R180"/>
+<attribute name="PACKAGE" value="None" x="15.24" y="58.42" size="1.016" layer="27" rot="R180" display="off"/>
+<attribute name="PRICE" value="None" x="15.24" y="58.42" size="1.016" layer="27" rot="R180" display="off"/>
+<attribute name="VALUE" x="19.70785" y="63.139959375" size="1.270459375" layer="27" rot="R180"/>
 </element>
 </elements>
@@
 </signal>
 <signal name="_12V">
-<contactref element="J1" pad="5"/>
 <contactref element="C9" pad="2"/>
 <contactref element="C11" pad="2"/>
@@
 <wire x1="9.9171" y1="44.2071" x2="9.9171" y2="42.69438125" width="0.6096" layer="1"/>
 <wire x1="11.43" y1="45.72" x2="9.9171" y2="44.2071" width="0.6096" layer="1"/>
-<wire x1="13.97" y1="52.07" x2="13.97" y2="54.61" width="0.6096" layer="1"/>
-<wire x1="13.98" y1="54.61" x2="14.00158125" y2="54.61" width="0.6096" layer="1"/>
-<wire x1="15.083" y1="55.713" x2="13.98" y2="54.61" width="0.6096" layer="1"/>
-<wire x1="13.98" y1="54.61" x2="13.97" y2="54.61" width="0.6096" layer="1"/>
+<contactref element="J2" pad="5"/>
+<wire x1="13.94" y1="55.72" x2="13.97" y2="55.69" width="0.4064" layer="1"/>
+<wire x1="13.97" y1="55.69" x2="13.97" y2="52.07" width="0.4064" layer="1"/>
 </signal>
 <signal name="N$20">
@@
 </signal>
 <signal name="N$11">
-<contactref element="J1" pad="1"/>
 <contactref element="C9" pad="1"/>
 <contactref element="U1" pad="4"/>
@@
 <wire x1="22.86" y1="55.88" x2="21.59" y2="54.61" width="0.3048" layer="1"/>
 <wire x1="17.78" y1="54.61" x2="21.59" y2="54.61" width="0.3048" layer="1"/>
-<wire x1="16.51" y1="53.34" x2="17.78" y2="54.61" width="0.6096" layer="1"/>
+<wire x1="16.51" y1="53.34" x2="17.145" y2="53.975" width="0.6096" layer="1"/>
+<wire x1="17.145" y1="53.975" x2="17.78" y2="54.61" width="0.6096" layer="1"/>
 <wire x1="15.24" y1="53.34" x2="16.51" y2="53.34" width="0.6096" layer="1"/>
-<wire x1="17.683" y1="55.713" x2="17.78" y2="55.616" width="0.6096" layer="1"/>
-<wire x1="17.78" y1="55.616" x2="17.78" y2="54.61" width="0.6096" layer="1"/>
+<contactref element="J2" pad="1"/>
+<wire x1="17.65" y1="54.61" x2="17.78" y2="54.61" width="0.6096" layer="1"/>
+<wire x1="16.54" y1="55.72" x2="16.51" y2="55.69" width="0.4064" layer="1"/>
+<wire x1="16.51" y1="55.69" x2="16.51" y2="54.61" width="0.4064" layer="1"/>
+<wire x1="16.51" y1="54.61" x2="17.145" y2="53.975" width="0.4064" layer="1"/>
 <wire x1="11.4601" y1="42.23" x2="11.43" y2="49.11" width="0" layer="19" extent="1-1"/>
 </signal>
