File: eagle/projects/smartBobber Mother Board/Mother Board Files/motherBoard.brd (EAGLE design)
At the start: 160 x 100 mm, 61 parts, among them J1 10118193-0001LF, J10 640456-5, J11 640456-2, J8 640456-2, J9 640456-3, Q3 2A/20V/150mΩ, Q4 MMBT3904, U1 MCP73831, U2 MT3608, U3 LTC3531ES6-3_3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

Commit message: Updates
Parts:
- removed GLED: (no value), led:LED5MM
- removed J10: 640456-5, 640456-5:TE_640456-5
- removed J11, J8: 640456-2, 640456-2:TE_640456-2
- removed J7: (no value), SparkFun-Connectors:1X06
- removed J9: 640456-3, 640456-3:CONN_640456-3
- removed R13: 2k, SparkFun-Resistors:0805
- added BLUE: 640456-5, 640456-5:TE_640456-5
- added D2: Green, SparkFun:LED-0603
- added PIC: (no value), SparkFun-Connectors:1X06
- added R1: 2k, SparkFun-Resistors:0603
- added SOLENOID, TSTSPPLY: 640456-2, 640456-2:TE_640456-2
- added TEMP: 640456-3, 640456-3:CONN_640456-3
- moved R26 135.2 mm to (45.7, 24.1), turned to 180 degrees
- moved C10 125.1 mm to (34.3, 10.2), flipped to the bottom, turned to 270 degrees
- moved C8 122.9 mm to (39.4, 10.2), flipped to the bottom, turned to 270 degrees
- moved U$6 119.8 mm to (15.2, 16.5)
- moved U$5 119.3 mm to (15.2, 26.7)
- moved D3 103.1 mm to (6.35, 8.89), turned to 180 degrees
- moved R19 103.1 mm to (45.7, 43.2), turned to 90 degrees
- moved R18 101.7 mm to (45.7, 38.1), turned to 180 degrees
- moved Q4 99.9 mm to (39.4, 43.2), turned to 90 degrees
- moved R12 99.2 mm to (54.6, 40.6)
- moved R21 99.0 mm to (17.8, 17.8), flipped to the bottom
- moved R22 98.1 mm to (12.7, 17.8), flipped to the bottom, turned to 180 degrees
- moved R20 94.9 mm to (33.0, 43.2), turned to 270 degrees
- moved C7 93.7 mm to (19.1, 26.7), flipped to the bottom, turned to 90 degrees
- moved U3 88.7 mm to (15.2, 26.7), flipped to the bottom
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Connections:
- removed net LVP: J7.6
- removed net N$2: GLED.K, R14.2
- removed net N$26: R25.1, S3.3, U$8.1
- new net N$1: D2.C, R14.2
- net 3.3V: now also BLUE.2, PIC.2, U3.3; no longer J10.2, J7.2
- net BLUETOOTH_ON/OFF: now also BLUE.5; no longer J10.5
- net DRIVER: now also SOLENOID.1; no longer J8.1
- net GND: now also BLUE.1, PIC.3, SOLENOID.2, TEMP.3, TSTSPPLY.1; no longer J10.1, J11.1, J7.3, J8.2, J9.3
- net MCLR: now also PIC.1, R25.1, S3.3, U$8.1; no longer J7.1
- net N$11: now also D2.A; no longer GLED.A
- net N$9: now also R1.2; no longer R13.2
- net PGC: now also PIC.5, U$8.27; no longer J7.5
- net PGD: now also PIC.4, U$8.28; no longer J7.4
- net RX: now also BLUE.3; no longer J10.3
- net TEMP_DQ: now also TEMP.2; no longer J9.2
- net TX: now also BLUE.4; no longer J10.4
- net VCC: now also TEMP.1, TSTSPPLY.2; no longer J11.2, J9.1
- net _12V: now also R1.1; no longer R13.1
Other:
- board size 160 x 100 mm -> 59.7 x 59.4 mm
