File: eagle/projects/smartBobber Mother Board/Mother Board Files/motherBoard.sch (EAGLE design)
At the start: 61 parts, among them J1 10118193-0001LF, J10 640456-5, J11 640456-2, J8 640456-2, J9 640456-3, Q3 2A/20V/150mΩ, Q4 MMBT3904, U1 MCP73831, U2 MT3608, U3 LTC3531ES6-3_3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

Commit message: Updates
Parts:
- removed GLED: (no value), led:LED5MM
- removed R13: 2k, SparkFun-Resistors:RESISTOR0805
- added D2: Green, SparkFun:LED0603
- added R1: 2k, SparkFun-Resistors:RESISTOR0603
- renumbered J10 to BLUE, J11 to TSTSPPLY, J7 to PIC, J8 to SOLENOID, J9 to TEMP
Connections:
- removed net LVP: PIC.6
- removed net N$2: GLED.C, R14.2
- removed net N$26: R25.1, S3.2, U$8.~MCLR/VPP
- new net N$1: D2.C, R14.2
- net 3.3V: now also U3.VOUT
- net MCLR: now also R25.1, S3.2, U$8.~MCLR/VPP
- net N$11: now also D2.A; no longer GLED.A
- net N$9: now also R1.2; no longer R13.2
- net PGC: now also U$8.RB6/PGC
- net PGD: now also U$8.RB7/PGD
- net _12V: now also R1.1; no longer R13.1
